File: pcb/sensactSe/sensactSe.sch (KiCad schematic (older format))
At the start: 22 parts, among them P1 Input, P2 CONN_01X07, P3 CONN_01X07, P4 CONN_01X01, P5 OUTPUT, U1 TLV70033DDC, U2 STM32F030F4, U3 NUD3124DMT1G, U4 SRV05, U5 DS18B20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

Commit message: sensactSE
Parts:
- added D1: LED, Resistors_SMD:R_0805_HandSoldering, symbol LED
- added R4: k1, Resistors_SMD:R_0805_HandSoldering, symbol R
- added R5: 0R, Resistors_SMD:R_0805_HandSoldering, symbol R
Connections:
- wire segments 113 -> 117
- no-connect marks 2 -> 1
Other:
- note added: "getauscht von 2 auf 3!!!!"
Changed lines of the file:
@@
 	1    0    0    -1
 $EndComp
-Text Label 3300 2050 0    60   ~ 0
+Text Label 3300 2150 0    60   ~ 0
 1Wr
 Text Label 6750 3250 0    60   ~ 0
@@
 	2550 2350 3500 2350
 Wire Wire Line
-	3500 2050 3300 2050
-Wire Wire Line
 	3500 2150 3300 2150
 Wire Wire Line
@@
 	0    1    1    0
 $EndComp
-NoConn ~ 3300 2150
 $Comp
 L R R3
@@
 	-1   0    0    1
 $EndComp
+Text Notes 1950 2000 0    60   ~ 0
+getauscht von 2 auf 3!!!!
+$Comp
+L R R4
+U 1 1 57838637
+P 3500 1150
+F 0 "R4" V 3580 1150 50  0000 C CNN
+F 1 "k1" V 3500 1150 50  0000 C CNN
+F 2 "Resistors_SMD:R_0805_HandSoldering" V 3430 1150 50  0001 C CNN
+F 3 "" H 3500 1150 50  0000 C CNN
+	1    3500 1150
+	1    0    0    -1
+$EndComp
+$Comp
+L LED D1
+U 1 1 57838692
+P 3500 1550
+F 0 "D1" H 3500 1650 50  0000 C CNN
+F 1 "LED" H 3500 1450 50  0000 C CNN
+F 2 "Resistors_SMD:R_0805_HandSoldering" H 3500 1550 50  0001 C CNN
+F 3 "" H 3500 1550 50  0000 C CNN
+	1    3500 1550
+	0    -1   -1   0
+$EndComp
+Wire Wire Line
+	3500 2050 3500 1750
+Wire Wire Line
+	3500 1300 3500 1350
+$Comp
+L +3V3 #PWR034
+U 1 1 57838958
+P 3500 950
+F 0 "#PWR034" H 3500 800 50  0001 C CNN
+F 1 "+3V3" H 3500 1090 50  0000 C CNN
+F 2 "" H 3500 950 50  0000 C CNN
+F 3 "" H 3500 950 50  0000 C CNN
+	1    3500 950
+	1    0    0    -1
+$EndComp
+Wire Wire Line
+	3500 1000 3500 950
+$Comp
+L R R5
+U 1 1 57839365
+P 8850 3000
+F 0 "R5" V 8930 3000 50  0000 C CNN
+F 1 "0R" V 8850 3000 50  0000 C CNN
+F 2 "Resistors_SMD:R_0805_HandSoldering" V 8780 3000 50  0001 C CNN
+F 3 "" H 8850 3000 50  0000 C CNN
+	1    8850 3000
+	1    0    0    -1
+$EndComp
+Wire Wire Line
+	8850 2850 9250 2850
+Wire Wire Line
+	8850 3150 9250 3150
+Text Label 9100 2850 0    60   ~ 0
+1W
+Text Label 9100 3150 0    60   ~ 0
+1Wr
 $EndSCHEMATC

Commit message: sensactSE Changes
Changed lines of the file:
@@
 F 3 "" H 3500 1550 50  0000 C CNN
 	1    3500 1550
-	0    -1   -1   0
+	0    1    1    0
 $EndComp
 Wire Wire Line
@@
 Wire Wire Line
 	3500 1300 3500 1350
-$Comp
-L +3V3 #PWR034
-U 1 1 57838958
-P 3500 950
-F 0 "#PWR034" H 3500 800 50  0001 C CNN
-F 1 "+3V3" H 3500 1090 50  0000 C CNN
-F 2 "" H 3500 950 50  0000 C CNN
-F 3 "" H 3500 950 50  0000 C CNN
-	1    3500 950
-	1    0    0    -1
-$EndComp
 Wire Wire Line
 	3500 1000 3500 950
@@
 Text Label 9100 3150 0    60   ~ 0
 1Wr
+$Comp
+L GND #PWR?
+U 1 1 57922B0D
+P 3500 950
+F 0 "#PWR?" H 3500 700 50  0001 C CNN
+F 1 "GND" H 3500 800 50  0000 C CNN
+F 2 "" H 3500 950 50  0000 C CNN
+F 3 "" H 3500 950 50  0000 C CNN
+	1    3500 950
+	-1   0    0    1
+$EndComp
 $EndSCHEMATC

Commit message: SensactUP gets LIN-Port and alternative 5V Power Supply
Parts:
- D1: symbol LED -> LED-RESCUE-sensactSe
Changed lines of the file:
@@
 EESchema Schematic File Version 2
+LIBS:sensactSe-rescue
 LIBS:power
 LIBS:device
@@
 F 0 "U1" H 1550 1050 50  0000 C CNN
 F 1 "TLV70033DDC" H 1900 1050 50  0000 C CNN
-F 2 "kl_footprints:SOT-23-6_handsolder" H 1800 950 50  0000 C CIN
+F 2 "kl_footprints:SOT-23-6_handsolder" H 1800 1150 50  0000 C CIN
 F 3 "" H 1800 850 50  0000 C CNN
 	1    1800 850
@@
 $EndComp
 $Comp
-L LED D1
+L LED-RESCUE-sensactSe D1
 U 1 1 57838692
 P 3500 1550
