File: pcb/sensactHs/ESDProtection.sch (KiCad schematic (older format))
At the start: 13 parts, among them U10 SRV05

Commit message: new version of sensactHs
Parts:
- R1, R2, R3, R4: footprint Resistors_SMD:R_1206_HandSoldering -> Resistors_SMD:R_0805_HandSoldering
- U5: renamed from U10; footprint kl_footprints:SOT-23-6_handsolder -> sensact:SOT-23-6_handsolder
- renumbered C1 to C5, C2 to C6, C3 to C7, C4 to C8

Commit message: sensactHS Backup
Changed lines of the file:
@@
 AR Path="/54E4FBDE/57EDB284/563891B1" Ref="U19"  Part="1"
 AR Path="/54E4FBDE/57EDB28E/563891B1" Ref="U20"  Part="1"
-F 0 "U5" H 5100 2550 60  0000 C CNN
+F 0 "U15" H 5100 2550 60  0000 C CNN
 F 1 "SRV05" H 5100 2050 60  0000 C CNN
 F 2 "sensact:SOT-23-6_handsolder" H 5100 2300 60  0001 C CNN
@@
 AR Path="/54E4FBDE/57EDB284/56389202" Ref="C62"  Part="1"
 AR Path="/54E4FBDE/57EDB28E/56389202" Ref="C66"  Part="1"
-F 0 "C6" H 6175 3000 50  0000 L CNN
+F 0 "C46" H 6175 3000 50  0000 L CNN
 F 1 "u1" H 6175 2800 50  0000 L CNN
 F 2 "Capacitors_SMD:C_0805_HandSoldering" H 6188 2750 30  0001 C CNN
@@
 AR Path="/54E4FBDE/57EDB284/5638926F" Ref="C64"  Part="1"
 AR Path="/54E4FBDE/57EDB28E/5638926F" Ref="C68"  Part="1"
-F 0 "C8" H 6425 3000 50  0000 L CNN
+F 0 "C48" H 6425 3000 50  0000 L CNN
 F 1 "u1" H 6425 2800 50  0000 L CNN
 F 2 "Capacitors_SMD:C_0805_HandSoldering" H 6438 2750 30  0001 C CNN
@@
 AR Path="/54E4FBDE/57EDB284/56389290" Ref="C61"  Part="1"
 AR Path="/54E4FBDE/57EDB28E/56389290" Ref="C65"  Part="1"
-F 0 "C5" H 6175 1800 50  0000 L CNN
+F 0 "C45" H 6175 1800 50  0000 L CNN
 F 1 "u1" H 6175 1600 50  0000 L CNN
 F 2 "Capacitors_SMD:C_0805_HandSoldering" H 6188 1550 30  0001 C CNN
@@
 AR Path="/54E4FBDE/57EDB284/563892AD" Ref="C63"  Part="1"
 AR Path="/54E4FBDE/57EDB28E/563892AD" Ref="C67"  Part="1"
-F 0 "C7" H 6425 1800 50  0000 L CNN
+F 0 "C47" H 6425 1800 50  0000 L CNN
 F 1 "u1" H 6425 1600 50  0000 L CNN
 F 2 "Capacitors_SMD:C_0805_HandSoldering" H 6438 1550 30  0001 C CNN
@@
 AR Path="/54E4FBDE/57EDB284/563892D2" Ref="R113"  Part="1"
 AR Path="/54E4FBDE/57EDB28E/563892D2" Ref="R121"  Part="1"
-F 0 "R1" V 4330 1900 50  0000 C CNN
+F 0 "R81" V 4330 1900 50  0000 C CNN
 F 1 "4k7" V 4250 1900 50  0000 C CNN
 F 2 "Resistors_SMD:R_0805_HandSoldering" V 4180 1900 30  0001 C CNN
@@
 AR Path="/54E4FBDE/57EDB284/563893A1" Ref="R114"  Part="1"
 AR Path="/54E4FBDE/57EDB28E/563893A1" Ref="R122"  Part="1"
-F 0 "R2" V 4330 2150 50  0000 C CNN
+F 0 "R82" V 4330 2150 50  0000 C CNN
 F 1 "4k7" V 4250 2150 50  0000 C CNN
 F 2 "Resistors_SMD:R_0805_HandSoldering" V 4180 2150 30  0001 C CNN
@@
 AR Path="/54E4FBDE/57EDB284/563893CA" Ref="R115"  Part="1"
 AR Path="/54E4FBDE/57EDB28E/563893CA" Ref="R123"  Part="1"
-F 0 "R3" V 4330 2450 50  0000 C CNN
+F 0 "R83" V 4330 2450 50  0000 C CNN
 F 1 "4k7" V 4250 2450 50  0000 C CNN
 F 2 "Resistors_SMD:R_0805_HandSoldering" V 4180 2450 30  0001 C CNN
@@
 AR Path="/54E4FBDE/57EDB284/563893F1" Ref="R116"  Part="1"
 AR Path="/54E4FBDE/57EDB28E/563893F1" Ref="R124"  Part="1"
-F 0 "R4" V 4330 2700 50  0000 C CNN
+F 0 "R84" V 4330 2700 50  0000 C CNN
 F 1 "4k7" V 4250 2700 50  0000 C CNN
 F 2 "Resistors_SMD:R_0805_HandSoldering" V 4180 2700 30  0001 C CNN
@@
 AR Path="/54E4FBDE/57EDB284/5638941E" Ref="R118"  Part="1"
 AR Path="/54E4FBDE/57EDB28E/5638941E" Ref="R126"  Part="1"
-F 0 "R6" V 5980 2050 50  0000 C CNN
+F 0 "R86" V 5980 2050 50  0000 C CNN
 F 1 "1k" V 5900 2050 50  0000 C CNN
 F 2 "Resistors_SMD:R_0805_HandSoldering" V 5830 2050 30  0001 C CNN
@@
 AR Path="/54E4FBDE/57EDB284/5638944B" Ref="R119"  Part="1"
 AR Path="/54E4FBDE/57EDB28E/5638944B" Ref="R127"  Part="1"
-F 0 "R7" V 5980 2550 50  0000 C CNN
+F 0 "R87" V 5980 2550 50  0000 C CNN
 F 1 "1k" V 5900 2550 50  0000 C CNN
 F 2 "Resistors_SMD:R_0805_HandSoldering" V 5830 2550 30  0001 C CNN
@@
 AR Path="/54E4FBDE/57EDB284/56389478" Ref="R120"  Part="1"
 AR Path="/54E4FBDE/57EDB28E/56389478" Ref="R128"  Part="1"
-F 0 "R8" V 5980 2700 50  0000 C CNN
+F 0 "R88" V 5980 2700 50  0000 C CNN
 F 1 "1k" V 5900 2700 50  0000 C CNN
 F 2 "Resistors_SMD:R_0805_HandSoldering" V 5830 2700 30  0001 C CNN
@@
 AR Path="/54E4FBDE/57EDB284/563894A5" Ref="R117"  Part="1"
 AR Path="/54E4FBDE/57EDB28E/563894A5" Ref="R125"  Part="1"
-F 0 "R5" V 5980 1900 50  0000 C CNN
+F 0 "R85" V 5980 1900 50  0000 C CNN
 F 1 "1k" V 5900 1900 50  0000 C CNN
 F 2 "Resistors_SMD:R_0805_HandSoldering" V 5830 1900 30  0001 C CNN

Commit message: sensact1.0 first ERC ok
Changed lines of the file:
@@
 AR Path="/54E4FBDE/57EDB284/563891B1" Ref="U19"  Part="1"
 AR Path="/54E4FBDE/57EDB28E/563891B1" Ref="U20"  Part="1"
-F 0 "U15" H 5100 2550 60  0000 C CNN
+F 0 "U20" H 5100 2550 60  0000 C CNN
 F 1 "SRV05" H 5100 2050 60  0000 C CNN
 F 2 "sensact:SOT-23-6_handsolder" H 5100 2300 60  0001 C CNN
@@
 AR Path="/54E4FBDE/57EDB284/56389202" Ref="C62"  Part="1"
 AR Path="/54E4FBDE/57EDB28E/56389202" Ref="C66"  Part="1"
-F 0 "C46" H 6175 3000 50  0000 L CNN
+F 0 "C66" H 6175 3000 50  0000 L CNN
 F 1 "u1" H 6175 2800 50  0000 L CNN
 F 2 "Capacitors_SMD:C_0805_HandSoldering" H 6188 2750 30  0001 C CNN
@@
 AR Path="/54E4FBDE/57EDB284/5638926F" Ref="C64"  Part="1"
 AR Path="/54E4FBDE/57EDB28E/5638926F" Ref="C68"  Part="1"
-F 0 "C48" H 6425 3000 50  0000 L CNN
+F 0 "C68" H 6425 3000 50  0000 L CNN
 F 1 "u1" H 6425 2800 50  0000 L CNN
 F 2 "Capacitors_SMD:C_0805_HandSoldering" H 6438 2750 30  0001 C CNN
@@
 AR Path="/54E4FBDE/57EDB284/56389290" Ref="C61"  Part="1"
 AR Path="/54E4FBDE/57EDB28E/56389290" Ref="C65"  Part="1"
-F 0 "C45" H 6175 1800 50  0000 L CNN
+F 0 "C65" H 6175 1800 50  0000 L CNN
 F 1 "u1" H 6175 1600 50  0000 L CNN
 F 2 "Capacitors_SMD:C_0805_HandSoldering" H 6188 1550 30  0001 C CNN
@@
 AR Path="/54E4FBDE/57EDB284/563892AD" Ref="C63"  Part="1"
 AR Path="/54E4FBDE/57EDB28E/563892AD" Ref="C67"  Part="1"
-F 0 "C47" H 6425 1800 50  0000 L CNN
+F 0 "C67" H 6425 1800 50  0000 L CNN
 F 1 "u1" H 6425 1600 50  0000 L CNN
 F 2 "Capacitors_SMD:C_0805_HandSoldering" H 6438 1550 30  0001 C CNN
@@
 AR Path="/54E4FBDE/57EDB284/563892D2" Ref="R113"  Part="1"
 AR Path="/54E4FBDE/57EDB28E/563892D2" Ref="R121"  Part="1"
-F 0 "R81" V 4330 1900 50  0000 C CNN
+F 0 "R121" V 4330 1900 50  0000 C CNN
 F 1 "4k7" V 4250 1900 50  0000 C CNN
 F 2 "Resistors_SMD:R_0805_HandSoldering" V 4180 1900 30  0001 C CNN
@@
 AR Path="/54E4FBDE/57EDB284/563893A1" Ref="R114"  Part="1"
 AR Path="/54E4FBDE/57EDB28E/563893A1" Ref="R122"  Part="1"
-F 0 "R82" V 4330 2150 50  0000 C CNN
+F 0 "R122" V 4330 2150 50  0000 C CNN
 F 1 "4k7" V 4250 2150 50  0000 C CNN
 F 2 "Resistors_SMD:R_0805_HandSoldering" V 4180 2150 30  0001 C CNN
@@
 AR Path="/54E4FBDE/57EDB284/563893CA" Ref="R115"  Part="1"
 AR Path="/54E4FBDE/57EDB28E/563893CA" Ref="R123"  Part="1"
-F 0 "R83" V 4330 2450 50  0000 C CNN
+F 0 "R123" V 4330 2450 50  0000 C CNN
 F 1 "4k7" V 4250 2450 50  0000 C CNN
 F 2 "Resistors_SMD:R_0805_HandSoldering" V 4180 2450 30  0001 C CNN
@@
 AR Path="/54E4FBDE/57EDB284/563893F1" Ref="R116"  Part="1"
 AR Path="/54E4FBDE/57EDB28E/563893F1" Ref="R124"  Part="1"
-F 0 "R84" V 4330 2700 50  0000 C CNN
+F 0 "R124" V 4330 2700 50  0000 C CNN
 F 1 "4k7" V 4250 2700 50  0000 C CNN
 F 2 "Resistors_SMD:R_0805_HandSoldering" V 4180 2700 30  0001 C CNN
@@
 AR Path="/54E4FBDE/57EDB284/5638941E" Ref="R118"  Part="1"
 AR Path="/54E4FBDE/57EDB28E/5638941E" Ref="R126"  Part="1"
-F 0 "R86" V 5980 2050 50  0000 C CNN
+F 0 "R126" V 5980 2050 50  0000 C CNN
 F 1 "1k" V 5900 2050 50  0000 C CNN
 F 2 "Resistors_SMD:R_0805_HandSoldering" V 5830 2050 30  0001 C CNN
@@
 AR Path="/54E4FBDE/57EDB284/5638944B" Ref="R119"  Part="1"
 AR Path="/54E4FBDE/57EDB28E/5638944B" Ref="R127"  Part="1"
-F 0 "R87" V 5980 2550 50  0000 C CNN
+F 0 "R127" V 5980 2550 50  0000 C CNN
 F 1 "1k" V 5900 2550 50  0000 C CNN
 F 2 "Resistors_SMD:R_0805_HandSoldering" V 5830 2550 30  0001 C CNN
@@
 AR Path="/54E4FBDE/57EDB284/56389478" Ref="R120"  Part="1"
 AR Path="/54E4FBDE/57EDB28E/56389478" Ref="R128"  Part="1"
-F 0 "R88" V 5980 2700 50  0000 C CNN
+F 0 "R128" V 5980 2700 50  0000 C CNN
 F 1 "1k" V 5900 2700 50  0000 C CNN
 F 2 "Resistors_SMD:R_0805_HandSoldering" V 5830 2700 30  0001 C CNN
@@
 AR Path="/54E4FBDE/57EDB284/563894A5" Ref="R117"  Part="1"
 AR Path="/54E4FBDE/57EDB28E/563894A5" Ref="R125"  Part="1"
-F 0 "R85" V 5980 1900 50  0000 C CNN
+F 0 "R125" V 5980 1900 50  0000 C CNN
 F 1 "1k" V 5900 1900 50  0000 C CNN
 F 2 "Resistors_SMD:R_0805_HandSoldering" V 5830 1900 30  0001 C CNN
