File: pcb/sensactHs/sensactHs.kicad_pcb (KiCad board)
At the start: 2 copper layers, 100 x 86.5 mm, 185 parts, among them M1 Hole, M2 Hole, P1 CONN_01X08, P2 USB, P3 ESP01, P4 MicroSD, P5 SWD, P6 PWR+CANH, P7 CANH+CANL, P8 !24V!, SW1 PC5-Key, SW2 BOOT0, SW3 RESET, SW4 BOOT1, U1 ULN2803, U10 SRV05, U11 SRV05, U12 SRV05, U13 SRV05, U14 SRV05, U15 SRV05, U16 SRV05, U17 SRV05, U18 PCA9555, U19 PCA9555, U2 DRV8860woPad, U20 DRV8860woPad, U3 DRV8860woPad, U4 STM32F103RG, U5 LM2674, U6 SN65HVD230, U7 PCA9685, U8 DS2482, U9 PCA9685, X1 8MHz

Commit message: new version of sensactHs
Parts:
- removed D16: RED, Resistors_SMD:R_0805_HandSoldering
- removed D17: SS14, kl_footprints:do214ac_handsolder
- removed D18: MBR0540, kl_footprints:do214ac_handsolder
- removed INP4: ROTENC, Pin_Headers:Pin_Header_Straight_1x05
- removed JP3: CAN_TERM, Pin_Headers:Pin_Header_Straight_1x02
- removed P8: !24V!, Pin_Headers:Pin_Header_Straight_1x02
- added C60: u1, Capacitors_SMD:C_0805_HandSoldering, F.Cu at (105.2, 41.9)
- added C61: u1, Capacitors_SMD:C_0805_HandSoldering, B.Cu at (112.8, 52.3)
- added C62: u1, Capacitors_SMD:C_0805_HandSoldering, B.Cu at (115.3, 48.8)
- added C63: u1, Capacitors_SMD:C_0805_HandSoldering, B.Cu at (110.7, 52.3)
- added C64: u1, Capacitors_SMD:C_0805_HandSoldering, B.Cu at (108.2, 48.8)
- added C65: u1, Capacitors_SMD:C_0805_HandSoldering, F.Cu at (110.7, 52.3)
- added C66: u1, Capacitors_SMD:C_0805_HandSoldering, F.Cu at (108.2, 48.8)
- added C67: u1, Capacitors_SMD:C_0805_HandSoldering, F.Cu at (112.8, 52.3)
- added C68: u1, Capacitors_SMD:C_0805_HandSoldering, F.Cu at (115.3, 48.8)
- added C69: u1, Capacitors_SMD:C_0805_HandSoldering, F.Cu at (61.5, 114.6)
- added C70: u1, Capacitors_SMD:C_0805_HandSoldering, F.Cu at (104.6, 122.7)
- added C71: u1, Capacitors_SMD:C_0805_HandSoldering, F.Cu at (61.0, 116.3)
- added C72: u1, Capacitors_SMD:C_0805_HandSoldering, F.Cu at (57.7, 113.0)
- added C73: u1, Capacitors_SMD:C_0805_HandSoldering, F.Cu at (57.7, 115.8)
- added C74: u1, Capacitors_SMD:C_0805_HandSoldering, F.Cu at (71.8, 120.0)
- added C75: 10u, Capacitors_SMD:C_1206_HandSoldering, F.Cu at (58.9, 125.2)
- added C76: 10u, Capacitors_SMD:C_1206_HandSoldering, F.Cu at (52.6, 110.2)
- added C77: 10u, Capacitors_SMD:C_1206_HandSoldering, F.Cu at (58.7, 122.7)
- added C78: 22p, Capacitors_SMD:C_0805_HandSoldering, B.Cu at (65.8, 56.9)
- added C79: 22p, Capacitors_SMD:C_0805_HandSoldering, B.Cu at (65.8, 61.2)
- added C80: u1, Capacitors_SMD:C_0805_HandSoldering, B.Cu at (70.0, 61.5)
- added C81: 2u2, Capacitors_SMD:C_0805_HandSoldering, F.Cu at (49.8, 65.0)
- added C82: 2u2, Capacitors_SMD:C_0805_HandSoldering, F.Cu at (49.4, 57.0)
- added C83: 1u, Capacitors_SMD:C_0805_HandSoldering, F.Cu at (52.1, 60.3)
- added C84: 1u, Capacitors_SMD:C_0805_HandSoldering, F.Cu at (54.9, 65.3)
- added C85: u1, Capacitors_SMD:C_0805_HandSoldering, F.Cu at (58.9, 120.7)
- added C86: u1, Capacitors_SMD:C_0805_HandSoldering, F.Cu at (64.8, 108.2)
- added C87: u1, Capacitors_SMD:C_0805_HandSoldering, F.Cu at (64.5, 110.2)
- added C88: u1, Capacitors_SMD:C_0805_HandSoldering, F.Cu at (104.5, 128.1)
- added C89: 10u, Capacitors_SMD:C_1206_HandSoldering, F.Cu at (104.6, 117.9)
- added C90: 10n, Capacitors_SMD:C_0805_HandSoldering, F.Cu at (64.0, 84.3)
- added C91: 4u7, Capacitors_SMD:C_1206_HandSoldering, F.Cu at (62.0, 130.6)
- added C92: 4u7, Capacitors_SMD:C_1206_HandSoldering, F.Cu at (65.5, 128.3)
- added C93: 10u, Capacitors_SMD:C_1206_HandSoldering, F.Cu at (56.4, 129.3)
- added C94: m1, Capacitors_SMD:C_1206_HandSoldering, F.Cu at (104.6, 115.1)
- added C95: 100n, Capacitors_SMD:C_0805_HandSoldering, F.Cu at (104.5, 131.7)
- added C96: u1, Capacitors_SMD:C_0805_HandSoldering, F.Cu at (104.5, 120.4)
- added C97: u1, Capacitors_SMD:C_0805_HandSoldering, F.Cu at (104.5, 125.2)
- added D1: RED, sensact:LED_5730, F.Cu at (70.4, 42.3)
- added D2: D, sensact:do214ac_handsolder, B.Cu at (63.5, 97.3)
- added D3: MBR0540, sensact:do214ac_handsolder, F.Cu at (60.5, 89.9)
- added INP3: PUSH_BUTTON_INPUT, w_conn_strip:vasch_strip_17x2, F.Cu at (97.8, 24.4)
- added JP1: JUMPER, Pin_Headers:Pin_Header_Straight_1x02, F.Cu at (32.0, 48.3)
- added JP2: CAN_TERM, Pin_Headers:Pin_Header_Straight_1x02, F.Cu at (22.2, 88.8)
- added Q1: Q_NPN_BEC, TO_SOT_Packages_SMD:SOT-23_Handsoldering, F.Cu at (68.7, 46.6)
- added R100: 4k7, Resistors_SMD:R_0805_HandSoldering, B.Cu at (103.1, 29.5)
- added R101: 1k, Resistors_SMD:R_0805_HandSoldering, B.Cu at (103.1, 40.6)
- added R102: 1k, Resistors_SMD:R_0805_HandSoldering, B.Cu at (100.1, 40.6)
- added R103: 1k, Resistors_SMD:R_0805_HandSoldering, B.Cu at (98.0, 37.3)
- added R104: 1k, Resistors_SMD:R_0805_HandSoldering, B.Cu at (105.2, 37.3)
- added R105: 4k7, Resistors_SMD:R_0805_HandSoldering, F.Cu at (98.0, 32.3)
- added R106: 4k7, Resistors_SMD:R_0805_HandSoldering, F.Cu at (105.2, 32.3)
- added R107: 4k7, Resistors_SMD:R_0805_HandSoldering, F.Cu at (103.1, 32.3)
- added R108: 4k7, Resistors_SMD:R_0805_HandSoldering, F.Cu at (100.1, 32.3)
- added R109: 1k, Resistors_SMD:R_0805_HandSoldering, F.Cu at (100.1, 40.6)
- added R110: 1k, Resistors_SMD:R_0805_HandSoldering, F.Cu at (103.1, 40.6)
- added R111: 1k, Resistors_SMD:R_0805_HandSoldering, F.Cu at (105.2, 37.3)
- added R112: 1k, Resistors_SMD:R_0805_HandSoldering, F.Cu at (98.0, 37.3)
- added R113: 4k7, Resistors_SMD:R_0805_HandSoldering, B.Cu at (115.3, 29.5)
- added R114: 4k7, Resistors_SMD:R_0805_HandSoldering, B.Cu at (108.2, 29.5)
- added R115: 4k7, Resistors_SMD:R_0805_HandSoldering, B.Cu at (110.2, 29.5)
- added R116: 4k7, Resistors_SMD:R_0805_HandSoldering, B.Cu at (113.3, 29.5)
- added R117: 1k, Resistors_SMD:R_0805_HandSoldering, B.Cu at (113.3, 47.5)
- added R118: 1k, Resistors_SMD:R_0805_HandSoldering, B.Cu at (110.2, 47.5)
- added R119: 1k, Resistors_SMD:R_0805_HandSoldering, B.Cu at (108.2, 43.9)
- added R120: 1k, Resistors_SMD:R_0805_HandSoldering, B.Cu at (115.3, 43.9)
- added R121: 4k7, Resistors_SMD:R_0805_HandSoldering, F.Cu at (108.2, 32.3)
- added R122: 4k7, Resistors_SMD:R_0805_HandSoldering, F.Cu at (118.6, 32.3)
- added R123: 4k7, Resistors_SMD:R_0805_HandSoldering, F.Cu at (114.8, 31.0)
- added R124: 4k7, Resistors_SMD:R_0805_HandSoldering, F.Cu at (108.2, 37.6)
- added R125: 1k, Resistors_SMD:R_0805_HandSoldering, F.Cu at (110.2, 47.5)
- added R126: 1k, Resistors_SMD:R_0805_HandSoldering, F.Cu at (113.3, 47.5)
- added R127: 1k, Resistors_SMD:R_0805_HandSoldering, F.Cu at (115.3, 43.9)
- added R128: 1k, Resistors_SMD:R_0805_HandSoldering, F.Cu at (108.2, 43.9)
- added R129: 330R, Resistors_SMD:R_1206_HandSoldering, F.Cu at (73.2, 47.8)
- added R130: 1k, Resistors_SMD:R_0805_HandSoldering, B.Cu at (43.9, 52.5)
- added R131: 22R, Resistors_SMD:R_0805_HandSoldering, B.Cu at (29.7, 57.7)
- added R132: 22R, Resistors_SMD:R_0805_HandSoldering, B.Cu at (34.3, 57.7)
- added R133: 10k, Resistors_SMD:R_0805_HandSoldering, F.Cu at (132.1, 35.4)
- added R134: 10k, Resistors_SMD:R_0805_HandSoldering, F.Cu at (129.4, 33.1)
- added R135: 220R, Resistors_SMD:R_0805_HandSoldering, B.Cu at (62.5, 59.4)
- added R136: 10k, Resistors_SMD:R_0805_HandSoldering, F.Cu at (147.6, 34.3)
- added R137: 4k7, Resistors_SMD:R_0805_HandSoldering, F.Cu at (95.0, 74.0)
- added R138: 4k7, Resistors_SMD:R_0805_HandSoldering, B.Cu at (39.2, 81.7)
- added R139: 10k, Resistors_SMD:R_0805_HandSoldering, F.Cu at (144.7, 36.6)
- added R140: 4k7, Resistors_SMD:R_0805_HandSoldering, F.Cu at (95.0, 71.6)
- added R141: 4k7, Resistors_SMD:R_0805_HandSoldering, B.Cu at (34.7, 81.7)
- added R142: 10k, Resistors_SMD:R_0805_HandSoldering, B.Cu at (24.0, 84.6)
- added R143: 120R, Resistors_SMD:R_1206_HandSoldering, B.Cu at (25.4, 97.3)
- added R144: 1k, Resistors_SMD:R_0805_HandSoldering, B.Cu at (42.9, 48.3)
- added R28: 4k7, Resistors_SMD:R_0805_HandSoldering, B.Cu at (89.9, 95.8)
- added R29: 1k, Resistors_SMD:R_0805_HandSoldering, B.Cu at (89.9, 84.8)
- added R82: 4k7, Resistors_SMD:R_0805_HandSoldering, B.Cu at (87.9, 29.5)
- added R83: 4k7, Resistors_SMD:R_0805_HandSoldering, B.Cu at (89.9, 29.5)
- added R84: 4k7, Resistors_SMD:R_0805_HandSoldering, B.Cu at (93.0, 29.5)
- added R85: 1k, Resistors_SMD:R_0805_HandSoldering, B.Cu at (93.0, 40.6)
- added R86: 1k, Resistors_SMD:R_0805_HandSoldering, B.Cu at (89.9, 40.6)
- added R87: 1k, Resistors_SMD:R_0805_HandSoldering, B.Cu at (87.9, 37.3)
- added R88: 1k, Resistors_SMD:R_0805_HandSoldering, B.Cu at (95.0, 37.3)
- added R89: 4k7, Resistors_SMD:R_0805_HandSoldering, F.Cu at (87.9, 32.3)
- added R90: 4k7, Resistors_SMD:R_0805_HandSoldering, F.Cu at (95.0, 32.3)
- added R91: 4k7, Resistors_SMD:R_0805_HandSoldering, F.Cu at (93.0, 32.3)
- added R92: 4k7, Resistors_SMD:R_0805_HandSoldering, F.Cu at (89.9, 32.3)
- added R93: 1k, Resistors_SMD:R_0805_HandSoldering, F.Cu at (89.9, 40.6)
- added R94: 1k, Resistors_SMD:R_0805_HandSoldering, F.Cu at (93.0, 40.6)
- added R95: 1k, Resistors_SMD:R_0805_HandSoldering, F.Cu at (95.0, 37.3)
- added R96: 1k, Resistors_SMD:R_0805_HandSoldering, F.Cu at (87.9, 37.3)
- added R97: 4k7, Resistors_SMD:R_0805_HandSoldering, B.Cu at (105.2, 29.5)
- added R98: 4k7, Resistors_SMD:R_0805_HandSoldering, B.Cu at (98.0, 29.5)
- added R99: 4k7, Resistors_SMD:R_0805_HandSoldering, B.Cu at (100.1, 29.5)
- added U21: DRV8860woPad, sensact:TSSOP-16_4.4x5mm_Pitch0.65mm_handsolder, F.Cu at (41.7, 35.8)
- added U22: DRV8860woPad, sensact:TSSOP-16_4.4x5mm_Pitch0.65mm_handsolder, F.Cu at (51.8, 35.8)
- added U23: DRV8860woPad, sensact:TSSOP-16_4.4x5mm_Pitch0.65mm_handsolder, F.Cu at (62.0, 35.8)
- added U24: ULN2803, sensact:SOIC-18_7.5x11.6mm_Pitch1.27mm_handsolder, B.Cu at (30.0, 36.1)
- added U25: PCA9685, sensact:TSSOP-28_4.4x9.7mm_Pitch0.65mm_handsolder, F.Cu at (103.4, 70.4)
- added U26: STM32F103RG, sensact:LQFP-64_10x10mm_Pitch0.5mm_handsolder, B.Cu at (51.8, 60.2)
- added U27: LM2674, sensact:SOIC-8_3.9x4.9mm_Pitch1.27mm_handsolder, F.Cu at (59.7, 84.1)
- added U28: SN65HVD230, sensact:SOIC-8_3.9x4.9mm_Pitch1.27mm_handsolder, B.Cu at (25.9, 77.7)
- added U29: DS2482, sensact:SOIC-8_3.9x4.9mm_Pitch1.27mm_handsolder, F.Cu at (35.1, 87.9)
- added U30: DS2482, sensact:SOIC-8_3.9x4.9mm_Pitch1.27mm_handsolder, B.Cu at (37.6, 87.9)
- C10, C11, C12, C17, C40, C45, C53, C9, R69, R70, R71: moved to B.Cu
- C13, C14, C15, C41, C49, C5, C57, C58, C6, C7, C8, R77, R78, R79: moved to F.Cu
- C18, C19, C36: value 10u -> u1; footprint Capacitors_SMD:C_1210_HandSoldering -> Capacitors_SMD:C_0805_HandSoldering; moved to B.Cu
- C20: value 22p -> u1; moved to B.Cu
- C21: value 22p -> u1
- C22, C29, C30: value 100n -> u1; moved to F.Cu
- C23, C24: value 2u2 -> u1
- C25: value 100n -> u1; moved to B.Cu
- C26: value 1u -> u1; moved to B.Cu
- C27, C28, C38: value 100n -> u1
- C31, C59: value 10u -> u1; footprint Capacitors_SMD:C_1210_HandSoldering -> Capacitors_SMD:C_0805_HandSoldering
- C32: value 4u7 -> u1; footprint Capacitors_SMD:C_1206_HandSoldering -> Capacitors_SMD:C_0805_HandSoldering
- C33: value 4u7 -> u1; footprint Capacitors_SMD:C_1206_HandSoldering -> Capacitors_SMD:C_0805_HandSoldering; moved to B.Cu
- C34: value 10n -> u1; moved to B.Cu
- C37: value m1 -> u1; footprint Capacitors_SMD:C_1206_HandSoldering -> Capacitors_SMD:C_0805_HandSoldering; moved to B.Cu
- L2: footprint kl_footprints:Inductor_CD104_handsolder -> sensact:Inductor_CD104_handsolder
- O2: value PWM OUTPUTS -> PWM_OUTPUTS; footprint w_conn_strip:vasch_strip_17x2 -> w_conn_strip:vasch_strip_10x2
- P1: value CONN_01X08 -> USB; footprint kl_footprints:KF141R-8p -> Pin_Headers:Pin_Header_Straight_1x04
- P2: value USB -> SWD; footprint Pin_Headers:Pin_Header_Straight_1x04 -> w_conn_strip:vasch_strip_5x2
- P3: value ESP01 -> 2; footprint Pin_Headers:Pin_Header_Straight_2x04 -> sensact:KF141R-3p
- P4: value MicroSD -> 1; footprint Pin_Headers:Pin_Header_Straight_1x08 -> sensact:KF141R-3p
- P5: value SWD -> 3; footprint w_conn_strip:vasch_strip_5x2 -> sensact:KF141R-8p
- P6: value PWR+CANH -> !24V!; footprint kl_footprints:KF141R-3p -> Pin_Headers:Pin_Header_Straight_1x02
- P7: value CANH+CANL -> 5V_IN; footprint kl_footprints:KF141R-3p -> Pin_Headers:Pin_Header_Straight_1x02
- R1, R10, R11, R12, R2, R3, R33, R34, R35, R4, R41, R42, R43, R49, R50, R51, R57, R58, R59, R9: footprint Resistors_SMD:R_1206_HandSoldering -> Resistors_SMD:R_0805_HandSoldering
- R16: value 330R -> 1k; moved to B.Cu
- R17, R18: value 22R -> 4k7; moved to F.Cu
- R19, R20: value 10k -> 4k7; moved to F.Cu
- R21: value 220R -> 1k; moved to F.Cu
- R22, R23, R80: value 4k7 -> 1k; moved to F.Cu
- R24: value 10k -> 1k; moved to F.Cu
- R25, R26: value 10k -> 4k7
- R27: value 120R -> 4k7; footprint Resistors_SMD:R_1206_HandSoldering -> Resistors_SMD:R_0805_HandSoldering
- R32, R48, R64: value 4k7 -> 1k; footprint Resistors_SMD:R_1206_HandSoldering -> Resistors_SMD:R_0805_HandSoldering; moved to B.Cu
- R36, R44, R52, R60: value 1k -> 4k7
- R40, R56: value 4k7 -> 1k; footprint Resistors_SMD:R_1206_HandSoldering -> Resistors_SMD:R_0805_HandSoldering; moved to F.Cu
- R65, R66, R67: footprint Resistors_SMD:R_1206_HandSoldering -> Resistors_SMD:R_0805_HandSoldering; moved to B.Cu
- R68: value 1k -> 4k7; moved to B.Cu
- R72: value 4k7 -> 1k; footprint Resistors_SMD:R_1206_HandSoldering -> Resistors_SMD:R_0805_HandSoldering
- R73, R74, R75: footprint Resistors_SMD:R_1206_HandSoldering -> Resistors_SMD:R_0805_HandSoldering; moved to F.Cu
- R76: value 1k -> 4k7; moved to F.Cu
- U1: value ULN2803 -> PCA9555; footprint kl_footprints:SOIC-18_7.5x11.6mm_Pitch1.27mm_handsolder -> sensact:TSSOP-24_4.4x7.8mm_Pitch0.65mm_handsolder
- U10, U12: footprint kl_footprints:SOT-23-6_handsolder -> sensact:SOT-23-6_handsolder; moved to B.Cu
- U11: footprint kl_footprints:SOT-23-6_handsolder -> sensact:SOT-23-6_handsolder; moved to F.Cu
- U13, U14, U15, U16, U17: footprint kl_footprints:SOT-23-6_handsolder -> sensact:SOT-23-6_handsolder
- U18: value PCA9555 -> SRV05; footprint kl_footprints:TSSOP-24_4.4x7.8mm_Pitch0.65mm_handsolder -> sensact:SOT-23-6_handsolder; moved to F.Cu
- U19: value PCA9555 -> SRV05; footprint kl_footprints:TSSOP-24_4.4x7.8mm_Pitch0.65mm_handsolder -> sensact:SOT-23-6_handsolder
- U2, U3: value DRV8860woPad -> PCA9555; footprint kl_footprints:TSSOP-16_4.4x5mm_Pitch0.65mm_handsolder -> sensact:TSSOP-24_4.4x7.8mm_Pitch0.65mm_handsolder; moved to B.Cu
- U20: value DRV8860woPad -> SRV05; footprint kl_footprints:TSSOP-16_4.4x5mm_Pitch0.65mm_handsolder -> sensact:SOT-23-6_handsolder
- U4: value STM32F103RG -> PCA9555; footprint kl_footprints:LQFP-64_10x10mm_Pitch0.5mm_handsolder -> sensact:TSSOP-24_4.4x7.8mm_Pitch0.65mm_handsolder
- U5: value LM2674 -> SRV05; footprint kl_footprints:SOIC-8_3.9x4.9mm_Pitch1.27mm_handsolder -> sensact:SOT-23-6_handsolder
- U6: value SN65HVD230 -> SRV05; footprint kl_footprints:SOIC-8_3.9x4.9mm_Pitch1.27mm_handsolder -> sensact:SOT-23-6_handsolder
- U7, U9: value PCA9685 -> SRV05; footprint kl_footprints:TSSOP-28_4.4x9.7mm_Pitch0.65mm_handsolder -> sensact:SOT-23-6_handsolder
- U8: value DS2482 -> SRV05; footprint kl_footprints:SOIC-8_3.9x4.9mm_Pitch1.27mm_handsolder -> sensact:SOT-23-6_handsolder
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Connections:
- C1 pad 1: GND -> +3V3
- C1 pad 2: /01 input/ESDProtection1/O1 -> GND
- C10 pad 1: /01 input/ESDProtection3/O4 -> /01 input/ESDProtection2/O4
- C11 pad 2: /01 input/ESDProtection3/O2 -> /01 input/ESDProtection2/O2
- C12 pad 1: /01 input/ESDProtection3/O3 -> /01 input/ESDProtection2/O3
- C13 pad 2: /01 input/ESDProtection4/O1 -> /01 input/ESDProtection3/O1
- C14 pad 1: /01 input/ESDProtection4/O4 -> /01 input/ESDProtection3/O4
- C15 pad 2: /01 input/ESDProtection4/O2 -> /01 input/ESDProtection3/O2
- C16 pad 1: VCC -> /01 input/ESDProtection3/O3
- C17 pad 1: VCC -> GND
- C17 pad 2: GND -> /01 input/ESDProtection4/O1
- C18 pad 1: VCC -> /01 input/ESDProtection4/O4
- C19 pad 1: VCC -> GND
- C19 pad 2: GND -> /01 input/ESDProtection4/O2
- C2 pad 1: /01 input/ESDProtection1/O4 -> +3V3
- C20 pad 1: Net-(C20-Pad1) -> /01 input/ESDProtection4/O3
- C21 pad 1: Net-(C21-Pad1) -> GND
- C21 pad 2: GND -> /01 input/ESDProtection5/O1
- C22 pad 1: /03 cpu/NRST -> /01 input/ESDProtection5/O4
- C23 pad 1: Net-(C23-Pad1) -> GND
- C23 pad 2: GND -> /01 input/ESDProtection5/O2
- C24 pad 1: Net-(C24-Pad1) -> /01 input/ESDProtection5/O3
- C25 pad 1: Net-(C25-Pad1) -> GND
- C25 pad 2: GND -> /01 input/ESDProtection6/O1
- C26 pad 1: Net-(C25-Pad1) -> /01 input/ESDProtection6/O4
- C27 pad 1: +3V3 -> GND
- C27 pad 2: GND -> /01 input/ESDProtection6/O2
- C28 pad 1: +3V3 -> /01 input/ESDProtection6/O3
- C29 pad 1: +3V3 -> GND
- C29 pad 2: GND -> /01 input/ESDProtection7/O1
- C3 pad 1: GND -> +3V3
- C3 pad 2: /01 input/ESDProtection1/O2 -> GND
- C30 pad 1: +3V3 -> /01 input/ESDProtection7/O4
- C31 pad 1: +3V3 -> GND
- C31 pad 2: GND -> /01 input/ESDProtection7/O2
- C32 pad 1: VCC -> /01 input/ESDProtection7/O3
- C33 pad 1: VCC -> GND
- C33 pad 2: GND -> /01 input/ESDProtection8/O1
- C34 pad 1: /04 power/V_SW -> /01 input/ESDProtection8/O4
- C34 pad 2: /04 power/V_CB -> GND
- C35 pad 1: +3V3 -> GND
- C35 pad 2: GND -> /01 input/ESDProtection8/O2
- C36 pad 1: +3V3 -> /01 input/ESDProtection8/O3
- C37 pad 1: +3V3 -> GND
- C37 pad 2: GND -> /01 input/ESDProtection9/O1
- C38 pad 1: +3V3 -> /01 input/ESDProtection9/O4
- C39 pad 1: +3V3 -> GND
- C39 pad 2: GND -> /01 input/ESDProtection9/O2
- C4 pad 1: /01 input/ESDProtection1/O3 -> +3V3
- C40 pad 1: VCC -> /01 input/ESDProtection9/O3
- C41 pad 1: /01 input/ESDProtection4/O3 -> GND
- C41 pad 2: GND -> /01 input/ESDProtection10/O1
- C42 pad 1: GND -> /01 input/ESDProtection10/O4
- C42 pad 2: /01 input/ESDProtection5/O1 -> GND
- C43 pad 1: /01 input/ESDProtection5/O4 -> GND
- C43 pad 2: GND -> /01 input/ESDProtection10/O2
- C44 pad 1: GND -> /01 input/ESDProtection10/O3
- C44 pad 2: /01 input/ESDProtection5/O2 -> GND
- C45 pad 1: /01 input/ESDProtection5/O3 -> GND
- C45 pad 2: GND -> /01 input/ESDProtection11/O1
- C46 pad 1: GND -> /01 input/ESDProtection11/O4
- C46 pad 2: /01 input/ESDProtection6/O1 -> GND
- C47 pad 1: /01 input/ESDProtection6/O4 -> GND
- C47 pad 2: GND -> /01 input/ESDProtection11/O2
- C48 pad 1: GND -> /01 input/ESDProtection11/O3
- C48 pad 2: /01 input/ESDProtection6/O2 -> GND
- C49 pad 1: /01 input/ESDProtection6/O3 -> GND
- C49 pad 2: GND -> /01 input/ESDProtection12/O1
- C5 pad 2: /01 input/ESDProtection2/O1 -> /01 input/ESDProtection1/O1
- C50 pad 1: GND -> /01 input/ESDProtection12/O4
- C50 pad 2: /01 input/ESDProtection7/O1 -> GND
- C51 pad 1: /01 input/ESDProtection7/O4 -> GND
- C51 pad 2: GND -> /01 input/ESDProtection12/O2
- C52 pad 1: GND -> /01 input/ESDProtection12/O3
- C52 pad 2: /01 input/ESDProtection7/O2 -> GND
- C53 pad 1: /01 input/ESDProtection7/O3 -> GND
- C53 pad 2: GND -> /01 input/ESDProtection13/O1
- C54 pad 1: GND -> /01 input/ESDProtection13/O4
- C54 pad 2: /01 input/ESDProtection8/O1 -> GND
- C55 pad 1: /01 input/ESDProtection8/O4 -> GND
- C55 pad 2: GND -> /01 input/ESDProtection13/O2
- C56 pad 1: GND -> /01 input/ESDProtection13/O3
- C56 pad 2: /01 input/ESDProtection8/O2 -> GND
- C57 pad 1: /01 input/ESDProtection8/O3 -> GND
- C57 pad 2: GND -> /01 input/ESDProtection14/O1
- C58 pad 1: +3V3 -> /01 input/ESDProtection14/O4
- C59 pad 1: VCC -> GND
- C59 pad 2: GND -> /01 input/ESDProtection14/O2
- C6 pad 1: /01 input/ESDProtection2/O4 -> /01 input/ESDProtection1/O4
- C7 pad 2: /01 input/ESDProtection2/O2 -> /01 input/ESDProtection1/O2
- C8 pad 1: /01 input/ESDProtection2/O3 -> /01 input/ESDProtection1/O3
- C9 pad 2: /01 input/ESDProtection3/O1 -> /01 input/ESDProtection2/O1
- L1 pad 1: Net-(C25-Pad1) -> Net-(C83-Pad1)
- O1 pad 10: /02 output/O1.8 -> Net-(O1-Pad10)
- O1 pad 3: /02 output/O1.1 -> Net-(O1-Pad3)
- O1 pad 4: /02 output/O1.2 -> Net-(O1-Pad4)
- O1 pad 5: /02 output/O1.3 -> Net-(O1-Pad5)
- O1 pad 6: /02 output/O1.4 -> Net-(O1-Pad6)
- O1 pad 7: /02 output/O1.5 -> Net-(O1-Pad7)
- O1 pad 8: /02 output/O1.6 -> Net-(O1-Pad8)
- O1 pad 9: /02 output/O1.7 -> Net-(O1-Pad9)
- O2 pad 16: Net-(O2-Pad16) -> GND
- O2 pad 17: Net-(O2-Pad17) -> GND
- O2 pad 18: Net-(O2-Pad18) -> GND
- O2 pad 19: Net-(O2-Pad19) -> GND
- O2 pad 20: Net-(O2-Pad20) -> GND
- P1 pad 1: +3V3 -> Net-(P1-Pad1)
- P1 pad 2: /03 cpu/1W -> Net-(P1-Pad2)
- P1 pad 3: SCL2 -> Net-(P1-Pad3)
- P1 pad 4: SDA2 -> GND
- P2 pad 1: Net-(P2-Pad1) -> /03 cpu/NRST
- P2 pad 2: Net-(P2-Pad2) -> /03 cpu/SWDIO
- P2 pad 3: Net-(P2-Pad3) -> GND
- P3 pad 1: /03 cpu/PC10 -> /04 power/CANH
- P3 pad 2: GND -> /04 power/CANH
- P3 pad 3: +3V3 -> /04 power/CANL
- P4 pad 1: +3V3 -> /04 power/CANL
- P4 pad 2: (no net) -> GND
- P4 pad 3: /03 cpu/PC8 -> +5V
- P5 pad 1: /03 cpu/NRST -> +3V3
- P5 pad 2: /03 cpu/SWDIO -> /04 power/1Wa
- P5 pad 3: GND -> SCL2
- P5 pad 4: GND -> SDA2
- P5 pad 5: (no net) -> /04 power/DCF77
- P5 pad 6: /03 cpu/SWCLK -> /04 power/1Wb
- P5 pad 7: +3V3 -> VCC
- P5 pad 8: +3V3 -> GND
- P7 pad 1: /04 power/CANH -> +5V
- P7 pad 2: /04 power/CANL -> GND
- R16 pad 1: GND -> /01 input/ESDProtection2/O4
- R16 pad 2: Net-(D16-Pad1) -> Net-(R12-Pad1)
- R17 pad 1: Net-(P2-Pad2) -> Net-(R17-Pad1)
- R17 pad 2: /03 cpu/PA11 -> /01 input/ESDProtection3/I1
- R18 pad 1: Net-(P2-Pad3) -> Net-(R18-Pad1)
- R18 pad 2: /03 cpu/PA12 -> /01 input/ESDProtection3/I2
- R19 pad 1: /03 cpu/BOOT0 -> Net-(R19-Pad1)
- R19 pad 2: GND -> /01 input/ESDProtection3/I3
- R20 pad 2: /03 cpu/BOOT0 -> /01 input/ESDProtection3/I4
- R21 pad 1: Net-(R21-Pad1) -> /01 input/ESDProtection3/O1
- R21 pad 2: Net-(C21-Pad1) -> Net-(R17-Pad1)
- R22 pad 1: +3V3 -> /01 input/ESDProtection3/O2
- R22 pad 2: SCL2 -> Net-(R18-Pad1)
- R23 pad 1: +3V3 -> /01 input/ESDProtection3/O3
- R23 pad 2: SDA2 -> Net-(R19-Pad1)
- R24 pad 1: Net-(R24-Pad1) -> /01 input/ESDProtection3/O4
- R24 pad 2: /03 cpu/PB2 -> Net-(R20-Pad1)
- R25 pad 1: GND -> Net-(R25-Pad1)
- R25 pad 2: Net-(R24-Pad1) -> /01 input/ESDProtection4/I1
- R26 pad 2: GND -> /01 input/ESDProtection4/I2
- R27 pad 1: Net-(JP3-Pad2) -> Net-(R27-Pad1)
- R27 pad 2: /04 power/CANL -> /01 input/ESDProtection4/I3
- R30 pad 1: Net-(P2-Pad1) -> /01 input/ESDProtection4/O2
- R30 pad 2: /03 cpu/PA15 -> Net-(R26-Pad1)
- R31 pad 1: /01 input/ESDProtection2/O4 -> /01 input/ESDProtection4/O3
- R31 pad 2: Net-(R12-Pad1) -> Net-(R27-Pad1)
- R32 pad 1: Net-(R32-Pad1) -> /01 input/ESDProtection4/O4
- R32 pad 2: /01 input/ESDProtection3/I1 -> Net-(R28-Pad1)
- R33 pad 2: /01 input/ESDProtection3/I2 -> /01 input/ESDProtection5/I1
- R34 pad 2: /01 input/ESDProtection3/I3 -> /01 input/ESDProtection5/I2
- R35 pad 2: /01 input/ESDProtection3/I4 -> /01 input/ESDProtection5/I3
- R36 pad 1: /01 input/ESDProtection3/O1 -> Net-(R36-Pad1)
- R36 pad 2: Net-(R32-Pad1) -> /01 input/ESDProtection5/I4
- R37 pad 1: /01 input/ESDProtection3/O2 -> /01 input/ESDProtection5/O1
- R38 pad 1: /01 input/ESDProtection3/O3 -> /01 input/ESDProtection5/O2
- R39 pad 1: /01 input/ESDProtection3/O4 -> /01 input/ESDProtection5/O3
- R40 pad 1: Net-(R40-Pad1) -> /01 input/ESDProtection5/O4
- R40 pad 2: /01 input/ESDProtection4/I1 -> Net-(R36-Pad1)
- R41 pad 2: /01 input/ESDProtection4/I2 -> /01 input/ESDProtection6/I1
- R42 pad 2: /01 input/ESDProtection4/I3 -> /01 input/ESDProtection6/I2
- R43 pad 2: /01 input/ESDProtection4/I4 -> /01 input/ESDProtection6/I3
- R44 pad 1: /01 input/ESDProtection4/O1 -> Net-(R44-Pad1)
- R44 pad 2: Net-(R40-Pad1) -> /01 input/ESDProtection6/I4
- R45 pad 1: /01 input/ESDProtection4/O2 -> /01 input/ESDProtection6/O1
- R46 pad 1: /01 input/ESDProtection4/O3 -> /01 input/ESDProtection6/O2
- R47 pad 1: /01 input/ESDProtection4/O4 -> /01 input/ESDProtection6/O3
- R48 pad 1: Net-(R48-Pad1) -> /01 input/ESDProtection6/O4
- R48 pad 2: /01 input/ESDProtection5/I1 -> Net-(R44-Pad1)
- R49 pad 2: /01 input/ESDProtection5/I2 -> /01 input/ESDProtection7/I1
- R50 pad 2: /01 input/ESDProtection5/I3 -> /01 input/ESDProtection7/I2
- R51 pad 2: /01 input/ESDProtection5/I4 -> /01 input/ESDProtection7/I3
- R52 pad 1: /01 input/ESDProtection5/O1 -> Net-(R52-Pad1)
- R52 pad 2: Net-(R48-Pad1) -> /01 input/ESDProtection7/I4
- R53 pad 1: /01 input/ESDProtection5/O2 -> /01 input/ESDProtection7/O1
- R54 pad 1: /01 input/ESDProtection5/O3 -> /01 input/ESDProtection7/O2
- R55 pad 1: /01 input/ESDProtection5/O4 -> /01 input/ESDProtection7/O3
- R56 pad 1: Net-(R56-Pad1) -> /01 input/ESDProtection7/O4
- R56 pad 2: /01 input/ESDProtection6/I1 -> Net-(R52-Pad1)
- R57 pad 2: /01 input/ESDProtection6/I2 -> /01 input/ESDProtection8/I1
- R58 pad 2: /01 input/ESDProtection6/I3 -> /01 input/ESDProtection8/I2
- R59 pad 2: /01 input/ESDProtection6/I4 -> /01 input/ESDProtection8/I3
- R60 pad 1: /01 input/ESDProtection6/O1 -> Net-(R60-Pad1)
- R60 pad 2: Net-(R56-Pad1) -> /01 input/ESDProtection8/I4
- R61 pad 1: /01 input/ESDProtection6/O2 -> /01 input/ESDProtection8/O1
- R62 pad 1: /01 input/ESDProtection6/O3 -> /01 input/ESDProtection8/O2
- R63 pad 1: /01 input/ESDProtection6/O4 -> /01 input/ESDProtection8/O3
- R64 pad 1: Net-(R64-Pad1) -> /01 input/ESDProtection8/O4
- R64 pad 2: /01 input/ESDProtection7/I1 -> Net-(R60-Pad1)
- R65 pad 2: /01 input/ESDProtection7/I2 -> /01 input/ESDProtection9/I1
- R66 pad 2: /01 input/ESDProtection7/I3 -> /01 input/ESDProtection9/I2
- R67 pad 2: /01 input/ESDProtection7/I4 -> /01 input/ESDProtection9/I3
- R68 pad 1: /01 input/ESDProtection7/O1 -> Net-(R68-Pad1)
- R68 pad 2: Net-(R64-Pad1) -> /01 input/ESDProtection9/I4
- R69 pad 1: /01 input/ESDProtection7/O2 -> /01 input/ESDProtection9/O1
- R70 pad 1: /01 input/ESDProtection7/O3 -> /01 input/ESDProtection9/O2
- R71 pad 1: /01 input/ESDProtection7/O4 -> /01 input/ESDProtection9/O3
- R72 pad 1: Net-(R72-Pad1) -> /01 input/ESDProtection9/O4
- R72 pad 2: /01 input/ESDProtection8/I1 -> Net-(R68-Pad1)
- R73 pad 2: /01 input/ESDProtection8/I2 -> /01 input/ESDProtection10/I1
- R74 pad 2: /01 input/ESDProtection8/I3 -> /01 input/ESDProtection10/I2
- R75 pad 2: /01 input/ESDProtection8/I4 -> /01 input/ESDProtection10/I3
- R76 pad 1: /01 input/ESDProtection8/O1 -> Net-(R76-Pad1)
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Routing:
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- removed copper zone on F.Cu, net /04 power/V_SW
- removed copper zone on B.Cu, net GND
Other:
- board text added: "Antennenmodul intern?"
- board text added: "sensact 2016-09-30 mail@klaus-liebler.de"
- board text removed: "3V3.....GND"
- board text removed: "B6 B7 C13 3V3 GND"
- board text removed: "GND BOOT0 NRST RX"
- board text removed: "sensact 2015-11-07 mail@klaus-liebler.de"

Commit message: sensactHS intermediate backup
Parts:
- added C100: 10u, Capacitors_SMD:C_1206_HandSoldering, F.Cu at (70.4, 31.1)
- added C101: u1, Capacitors_SMD:C_0805_HandSoldering, F.Cu at (72.0, 35.1)
- added C102: u1, Capacitors_SMD:C_0805_HandSoldering, F.Cu at (31.6, 35.3)
- added C103: u1, Capacitors_SMD:C_0805_HandSoldering, F.Cu at (36.2, 37.1)
- added C98: 10u, Capacitors_SMD:C_1206_HandSoldering, F.Cu at (33.9, 36.1)
- added C99: 10u, Capacitors_SMD:C_1206_HandSoldering, F.Cu at (29.5, 36.1)
- added JP3: JUMPER3, sensact:SMD-solder-bridge-3pin, B.Cu at (36.1, 73.3)
- added JP4: JUMPER3, sensact:SMD-solder-bridge-3pin, B.Cu at (40.6, 73.3)
- added JP5: JUMPER3, sensact:SMD-solder-bridge-3pin, B.Cu at (35.6, 97.3)
- added JP6: JUMPER3, sensact:SMD-solder-bridge-3pin, B.Cu at (43.2, 97.3)
- added O3: POWERED OUTPUTS, w_conn_strip:vasch_strip_17x2, F.Cu at (47.8, 48.3)
- added R145: 1k, Resistors_SMD:R_0805_HandSoldering, F.Cu at (63.6, 58.7)
- added R146, R147: 4k7, Resistors_SMD:R_0805_HandSoldering, F.Cu at (70.0, 116.1)
- added U31: DRV8860woPad, sensact:TSSOP-16_4.4x5mm_Pitch0.65mm_handsolder, B.Cu at (44.2, 40.1)
- added U32: DRV8860woPad, sensact:TSSOP-16_4.4x5mm_Pitch0.65mm_handsolder, B.Cu at (54.5, 40.1)
- added U33: DRV8860woPad, sensact:TSSOP-16_4.4x5mm_Pitch0.65mm_handsolder, B.Cu at (64.6, 40.1)
- R134, R140: moved to B.Cu
- moved INP2 95.3 mm to (89.9, 164.1)
- moved SW2 57.9 mm to (80.9, 63.6)
- moved R134 52.1 mm to (83.8, 58.3)
- moved JP1 17.4 mm to (27.8, 65.2), turned to 90 degrees
- moved R140 14.3 mm to (108.7, 67.7), turned to 180 degrees
- moved R131 14.3 mm to (42.7, 63.6), turned to 90 degrees
- moved R130 14.0 mm to (34.2, 62.5)
- moved Q1 10.9 mm to (69.5, 57.5)
- moved C82 10.9 mm to (50.2, 67.9)
- moved P1 10.8 mm to (32.9, 65.2), turned to 90 degrees
- moved L1 8.73 mm to (57.9, 68.5)
- moved R144 8.60 mm to (41.0, 56.6)
- moved C81 8.36 mm to (54.7, 71.8), turned to 90 degrees
- moved P2 8.05 mm to (32.5, 58.7), turned to 180 degrees
- moved R132 6.83 mm to (39.4, 62.2), turned to 0 degrees
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Connections:
- net /03 cpu/BOOT0 renamed /BOOT0
- net /03 cpu/NRST renamed /NRST
- D2 pad 2: VCC -> (no net)
- O1 pad 1: VCC -> +24V
- O1 pad 2: VCC -> +24V
- O2 pad 16: GND -> Net-(O2-Pad16)
- P3 pad 1: /04 power/CANH -> Net-(P3-Pad1)
- P3 pad 2: /04 power/CANH -> Net-(P3-Pad2)
- P3 pad 3: /04 power/CANL -> Net-(P3-Pad3)
- P4 pad 1: /04 power/CANL -> Net-(P4-Pad1)
- P5 pad 1: +3V3 -> /04 power/CANH
- P5 pad 2: /04 power/1Wa -> /04 power/CANH
- P5 pad 3: SCL2 -> /04 power/CANL
- P5 pad 4: SDA2 -> /04 power/CANL
- P5 pad 5: /04 power/DCF77 -> Net-(JP5-Pad2)
- P5 pad 6: /04 power/1Wb -> /04 power/1Wa
- P5 pad 7: VCC -> /04 power/1Wb
- P5 pad 8: GND -> Net-(JP6-Pad2)
- Q1 pad 1: /03 cpu/PB7 -> Net-(Q1-Pad1)
- U22 pad 2: Net-(U21-Pad6) -> Net-(U22-Pad2)
- U23 pad 2: Net-(U22-Pad6) -> Net-(U23-Pad2)
- U23 pad 6: MISO1 -> Net-(U23-Pad6)
- U24 pad 10: VCC -> +24V
- U24 pad 3: /02 output/PA8 -> PWM6
- U24 pad 4: /02 output/PC9 -> PWM5
- U25 pad 10: Net-(O2-Pad11) -> Net-(O2-Pad12)
- U25 pad 11: Net-(O2-Pad10) -> Net-(O2-Pad11)
- U25 pad 12: Net-(O2-Pad9) -> Net-(O2-Pad10)
- U25 pad 13: Net-(O2-Pad8) -> Net-(O2-Pad9)
- U25 pad 15: (no net) -> Net-(O2-Pad1)
- U25 pad 16: Net-(O2-Pad1) -> Net-(O2-Pad2)
- U25 pad 17: Net-(O2-Pad2) -> Net-(O2-Pad3)
- U25 pad 18: Net-(O2-Pad3) -> Net-(O2-Pad4)
- U25 pad 19: Net-(O2-Pad4) -> Net-(O2-Pad5)
- U25 pad 20: Net-(O2-Pad5) -> Net-(O2-Pad6)
- U25 pad 21: Net-(O2-Pad6) -> Net-(O2-Pad7)
- U25 pad 22: Net-(O2-Pad7) -> Net-(O2-Pad8)
- U25 pad 6: Net-(O2-Pad15) -> Net-(O2-Pad16)
- U25 pad 7: Net-(O2-Pad14) -> Net-(O2-Pad15)
- U25 pad 8: Net-(O2-Pad13) -> Net-(O2-Pad14)
- U25 pad 9: Net-(O2-Pad12) -> Net-(O2-Pad13)
- U26 pad 40: /02 output/PC9 -> /03 cpu/PC9
- U26 pad 41: /02 output/PA8 -> /03 cpu/PA8
- U3 pad 10: /01 input/ESDProtection12/O1 -> /01 input/ESDProtection9/O1
- U3 pad 11: /01 input/ESDProtection11/O2 -> /01 input/ESDProtection10/O2
- U3 pad 13: /01 input/ESDProtection9/O1 -> /01 input/ESDProtection12/O1
- U3 pad 14: /01 input/ESDProtection10/O2 -> /01 input/ESDProtection11/O2
- U3 pad 15: /01 input/ESDProtection10/O3 -> /01 input/ESDProtection11/O3
- U3 pad 16: /01 input/ESDProtection9/O4 -> /01 input/ESDProtection12/O4
- U3 pad 17: /01 input/ESDProtection9/O2 -> /01 input/ESDProtection12/O2
- U3 pad 18: /01 input/ESDProtection10/O1 -> /01 input/ESDProtection11/O1
- U3 pad 19: /01 input/ESDProtection10/O4 -> /01 input/ESDProtection11/O4
- U3 pad 20: /01 input/ESDProtection9/O3 -> /01 input/ESDProtection12/O3
- U3 pad 4: /01 input/ESDProtection11/O4 -> /01 input/ESDProtection10/O4
- U3 pad 5: /01 input/ESDProtection12/O3 -> /01 input/ESDProtection9/O3
- U3 pad 6: /01 input/ESDProtection12/O2 -> /01 input/ESDProtection9/O2
- U3 pad 7: /01 input/ESDProtection11/O1 -> /01 input/ESDProtection10/O1
- U3 pad 8: /01 input/ESDProtection11/O3 -> /01 input/ESDProtection10/O3
- U3 pad 9: /01 input/ESDProtection12/O4 -> /01 input/ESDProtection9/O4
- U4 pad 10: /01 input/ESDProtection16/O1 -> /01 input/ESDProtection13/O3
- U4 pad 11: /01 input/ESDProtection15/O2 -> /01 input/ESDProtection14/O4
- U4 pad 13: /01 input/ESDProtection13/O1 -> /01 input/ESDProtection16/O4
- U4 pad 14: /01 input/ESDProtection14/O2 -> /01 input/ESDProtection15/O3
- U4 pad 15: /01 input/ESDProtection14/O3 -> /01 input/ESDProtection15/O2
- U4 pad 16: /01 input/ESDProtection13/O4 -> /01 input/ESDProtection16/O1
- U4 pad 17: /01 input/ESDProtection13/O2 -> /01 input/ESDProtection16/O2
- U4 pad 18: /01 input/ESDProtection14/O1 -> /01 input/ESDProtection15/O1
- U4 pad 19: /01 input/ESDProtection14/O4 -> /01 input/ESDProtection15/O4
- U4 pad 20: /01 input/ESDProtection13/O3 -> /01 input/ESDProtection16/O3
- U4 pad 4: /01 input/ESDProtection15/O4 -> /01 input/ESDProtection14/O3
- U4 pad 5: /01 input/ESDProtection16/O3 -> /01 input/ESDProtection13/O4
- U4 pad 6: /01 input/ESDProtection16/O2 -> /01 input/ESDProtection13/O1
- U4 pad 7: /01 input/ESDProtection15/O1 -> /01 input/ESDProtection14/O2
- U4 pad 8: /01 input/ESDProtection15/O3 -> /01 input/ESDProtection14/O1
- U4 pad 9: /01 input/ESDProtection16/O4 -> /01 input/ESDProtection13/O2
Routing:
- net SCL1: track 0.00 -> 88.5 mm
- net SDA1: track 0.00 -> 87.1 mm
- net +3V3: track 10.9 -> 93.1 mm, vias 1 -> 4
- net /02 output/PC14: track 0.00 -> 63.9 mm, vias 0 -> 6
- net SCL3: track 0.00 -> 58.2 mm, vias 0 -> 2
- net /02 output/PC9: track 44.6 -> 0.00 mm
- net /02 output/PA8: track 44.4 -> 0.00 mm
- net /02 output/PC7: track 44.6 -> 3.27 mm
- net /02 output/PA10: track 44.0 -> 4.56 mm
- net GND: track 5.66 -> 44.8 mm, vias 1 -> 4
- net /02 output/PA9: track 44.2 -> 5.78 mm
- net SCK1: track 0.00 -> 38.1 mm, vias 0 -> 3
- net /01 input/PC3: track 0.00 -> 38.0 mm, vias 0 -> 2
- net MOSI1: track 0.00 -> 35.4 mm, vias 0 -> 1
- net /04 power/CANL: track 0.00 -> 33.1 mm
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Other:
- board text removed: "TX 3V3 NC 3V3"

Commit message: sensactHS Backup
Parts:
- C1, C100, C101, C2, C3, C4, C73, C74, C76, C77: moved to B.Cu
- moved INP2 93.4 mm to (70.4, 72.8)
- moved C75 91.0 mm to (56.1, 34.3), turned to 90 degrees
- moved C77 90.1 mm to (38.2, 34.9), turned to 90 degrees
- moved C74 85.4 mm to (60.8, 35.3), turned to 90 degrees
- moved C73 80.8 mm to (50.7, 35.3), turned to 90 degrees
- moved C72 77.7 mm to (58.3, 35.3), turned to 90 degrees
- moved C76 76.1 mm to (48.5, 34.3), turned to 90 degrees
- moved C2 50.1 mm to (79.8, 69.1), turned to 180 degrees
- moved C3 36.4 mm to (88.4, 58.9)
- moved C101 31.6 mm to (40.4, 35.9), turned to 90 degrees
- moved C4 28.5 mm to (99.1, 68.8), turned to 180 degrees
- moved C1 23.6 mm to (106.7, 56.5), turned to 0 degrees
- moved C92 22.0 mm to (43.7, 130.6)
- moved C91 18.9 mm to (43.3, 127.8)
- moved C99 16.5 mm to (45.8, 34.2)
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Connections:
- INP2 pad 11: /01 input/PC4 -> /01 input/PA4
- INP2 pad 12: /PB1 -> /01 input/PA5
- INP2 pad 13: /01 input/PB0 -> /01 input/PA3
- INP2 pad 6: /01 input/PA3 -> /PB1
- INP2 pad 7: /01 input/PA4 -> /01 input/PC4
- INP2 pad 8: /01 input/PA5 -> /01 input/PB0
- R145 pad 1: /03 cpu/PB7 -> /01 input/PB7
- U26 pad 58: (no net) -> /01 input/PB6
- U26 pad 59: /03 cpu/PB7 -> /01 input/PB7
- U3 pad 1: /01 input/PC2 -> /01 input/PB7
- U4 pad 1: /01 input/PC3 -> /01 input/PB6
Routing:
- net +3V3: track 93.1 -> 320.2 mm, vias 4 -> 11
- net +24V: track 0.00 -> 75.9 mm, vias 0 -> 3
- net /NRST: track 0.00 -> 54.3 mm, vias 0 -> 2
- net /01 input/PC0: track 0.00 -> 53.4 mm, vias 0 -> 2
- net /02 output/PA10: track 4.56 -> 57.4 mm
- net /02 output/PC7: track 3.27 -> 56.0 mm
- net /02 output/PC6: track 3.09 -> 55.6 mm
- net /02 output/PB14: track 2.72 -> 54.9 mm
- net /02 output/PB15: track 4.18 -> 55.2 mm
- net /02 output/PA9: track 5.78 -> 56.7 mm
- net PWM5: track 0.00 -> 46.9 mm
- net /01 input/PB6: track 0.00 -> 46.2 mm, vias 0 -> 2
- net PWM6: track 1.13 -> 40.0 mm
- net /01 input/PC1: track 0.00 -> 31.7 mm, vias 0 -> 2
- net /01 input/PB7: track 0.00 -> 30.5 mm
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
Commit message: sensact1.0 first ERC ok
Parts:
- removed C70, C71: u1, Capacitors_SMD:C_0805_HandSoldering
- removed P7: 5V_IN, Pin_Headers:Pin_Header_Straight_1x02
- removed R139: 10k, Resistors_SMD:R_0805_HandSoldering
- removed SW1: PC5-Key, Buttons_Switches_ThroughHole:SW_PUSH_SMALL
- removed SW4: BOOT1, Buttons_Switches_ThroughHole:SW_PUSH_SMALL
- added JP7: JUMPER3, sensact:SMD-solder-bridge-3pin, B.Cu at (69.1, 39.2)
- added PWR2: CONN_02X05, w_conn_strip:vasch_strip_5x2, F.Cu at (46.6, 86.0)
- C85, C86, C87, C88, C95, C96, C97, R133, R136, R146, R147: moved to B.Cu
- P6: value !24V! -> CONN_01X04; footprint Pin_Headers:Pin_Header_Straight_1x02 -> Pin_Headers:Pin_Header_Straight_2x02
- X1: value 8MHz -> CRYSTAL_SMD_4pol; footprint Crystals:Crystal_HC49-U_Vertical -> sensact:quartz3225; moved to B.Cu
- moved PWR1 113.6 mm to (37.5, 75.7), turned to 180 degrees
- moved R136 105.8 mm to (50.9, 77.2)
- moved C95 98.7 mm to (26.7, 71.0), turned to 0 degrees
- moved C97 86.2 mm to (30.6, 80.9), turned to 90 degrees
- moved C88 79.1 mm to (47.6, 73.2), turned to 90 degrees
- moved C96 68.6 mm to (42.5, 91.1)
- moved C89 67.0 mm to (54.0, 74.0), turned to 180 degrees
- moved C94 63.8 mm to (54.0, 76.3), turned to 180 degrees
- moved C87 53.7 mm to (46.4, 59.7)
- moved C69 53.6 mm to (96.4, 76.8)
- moved R133 53.4 mm to (85.3, 61.2)
- moved C93 50.7 mm to (54.0, 78.6), turned to 180 degrees
- moved C86 48.2 mm to (61.6, 60.1)
- moved P6 47.8 mm to (71.5, 40.5), turned to 90 degrees
- moved C85 47.4 mm to (60.6, 73.3), turned to 90 degrees
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Connections:
- D2 pad 2: (no net) -> VCC
- P3 pad 1: Net-(P3-Pad1) -> GND
- P3 pad 2: Net-(P3-Pad2) -> GND
- P3 pad 3: Net-(P3-Pad3) -> +3V3
- P4 pad 1: Net-(P4-Pad1) -> +5V
- P4 pad 2: GND -> VCC
- P4 pad 3: +5V -> GND
- P6 pad 1: +24V -> MISO1
- P6 pad 2: GND -> Net-(JP7-Pad1)
- R136 pad 1: Net-(R136-Pad1) -> GND
- R145 pad 1: /01 input/PB7 -> /03 cpu/PC14
- R146 pad 2: (no net) -> SDA3
- R147 pad 2: (no net) -> SCL3
- U21 pad 4: /02 output/PC14 -> /02 output/PC13
- U22 pad 4: /02 output/PC14 -> /02 output/PC13
- U23 pad 4: /02 output/PC14 -> /02 output/PC13
- U26 pad 2: (no net) -> /02 output/PC13
- U26 pad 25: /03 cpu/DCF77 -> (no net)
- U26 pad 3: /02 output/PC14 -> /03 cpu/PC14
- U31 pad 4: /02 output/PC14 -> /02 output/PC13
- U32 pad 4: /02 output/PC14 -> /02 output/PC13
- U33 pad 4: /02 output/PC14 -> /02 output/PC13
- U33 pad 6: MISO1 -> Net-(JP7-Pad2)
- X1 pad 2: Net-(C79-Pad1) -> GND
Routing:
- net GND: track 34.1 -> 223.7 mm, vias 4 -> 45
- net +24V: track 75.9 -> 258.3 mm, vias 3 -> 6
- net +3V3: track 320.2 -> 481.1 mm, vias 11 -> 23
- net /02 output/PC13: track 0.00 -> 83.6 mm, vias 0 -> 7
- net /02 output/PC14: track 63.9 -> 0.00 mm, vias 6 -> 0
- net SCL1: track 77.4 -> 115.9 mm
- net SDA1: track 81.2 -> 111.9 mm
- net +5V: track 0.00 -> 28.4 mm
- net SDA3: track 22.0 -> 37.5 mm, vias 1 -> 2
- net SCK1: track 59.8 -> 74.6 mm
- net Net-(O2-Pad12): track 0.00 -> 13.3 mm
- net Net-(Q1-Pad1): track 0.00 -> 13.3 mm
- net /02 output/O1.32: track 0.00 -> 9.18 mm
- net /02 output/O1.24: track 0.00 -> 9.03 mm
- net /02 output/O1.16: track 0.00 -> 9.03 mm
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- added copper zone on F.Cu, net /04 power/V_SW
- added copper zone on B.Cu, net GND

Commit message: Finalizing sensactHS 1.0
Parts:
- removed JP7: JUMPER3, sensact:SMD-solder-bridge-3pin
- C84: value 1u -> u1
- C95: value 100n -> u1
- moved C80 4.26 mm to (73.9, 59.9)
- moved C79 1.78 mm to (69.7, 62.4)
- moved C96 1.02 mm to (41.5, 91.1), turned to 90 degrees
- moved R135 0.76 mm to (66.5, 65.4)
- moved R122 0.63 mm to (118.0, 32.3)
- moved C100 0.51 mm to (58.7, 33.8)
- moved C75 0.51 mm to (56.1, 33.8)
- moved C76 0.51 mm to (48.5, 33.8)
- moved C102 0.51 mm to (48.0, 34.8)
- moved C72 0.51 mm to (58.3, 34.8)
- moved C73 0.51 mm to (50.7, 34.8)
- moved C74 0.51 mm to (60.8, 34.8)
- moved C86 0.38 mm to (61.6, 59.7)
- moved C99 0.38 mm to (45.8, 33.8)
- moved C69 0.25 mm to (96.6, 76.8)
Connections:
- net Net-(JP2-Pad2) renamed /04 power/CANH2
- P6 pad 2: Net-(JP7-Pad1) -> SCK1
- P6 pad 3: /02 output/PC13 -> Net-(P6-Pad3)
- P6 pad 4: SCK1 -> /02 output/PC13
- U33 pad 6: Net-(JP7-Pad2) -> Net-(P6-Pad3)
Routing:
- net +3V3: track 481.1 -> 463.2 mm, vias 23 -> 26
- net Net-(P6-Pad3): track 0.00 -> 16.3 mm
- net GND: track 223.7 -> 238.2 mm, vias 45 -> 56
- net Net-(JP7-Pad2): track 5.16 -> 0.00 mm
- net /02 output/O3.2: track 4.88 -> 9.14 mm
- net /02 output/O3.18: track 5.07 -> 9.08 mm
- net /02 output/O3.10: track 5.01 -> 9.01 mm
- net SCK1: track 74.6 -> 70.8 mm
- net /04 power/CANL: track 34.5 -> 31.3 mm
- net Net-(JP7-Pad1): track 2.44 -> 0.00 mm
- net SCL3: track 41.4 -> 39.6 mm
- net /02 output/O3.1: track 7.04 -> 8.53 mm
- net /02 output/O3.9: track 7.22 -> 8.66 mm
- net +24V: track 258.3 -> 259.7 mm, vias 6 -> 5
- net Net-(R135-Pad1): track 4.24 -> 5.00 mm
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Other:
- board text added: "3V3 GND"
- board text added: "A3 A4 A6 C4 A2 A0 C2 GND A5 A7 B0 B1 A1 C3"
- board text added: "CH CH CL CL SD 1Wa 1Wb SC GN GN 3V 5V 24 GN"
- board text added: "CLK LAT INP OUT"
- board text added: "EX3V"
- board text added: "GND 5 5 24 24"
- board text added: "I33..64"
- board text added: "ID DM DP GND"
- board text added: "INP1..32"
- board text added: "P1...32"
- board text added: "P33..64"
- board text added: "PWM 1..16 + 4*GND"
- board text added: "TERM"
- board text added: "TX 3V NC GN RE RX 3V CL GN DI"
- board text added: "sensact 2016-10-18 mail@klaus-liebler.de"
- board text removed: "B0 C4 A6 A4 A2 A0 C2 GND B1 A7 A5 A3 A1 C3"
- board text removed: "GND 24V"
- board text removed: "GND 3V3"
- board text removed: "sensact 2016-09-30 mail@klaus-liebler.de"
