File: pcb/sensactInpExt/sensactInpExt.sch (KiCad schematic (older format))
At the start: 70 parts, among them M1 CONN_01X01, M2 CONN_01X01, P2 CONN_02X05, P3 CONN_02X16, P4 CONN_01X02, U1 SRV05, U2 SRV05, U3 SRV05, U4 SRV05, U5 DS2482

Commit message: PCB Order @ smart-prototyping 2017-07-26
Connections:
- wire segments 181 -> 180
- no-connect marks 0 -> 3
Changed lines of the file:
@@
 $EndComp
 Wire Wire Line
-	2750 4400 2750 4250
+	2750 4250 2750 4400
 $Comp
 L +3V3 #PWR032
@@
 	5950 4750 7100 4750
 Wire Wire Line
-	5950 4850 6350 4850
-Wire Wire Line
 	5950 4950 6350 4950
 Wire Wire Line
@@
 L GND #PWR044
 U 1 1 58473327
-P 2650 4800
-F 0 "#PWR044" H 2650 4550 50  0001 C CNN
-F 1 "GND" H 2650 4650 50  0000 C CNN
-F 2 "" H 2650 4800 50  0000 C CNN
-F 3 "" H 2650 4800 50  0000 C CNN
-	1    2650 4800
-	1    0    0    -1
-$EndComp
-Wire Wire Line
-	2750 4800 2650 4800
+P 2000 4800
+F 0 "#PWR044" H 2000 4550 50  0001 C CNN
+F 1 "GND" H 2000 4650 50  0000 C CNN
+F 2 "" H 2000 4800 50  0000 C CNN
+F 3 "" H 2000 4800 50  0000 C CNN
+	1    2000 4800
+	1    0    0    -1
+$EndComp
+Wire Wire Line
+	2750 4800 2000 4800
 $Comp
 L JUMPER JP6
@@
 	1    0    0    -1
 $EndComp
+NoConn ~ 2050 6000
+NoConn ~ 1650 6000
+NoConn ~ 5950 4850
+$Comp
+L PWR_FLAG #FLG045
+U 1 1 5979A999
+P 2750 4300
+F 0 "#FLG045" H 2750 4395 50  0001 C CNN
+F 1 "PWR_FLAG" H 2750 4480 50  0000 C CNN
+F 2 "" H 2750 4300 50  0000 C CNN
+F 3 "" H 2750 4300 50  0000 C CNN
+	1    2750 4300
+	0    -1   -1   0
+$EndComp
+$Comp
+L PWR_FLAG #FLG046
+U 1 1 5979AA37
+P 3450 4700
+F 0 "#FLG046" H 3450 4795 50  0001 C CNN
+F 1 "PWR_FLAG" H 3450 4880 50  0000 C CNN
+F 2 "" H 3450 4700 50  0000 C CNN
+F 3 "" H 3450 4700 50  0000 C CNN
+	1    3450 4700
+	-1   0    0    1
+$EndComp
+Connection ~ 2750 4300
+$Comp
+L PWR_FLAG #FLG047
+U 1 1 5979C0FC
+P 2100 4800
+F 0 "#FLG047" H 2100 4895 50  0001 C CNN
+F 1 "PWR_FLAG" H 2100 4980 50  0000 C CNN
+F 2 "" H 2100 4800 50  0000 C CNN
+F 3 "" H 2100 4800 50  0000 C CNN
+	1    2100 4800
+	1    0    0    -1
+$EndComp
+Connection ~ 2100 4800
+Connection ~ 3450 4700
 $EndSCHEMATC
