File: pcb/RPi_Hat_Template/RPi_GPIO.sch (KiCad schematic (older format))
At the start: 1 part, among them J1 RPi_GPIO

Commit message: sensactPI
sensactPI
Connections:
- net LCD_DC: now also J1.36 (BCM16); no longer J1.33 (BCM13)
- net LCD_PWM: now also J1.37 (BCM26); no longer J1.36 (BCM16)
- net LCD_RES: now also J1.33 (BCM13); no longer J1.37 (BCM26)
Changed lines of the file:
@@
 $Descr A4 11693 8268
 encoding utf-8
-Sheet 2 4
+Sheet 2 5
 Title ""
 Date ""
@@
 NoConn ~ 7300 3500
 $Comp
-L +5V #PWR034
+L +5V #PWR029
 U 1 1 5AA0633D
 P 9250 2750
-F 0 "#PWR034" H 9250 2600 50  0001 C CNN
+F 0 "#PWR029" H 9250 2600 50  0001 C CNN
 F 1 "+5V" H 9250 2890 50  0000 C CNN
 F 2 "" H 9250 2750 50  0000 C CNN
@@
 $EndComp
 $Comp
-L GND #PWR035
+L GND #PWR030
 U 1 1 5AA0636A
 P 9300 2900
-F 0 "#PWR035" H 9300 2650 50  0001 C CNN
+F 0 "#PWR030" H 9300 2650 50  0001 C CNN
 F 1 "GND" H 9300 2750 50  0000 C CNN
 F 2 "" H 9300 2900 50  0000 C CNN
@@
 $EndComp
 $Comp
-L GND #PWR036
+L GND #PWR031
 U 1 1 5AA06380
 P 9250 3300
-F 0 "#PWR036" H 9250 3050 50  0001 C CNN
+F 0 "#PWR031" H 9250 3050 50  0001 C CNN
 F 1 "GND" H 9250 3150 50  0000 C CNN
 F 2 "" H 9250 3300 50  0000 C CNN
@@
 $EndComp
 $Comp
-L GND #PWR037
+L GND #PWR032
 U 1 1 5AA06396
 P 9250 3600
-F 0 "#PWR037" H 9250 3350 50  0001 C CNN
+F 0 "#PWR032" H 9250 3350 50  0001 C CNN
 F 1 "GND" H 9250 3450 50  0000 C CNN
 F 2 "" H 9250 3600 50  0000 C CNN
@@
 $EndComp
 $Comp
-L GND #PWR038
+L GND #PWR033
 U 1 1 5AA063AC
 P 9250 4100
-F 0 "#PWR038" H 9250 3850 50  0001 C CNN
+F 0 "#PWR033" H 9250 3850 50  0001 C CNN
 F 1 "GND" H 9250 3950 50  0000 C CNN
 F 2 "" H 9250 4100 50  0000 C CNN
@@
 $EndComp
 $Comp
-L GND #PWR039
+L GND #PWR034
 U 1 1 5AA063C2
 P 9250 4300
-F 0 "#PWR039" H 9250 4050 50  0001 C CNN
+F 0 "#PWR034" H 9250 4050 50  0001 C CNN
 F 1 "GND" H 9250 4150 50  0000 C CNN
 F 2 "" H 9250 4300 50  0000 C CNN
@@
 $EndComp
 $Comp
-L GND #PWR040
+L GND #PWR035
 U 1 1 5AA063D8
 P 7250 4600
-F 0 "#PWR040" H 7250 4350 50  0001 C CNN
+F 0 "#PWR035" H 7250 4350 50  0001 C CNN
 F 1 "GND" H 7250 4450 50  0000 C CNN
 F 2 "" H 7250 4600 50  0000 C CNN
@@
 $EndComp
 $Comp
-L GND #PWR041
+L GND #PWR036
 U 1 1 5AA063EE
 P 7250 3900
-F 0 "#PWR041" H 7250 3650 50  0001 C CNN
+F 0 "#PWR036" H 7250 3650 50  0001 C CNN
 F 1 "GND" H 7250 3750 50  0000 C CNN
 F 2 "" H 7250 3900 50  0000 C CNN
@@
 $EndComp
 $Comp
-L GND #PWR042
+L GND #PWR037
 U 1 1 5AA06404
 P 7250 3100
-F 0 "#PWR042" H 7250 2850 50  0001 C CNN
+F 0 "#PWR037" H 7250 2850 50  0001 C CNN
 F 1 "GND" H 7250 2950 50  0000 C CNN
 F 2 "" H 7250 3100 50  0000 C CNN
@@
 Text GLabel 7250 4400 0    60   Output ~ 0
 AUDIO_LCK
-Text GLabel 7250 4500 0    60   Output ~ 0
+Text GLabel 7250 4300 0    60   Output ~ 0
 LCD_RES
-Text GLabel 7250 4300 0    60   Output ~ 0
+Text GLabel 9250 4400 2    60   Output ~ 0
 LCD_DC
 Text GLabel 7300 3000 0    60   BiDi ~ 0
 1Wire
-Text GLabel 9250 4400 2    60   Output ~ 0
+Text GLabel 7250 4500 0    60   Output ~ 0
 LCD_PWM
 Wire Wire Line

Commit message: RaspiHat
Connections:
- net labels added: SHUTDOWN
- net labels removed: 1Wire
- wire segments 43 -> 44
Changed lines of the file:
@@
 NoConn ~ 7300 3500
 $Comp
-L +5V #PWR029
+L +5V #PWR044
 U 1 1 5AA0633D
 P 9250 2750
-F 0 "#PWR029" H 9250 2600 50  0001 C CNN
+F 0 "#PWR044" H 9250 2600 50  0001 C CNN
 F 1 "+5V" H 9250 2890 50  0000 C CNN
 F 2 "" H 9250 2750 50  0000 C CNN
@@
 $EndComp
 $Comp
-L GND #PWR030
+L GND #PWR045
 U 1 1 5AA0636A
 P 9300 2900
-F 0 "#PWR030" H 9300 2650 50  0001 C CNN
+F 0 "#PWR045" H 9300 2650 50  0001 C CNN
 F 1 "GND" H 9300 2750 50  0000 C CNN
 F 2 "" H 9300 2900 50  0000 C CNN
@@
 $EndComp
 $Comp
-L GND #PWR031
+L GND #PWR046
 U 1 1 5AA06380
 P 9250 3300
-F 0 "#PWR031" H 9250 3050 50  0001 C CNN
+F 0 "#PWR046" H 9250 3050 50  0001 C CNN
 F 1 "GND" H 9250 3150 50  0000 C CNN
 F 2 "" H 9250 3300 50  0000 C CNN
@@
 $EndComp
 $Comp
-L GND #PWR032
+L GND #PWR047
 U 1 1 5AA06396
 P 9250 3600
-F 0 "#PWR032" H 9250 3350 50  0001 C CNN
+F 0 "#PWR047" H 9250 3350 50  0001 C CNN
 F 1 "GND" H 9250 3450 50  0000 C CNN
 F 2 "" H 9250 3600 50  0000 C CNN
@@
 $EndComp
 $Comp
-L GND #PWR033
+L GND #PWR048
 U 1 1 5AA063AC
 P 9250 4100
-F 0 "#PWR033" H 9250 3850 50  0001 C CNN
+F 0 "#PWR048" H 9250 3850 50  0001 C CNN
 F 1 "GND" H 9250 3950 50  0000 C CNN
 F 2 "" H 9250 4100 50  0000 C CNN
@@
 $EndComp
 $Comp
-L GND #PWR034
+L GND #PWR049
 U 1 1 5AA063C2
 P 9250 4300
-F 0 "#PWR034" H 9250 4050 50  0001 C CNN
+F 0 "#PWR049" H 9250 4050 50  0001 C CNN
 F 1 "GND" H 9250 4150 50  0000 C CNN
 F 2 "" H 9250 4300 50  0000 C CNN
@@
 $EndComp
 $Comp
-L GND #PWR035
+L GND #PWR050
 U 1 1 5AA063D8
 P 7250 4600
-F 0 "#PWR035" H 7250 4350 50  0001 C CNN
+F 0 "#PWR050" H 7250 4350 50  0001 C CNN
 F 1 "GND" H 7250 4450 50  0000 C CNN
 F 2 "" H 7250 4600 50  0000 C CNN
@@
 $EndComp
 $Comp
-L GND #PWR036
+L GND #PWR051
 U 1 1 5AA063EE
 P 7250 3900
-F 0 "#PWR036" H 7250 3650 50  0001 C CNN
+F 0 "#PWR051" H 7250 3650 50  0001 C CNN
 F 1 "GND" H 7250 3750 50  0000 C CNN
 F 2 "" H 7250 3900 50  0000 C CNN
@@
 $EndComp
 $Comp
-L GND #PWR037
+L GND #PWR052
 U 1 1 5AA06404
 P 7250 3100
-F 0 "#PWR037" H 7250 2850 50  0001 C CNN
+F 0 "#PWR052" H 7250 2850 50  0001 C CNN
 F 1 "GND" H 7250 2950 50  0000 C CNN
 F 2 "" H 7250 3100 50  0000 C CNN
@@
 Text GLabel 9250 4400 2    60   Output ~ 0
 LCD_DC
-Text GLabel 7300 3000 0    60   BiDi ~ 0
-1Wire
 Text GLabel 7250 4500 0    60   Output ~ 0
 LCD_PWM
@@
 Wire Wire Line
 	7300 4500 7250 4500
-Text GLabel 7250 3400 0    60   Input ~ 0
+Text GLabel 7250 3000 0    60   Input ~ 0
 INT1_1
 Text GLabel 7250 3200 0    60   Input ~ 0
@@
 Wire Wire Line
 	7300 4300 7250 4300
+Text GLabel 9200 4200 2    60   Output ~ 0
+SHUTDOWN
+Wire Wire Line
+	7300 3000 7250 3000
 $EndSCHEMATC

Commit message: rpihat release candidate
Parts:
- added D4: LED, sensact:LED_0805_handsolder, symbol LED
- added R21: k22, Resistors_SMD:R_0805_HandSoldering, symbol R
Connections:
- wire segments 44 -> 53
- no-connect marks 4 -> 3
Changed lines of the file:
@@
 SDA1
 NoConn ~ 7300 2700
-NoConn ~ 7300 3500
-$Comp
-L +5V #PWR044
+$Comp
+L +5V #PWR052
 U 1 1 5AA0633D
 P 9250 2750
-F 0 "#PWR044" H 9250 2600 50  0001 C CNN
+F 0 "#PWR052" H 9250 2600 50  0001 C CNN
 F 1 "+5V" H 9250 2890 50  0000 C CNN
 F 2 "" H 9250 2750 50  0000 C CNN
@@
 $EndComp
 $Comp
-L GND #PWR045
+L GND #PWR053
 U 1 1 5AA0636A
 P 9300 2900
-F 0 "#PWR045" H 9300 2650 50  0001 C CNN
+F 0 "#PWR053" H 9300 2650 50  0001 C CNN
 F 1 "GND" H 9300 2750 50  0000 C CNN
 F 2 "" H 9300 2900 50  0000 C CNN
@@
 $EndComp
 $Comp
-L GND #PWR046
+L GND #PWR054
 U 1 1 5AA06380
 P 9250 3300
-F 0 "#PWR046" H 9250 3050 50  0001 C CNN
+F 0 "#PWR054" H 9250 3050 50  0001 C CNN
 F 1 "GND" H 9250 3150 50  0000 C CNN
 F 2 "" H 9250 3300 50  0000 C CNN
@@
 $EndComp
 $Comp
-L GND #PWR047
+L GND #PWR055
 U 1 1 5AA06396
 P 9250 3600
-F 0 "#PWR047" H 9250 3350 50  0001 C CNN
+F 0 "#PWR055" H 9250 3350 50  0001 C CNN
 F 1 "GND" H 9250 3450 50  0000 C CNN
 F 2 "" H 9250 3600 50  0000 C CNN
@@
 $EndComp
 $Comp
-L GND #PWR048
+L GND #PWR056
 U 1 1 5AA063AC
 P 9250 4100
-F 0 "#PWR048" H 9250 3850 50  0001 C CNN
+F 0 "#PWR056" H 9250 3850 50  0001 C CNN
 F 1 "GND" H 9250 3950 50  0000 C CNN
 F 2 "" H 9250 4100 50  0000 C CNN
@@
 $EndComp
 $Comp
-L GND #PWR049
+L GND #PWR057
 U 1 1 5AA063C2
 P 9250 4300
-F 0 "#PWR049" H 9250 4050 50  0001 C CNN
+F 0 "#PWR057" H 9250 4050 50  0001 C CNN
 F 1 "GND" H 9250 4150 50  0000 C CNN
 F 2 "" H 9250 4300 50  0000 C CNN
@@
 $EndComp
 $Comp
-L GND #PWR050
+L GND #PWR058
 U 1 1 5AA063D8
 P 7250 4600
-F 0 "#PWR050" H 7250 4350 50  0001 C CNN
+F 0 "#PWR058" H 7250 4350 50  0001 C CNN
 F 1 "GND" H 7250 4450 50  0000 C CNN
 F 2 "" H 7250 4600 50  0000 C CNN
@@
 $EndComp
 $Comp
-L GND #PWR051
+L GND #PWR059
 U 1 1 5AA063EE
 P 7250 3900
-F 0 "#PWR051" H 7250 3650 50  0001 C CNN
+F 0 "#PWR059" H 7250 3650 50  0001 C CNN
 F 1 "GND" H 7250 3750 50  0000 C CNN
 F 2 "" H 7250 3900 50  0000 C CNN
@@
 $EndComp
 $Comp
-L GND #PWR052
+L GND #PWR060
 U 1 1 5AA06404
 P 7250 3100
-F 0 "#PWR052" H 7250 2850 50  0001 C CNN
+F 0 "#PWR060" H 7250 2850 50  0001 C CNN
 F 1 "GND" H 7250 2950 50  0000 C CNN
 F 2 "" H 7250 3100 50  0000 C CNN
@@
 Wire Wire Line
 	9200 4400 9250 4400
-Text GLabel 9250 3500 2    60   Output ~ 0
+Text GLabel 9250 3700 2    60   Output ~ 0
 NRST
 Text GLabel 8900 5150 2    60   Output ~ 0
@@
 Wire Wire Line
 	7300 3200 7250 3200
-Wire Wire Line
-	7300 3400 7250 3400
 NoConn ~ 9250 4500
 NoConn ~ 9550 4450
@@
 Wire Wire Line
 	7300 3000 7250 3000
+Text GLabel 7250 4100 0    60   Output ~ 0
+BOOT0
+Wire Wire Line
+	7300 4100 7250 4100
+$Comp
+L LED D4
+U 1 1 5AD99C6F
+P 6450 3150
+F 0 "D4" H 6450 3250 50  0000 C CNN
+F 1 "LED" H 6450 3050 50  0000 C CNN
+F 2 "sensact:LED_0805_handsolder" H 6450 3150 50  0001 C CNN
+F 3 "" H 6450 3150 50  0000 C CNN
+	1    6450 3150
+	1    0    0    -1
+$EndComp
+$Comp
+L R R21
+U 1 1 5AD99C88
+P 6050 3150
+F 0 "R21" V 6130 3150 50  0000 C CNN
+F 1 "k22" V 6050 3150 50  0000 C CNN
+F 2 "Resistors_SMD:R_0805_HandSoldering" V 5980 3150 50  0001 C CNN
+F 3 "" H 6050 3150 50  0000 C CNN
+	1    6050 3150
+	0    1    1    0
+$EndComp
+Wire Wire Line
+	5900 3350 5900 3150
+Wire Wire Line
+	6200 3150 6300 3150
+Wire Wire Line
+	7300 3500 7300 3450
+Wire Wire Line
+	7300 3450 7250 3450
+Wire Wire Line
+	7250 3450 7250 3400
+Wire Wire Line
+	7250 3400 6600 3400
+Wire Wire Line
+	6600 3400 6600 3150
+Wire Wire Line
+	7300 3400 7300 3350
+Wire Wire Line
+	7300 3350 5900 3350
 $EndSCHEMATC

Commit message: Unspecified
Connections:
- no-connect marks 3 -> 4
Changed lines of the file:
@@
 NoConn ~ 7300 2700
 $Comp
-L +5V #PWR054
+L +5V #PWR056
 U 1 1 5AA0633D
-P 9250 2750
-F 0 "#PWR054" H 9250 2600 50  0001 C CNN
-F 1 "+5V" H 9250 2890 50  0000 C CNN
-F 2 "" H 9250 2750 50  0000 C CNN
-F 3 "" H 9250 2750 50  0000 C CNN
-	1    9250 2750
-	0    1    1    0
-$EndComp
-$Comp
-L GND #PWR055
+P 9600 2700
+F 0 "#PWR056" H 9600 2550 50  0001 C CNN
+F 1 "+5V" H 9600 2840 50  0000 C CNN
+F 2 "" H 9600 2700 50  0000 C CNN
+F 3 "" H 9600 2700 50  0000 C CNN
+	1    9600 2700
+	0    1    1    0
+$EndComp
+$Comp
+L GND #PWR057
 U 1 1 5AA0636A
 P 9300 2900
-F 0 "#PWR055" H 9300 2650 50  0001 C CNN
+F 0 "#PWR057" H 9300 2650 50  0001 C CNN
 F 1 "GND" H 9300 2750 50  0000 C CNN
 F 2 "" H 9300 2900 50  0000 C CNN
@@
 $EndComp
 $Comp
-L GND #PWR056
+L GND #PWR058
 U 1 1 5AA06380
 P 9250 3300
-F 0 "#PWR056" H 9250 3050 50  0001 C CNN
+F 0 "#PWR058" H 9250 3050 50  0001 C CNN
 F 1 "GND" H 9250 3150 50  0000 C CNN
 F 2 "" H 9250 3300 50  0000 C CNN
@@
 $EndComp
 $Comp
-L GND #PWR057
+L GND #PWR059
 U 1 1 5AA06396
 P 9250 3600
-F 0 "#PWR057" H 9250 3350 50  0001 C CNN
+F 0 "#PWR059" H 9250 3350 50  0001 C CNN
 F 1 "GND" H 9250 3450 50  0000 C CNN
 F 2 "" H 9250 3600 50  0000 C CNN
@@
 $EndComp
 $Comp
-L GND #PWR058
+L GND #PWR060
 U 1 1 5AA063AC
 P 9250 4100
-F 0 "#PWR058" H 9250 3850 50  0001 C CNN
+F 0 "#PWR060" H 9250 3850 50  0001 C CNN
 F 1 "GND" H 9250 3950 50  0000 C CNN
 F 2 "" H 9250 4100 50  0000 C CNN
@@
 $EndComp
 $Comp
-L GND #PWR059
+L GND #PWR061
 U 1 1 5AA063C2
 P 9250 4300
-F 0 "#PWR059" H 9250 4050 50  0001 C CNN
+F 0 "#PWR061" H 9250 4050 50  0001 C CNN
 F 1 "GND" H 9250 4150 50  0000 C CNN
 F 2 "" H 9250 4300 50  0000 C CNN
@@
 $EndComp
 $Comp
-L GND #PWR060
+L GND #PWR062
 U 1 1 5AA063D8
 P 7250 4600
-F 0 "#PWR060" H 7250 4350 50  0001 C CNN
+F 0 "#PWR062" H 7250 4350 50  0001 C CNN
 F 1 "GND" H 7250 4450 50  0000 C CNN
 F 2 "" H 7250 4600 50  0000 C CNN
@@
 $EndComp
 $Comp
-L GND #PWR061
+L GND #PWR063
 U 1 1 5AA063EE
 P 7250 3900
-F 0 "#PWR061" H 7250 3650 50  0001 C CNN
+F 0 "#PWR063" H 7250 3650 50  0001 C CNN
 F 1 "GND" H 7250 3750 50  0000 C CNN
 F 2 "" H 7250 3900 50  0000 C CNN
@@
 $EndComp
 $Comp
-L GND #PWR062
+L GND #PWR064
 U 1 1 5AA06404
-P 7250 3100
-F 0 "#PWR062" H 7250 2850 50  0001 C CNN
-F 1 "GND" H 7250 2950 50  0000 C CNN
-F 2 "" H 7250 3100 50  0000 C CNN
-F 3 "" H 7250 3100 50  0000 C CNN
-	1    7250 3100
+P 7000 3100
+F 0 "#PWR064" H 7000 2850 50  0001 C CNN
+F 1 "GND" H 7000 2950 50  0000 C CNN
+F 2 "" H 7000 3100 50  0000 C CNN
+F 3 "" H 7000 3100 50  0000 C CNN
+	1    7000 3100
 	0    1    1    0
 $EndComp
@@
 	9200 4000 9250 4000
 Wire Wire Line
-	7250 3100 7300 3100
+	7000 3100 7300 3100
 Wire Wire Line
 	7250 3900 7300 3900
@@
 Wire Wire Line
 	9200 2900 9300 2900
-Connection ~ 9250 2750
-Wire Wire Line
-	9250 2800 9200 2800
-Wire Wire Line
-	9250 2700 9250 2800
-Wire Wire Line
-	9200 2700 9250 2700
+Connection ~ 9500 2700
+Wire Wire Line
+	9200 2700 9600 2700
 Wire Wire Line
 	7250 2900 7300 2900
@@
 Text GLabel 6500 3750 0    60   Output ~ 0
 LCD_SCLK
-Text GLabel 7100 3700 0    60   Input ~ 0
-LCD_MISO
 Wire Wire Line
 	7250 4400 7300 4400
@@
 	7200 3600 7200 3450
 Wire Wire Line
-	7300 3700 7100 3700
-Wire Wire Line
 	6550 3900 6500 3900
 Wire Wire Line
@@
 Wire Wire Line
 	7150 3550 7150 3700
-Connection ~ 7150 3700
 Wire Wire Line
 	6500 3600 6550 3600
@@
 	7300 3200 7250 3200
 NoConn ~ 9250 4500
-NoConn ~ 9550 4450
 Wire Wire Line
 	7300 4300 7250 4300
@@
 Wire Wire Line
 	7300 3350 5900 3350
+NoConn ~ 7300 4200
+NoConn ~ 9250 3500
+Connection ~ 6600 3150
+Wire Wire Line
+	7150 3700 7300 3700
+Wire Wire Line
+	9200 2800 9500 2800
+Wire Wire Line
+	9500 2800 9500 2700
+$Comp
+L PWR_FLAG #FLG065
+U 1 1 5AF18155
+P 6600 3150
+F 0 "#FLG065" H 6600 3245 50  0001 C CNN
+F 1 "PWR_FLAG" H 6600 3330 50  0000 C CNN
+F 2 "" H 6600 3150 50  0000 C CNN
+F 3 "" H 6600 3150 50  0000 C CNN
+	1    6600 3150
+	1    0    0    -1
+$EndComp
 $EndSCHEMATC
