File: pcb/RPi_Hat_Template/RPi_Hat - Kopie.kicad_pcb (KiCad board)
At the start: 2 copper layers, 84.4 x 56.8 mm, 120 parts, among them J1 RPi_GPIO, P1 24V, P2 IN_OUT, P3 BUS1, P4 CONN_01X06, P5 USB, P6 AUDIO OUT, P7 CONN_02X20, P8 SI7021, U1 MODULE_ST7735_1_8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

Commit message: Unspecified
Parts:
- added D4: LED, sensact:LED_0805_handsolder, F.Cu at (91.1, 49.5)
- added P10: CONN_01X05, Pin_Headers:Pin_Header_Straight_1x05_Pitch2.00mm, F.Cu at (111.3, 56.5)
- added P11: SI7021-2, sensact:MODULE_SI7021, F.Cu at (61.5, 87.8)
- added P12: CONN_01X03, Pin_Headers:Pin_Header_Straight_1x03_Pitch2.00mm, F.Cu at (113.5, 56.5)
- added P13: EXT, Pin_Headers:Pin_Header_Straight_1x04_Pitch1.27mm, F.Cu at (99.0, 48.9)
- added P9: CPU_IO, Pin_Headers:Pin_Header_Straight_1x03_Pitch2.54mm, F.Cu at (96.8, 71.0)
- added R21: k22, Resistors_SMD:R_0805_HandSoldering, F.Cu at (89.2, 49.5)
- added R22: 1k, Resistors_SMD:R_0805_HandSoldering, F.Cu at (95.8, 80.9)
- added R23: 1k, Resistors_SMD:R_0805_HandSoldering, F.Cu at (97.5, 80.9)
- added R6: M1, Resistors_SMD:R_0805_HandSoldering, F.Cu at (103.9, 62.9)
- added SW1: ROTARY_ENCODER_SWITCH, sensact:encoder_alps-ec12d_case, F.Cu at (81.9, 83.7)
- D1, R11, R18: moved to B.Cu
- L8: value Ferrite_Bead_Small -> FB
- P5: footprint Pin_Headers:Pin_Header_Straight_1x03_Pitch2.54mm -> sensact:MicroUsbVertical
- P7: value CONN_02X20 -> EXT_CONN
- P8: value SI7021 -> SI7021-1
- R20: moved to F.Cu
- moved R3 22.6 mm to (70.6, 60.5), turned to 90 degrees
- moved R18 20.3 mm to (128.5, 43.9), turned to 90 degrees
- moved R20 12.2 mm to (67.8, 89.7), turned to 0 degrees
- moved R11 9.27 mm to (106.6, 49.4)
- moved C54 5.97 mm to (76.7, 75.8), turned to 90 degrees
- moved D1 5.22 mm to (102.2, 49.4), turned to 0 degrees
- moved R8 3.84 mm to (86.5, 76.7)
- moved P5 3.69 mm to (107.2, 58.2), turned to 270 degrees
- moved C53 2.62 mm to (78.7, 76.1), turned to 90 degrees
- moved DD1 2.22 mm to (81.8, 83.4)
- moved R19 1.82 mm to (124.8, 65.9)
- moved C22 1.78 mm to (75.9, 48.5)
- moved C55 1.69 mm to (92.2, 77.6)
- moved C56 1.67 mm to (90.2, 76.6)
- moved C3 1.47 mm to (102.2, 54.2), turned to 180 degrees
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Connections:
- J1 pad 15: (no net) -> Net-(J1-Pad15)
- J1 pad 17: (no net) -> Net-(D4-Pad2)
- P5 pad 1: GND -> (no net)
- P7 pad 1: Net-(P7-Pad1) -> +3V3
- P7 pad 12: /IO10 -> /IO8
- P7 pad 14: /IO8 -> /IO10
- P7 pad 2: Net-(P7-Pad1) -> +3V3
- P7 pad 5: +3V3 -> GND
- P7 pad 6: +3V3 -> GND
- U8 pad 14: (no net) -> Net-(P13-Pad4)
- U8 pad 15: (no net) -> Net-(P13-Pad3)
- U8 pad 16: (no net) -> Net-(P13-Pad2)
- U8 pad 17: (no net) -> Net-(P13-Pad1)
- U8 pad 25: (no net) -> PB12
- U8 pad 26: (no net) -> PB13
- U8 pad 27: (no net) -> PB14
- U8 pad 28: (no net) -> PB15
- U8 pad 29: (no net) -> WS2812
- U8 pad 38: (no net) -> ENC_B
- U8 pad 39: (no net) -> ENC_A
- U8 pad 40: (no net) -> ENC_SW
Routing:
- net GND: track 121.3 -> 388.9 mm, vias 19 -> 124
- net ENC_B: track 0.00 -> 54.3 mm, vias 0 -> 1
- net ENC_A: track 0.00 -> 48.4 mm, vias 0 -> 1
- net ENC_SW: track 0.00 -> 31.5 mm, vias 0 -> 1
- net Net-(R18-Pad1): track 6.69 -> 29.9 mm, vias 1 -> 3
- net SCL2: track 39.5 -> 61.8 mm
- net SCL1: track 76.8 -> 57.8 mm
- net SHUTDOWN: track 41.8 -> 23.3 mm
- net SDA2: track 39.0 -> 55.2 mm
- net TX: track 39.6 -> 55.3 mm
- net PB15: track 0.00 -> 12.9 mm, vias 0 -> 1
- net PB14: track 0.00 -> 12.2 mm
- net /IO5: track 10.9 -> 23.1 mm, vias 0 -> 2
- net PB12: track 0.00 -> 12.0 mm
- net WS2812: track 0.00 -> 11.4 mm, vias 0 -> 1
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Other:
- rule trace_min: 0.22 -> 0
- board text added: "24V GND"
- board text added: "3V 24 GN IO15..11. 8..10.7..0, LED8..15.7..0, GN"
- board text added: "3V3 1Wi CAL CAH LIN GND 3V3 24V"
- board text added: "R+ R- L- L+"
- board text added: "SC 3V I1 SD I3 I2 24 24 GN GN"
