File: pcb/sensactHsMini/STM32F407VET.sch (KiCad schematic (older format))
At the start: 16 parts, among them U1 STM32F407VETx, Y1 8MHz

Commit message: updated pcb
Connections:
- net +3V3: now also U1.15 (ADC1_IN10/ADC2_IN10/ADC3_IN10/USB_OTG_HS_ULPI_STP/PC0)
Changed lines of the file:
@@
 Text GLabel 1300 5100 0    60   Input ~ 0
 INT2_3
+$Comp
+L +3V3 #PWR?
+U 1 1 58919782
+P 10450 4600
+F 0 "#PWR?" H 10450 4450 50  0001 C CNN
+F 1 "+3V3" H 10450 4740 50  0000 C CNN
+F 2 "" H 10450 4600 50  0000 C CNN
+F 3 "" H 10450 4600 50  0000 C CNN
+	1    10450 4600
+	0    1    1    0
+$EndComp
+Wire Wire Line
+	10450 4600 10400 4600
+Wire Wire Line
+	10400 4600 10400 4700
 $EndSCHEMATC

Commit message: sesnactHsMini &  RPi Hat
Parts:
- removed L1: Ferrite_Bead, Resistors_SMD:R_1206_HandSoldering, symbol Ferrite_Bead
- removed Y1: 8MHz, Crystals:Crystal_HC49-U_Vertical, symbol Crystal
- added C14: u1, Capacitors_SMD:C_0805_HandSoldering, symbol C
- added D2: D, sensact:sod123_handsolder, symbol D
- added D3: LED, Resistors_SMD:R_0805_HandSoldering, symbol LED
- added P9: BACKUP, Pin_Headers:Pin_Header_Straight_1x02_Pitch2.54mm, symbol CONN_01X02
- added R1: K22, Resistors_SMD:R_0805_HandSoldering, symbol R
- added R2: k1, Resistors_SMD:R_0805_HandSoldering, symbol R
- added Y1: Crystal_GND24, sensact:quartz3225, symbol Crystal_GND24
Connections:
- net labels added: ETH_CRS, ETH_MDC, ETH_MDIO, ETH_RX0, ETH_RX1, ETH_TX0, ETH_TX1, ETH_TXEN, LCD_A0, LCD_CS, LCD_LED, LCD_MOSI, LCD_RESET, LCD_SCK, LIN_RX, LIN_SLP, LIN_TX, OSC_IN, OSC_OUT, OSC_OUT_X, VBAT, VCAP1, VCAP2
- net labels removed: COL, CRS, MDC, MDIO, RXC, RXD0, RXD1, RXD2, RXD3, RXDV, RXER, TXC, TXD0, TXD1, TXD2, TXD3, TXEN
- wire segments 60 -> 72
- no-connect marks 0 -> 40
Other:
- moved on the sheet: C1, C2
