File: pcb/sensactHsExt/sensactHsExt.kicad_pcb (KiCad board)
At the start: 2 copper layers, 86.5 x 70.2 mm, 163 parts, among them J2 CONN_LINKS1, J3 SO8, J4 SensactBusConnector, J5 PROG, J6 CONN_LINKS2, J7 SO8, J8 USB_C_Receptacle_USB2.0, SW1 Reset, SW2 SW_Push, SW3 Mitsumi_SIQ-02FVS3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

Commit message: sensactHSExt and sensactAudioExt
Parts:
- removed Z115, Z116, Z117, Z118, Z119, Z120, Z121: StripRow3, sensact:StripRow3
- added C17: u1, Capacitor_SMD:C_0805_2012Metric_Pad1.15x1.40mm_HandSolder, B.Cu at (94.1, 53.5)
- added J1: B3, TestPoint:TestPoint_Pad_2.5x2.5mm, F.Cu at (88.8, 48.5)
- added J10: B5, TestPoint:TestPoint_Pad_2.5x2.5mm, F.Cu at (88.8, 52.2)
- added J11: B6, TestPoint:TestPoint_Pad_2.5x2.5mm, F.Cu at (96.4, 48.5)
- added J12: B7, TestPoint:TestPoint_Pad_2.5x2.5mm, F.Cu at (96.4, 52.2)
- added J13: A15, TestPoint:TestPoint_Pad_2.5x2.5mm, F.Cu at (92.6, 48.5)
- added J14: Conn_01x04, sensact:PhoenixContact_MC_0,5_4-G-2.5_1x04_P2.50mm_Horizontal, B.Cu at (135.9, 91.3)
- added J15: P0A, TestPoint:TestPoint_Pad_2.5x2.5mm, F.Cu at (107.8, 53.3)
- added J16: P0W, TestPoint:TestPoint_Pad_2.5x2.5mm, F.Cu at (104.0, 53.3)
- added J17: P0B, TestPoint:TestPoint_Pad_2.5x2.5mm, F.Cu at (100.2, 53.3)
- added J18: P1A, TestPoint:TestPoint_Pad_2.5x2.5mm, F.Cu at (107.8, 49.8)
- added J19: P1W, TestPoint:TestPoint_Pad_2.5x2.5mm, F.Cu at (104.0, 49.8)
- added J20: P1B, TestPoint:TestPoint_Pad_2.5x2.5mm, F.Cu at (100.2, 49.8)
- added J9: B4, TestPoint:TestPoint_Pad_2.5x2.5mm, F.Cu at (92.6, 52.2)
- added JP1: 3V3_INT, Jumper:SolderJumper-2_P1.3mm_Open_Pad1.0x1.5mm, F.Cu at (132.3, 87.1)
- added U5: MCP42010, sensact:SOIC-14_3.9x8.7mm_P1.27mm_handsolder, B.Cu at (100.7, 51.1)
- added Z3: StripRow3, sensact:StripRow3, F.Cu at (128.3, 82.5)
- added Z4: StripRow3, sensact:StripRow3, F.Cu at (128.3, 74.9)
- added Z5: StripRow3, sensact:StripRow3, F.Cu at (128.3, 67.3)
- C10, C11, C8, D1, R1, R10, R7, R8: moved to F.Cu
- C12, C13, C14, C2, C9, D2, L1, R17, U3: moved to B.Cu
- J2: value CONN_LINKS1 -> LINKS1
- J6: value CONN_LINKS2 -> LINKS2; footprint sensact:PhoenixContact_FFKDS_1x08_P2.54mm -> sensact:PhoenixContact_MC_0,5_8-G-2.5_1x08_P2.50mm_Horizontal
- moved Z110 44.5 mm to (115.6, 87.6)
- moved Z41 41.9 mm to (100.3, 95.2)
- moved Z83 41.7 mm to (100.3, 77.5)
- moved Z67 39.6 mm to (123.2, 72.4)
- moved C14 34.5 mm to (126.7, 88.0), turned to 0 degrees
- moved C13 32.0 mm to (122.3, 88.3)
- moved L1 31.3 mm to (124.0, 93.2), turned to 0 degrees
- moved Z96 30.6 mm to (123.2, 74.9)
- moved Z81 25.4 mm to (123.2, 69.8)
- moved C9 24.8 mm to (131.4, 96.8), turned to 0 degrees
- moved C12 24.7 mm to (129.2, 91.2), turned to 90 degrees
- moved D2 23.6 mm to (131.3, 94.4), turned to 0 degrees
- moved R13 23.0 mm to (136.1, 86.9), turned to 0 degrees
- moved U3 22.9 mm to (132.1, 91.2), turned to 270 degrees
- moved R14 21.8 mm to (136.1, 88.9)
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Connections:
- net Net-(C12-Pad1) renamed /SW
- net Net-(C12-Pad2) renamed /CB
- net Net-(R13-Pad2) renamed /FB
- J4 pad 1: (no net) -> Net-(J4-Pad1)
- R3 pad 2: Net-(R3-Pad2) -> VBUS
- R4 pad 1: Net-(R3-Pad2) -> VBUS
- SW3 pad M: Net-(SW3-PadM) -> (no net)
- U1 pad MP: Net-(U1-PadMP) -> (no net)
- U2 pad 10: ROTA -> ROTB
- U2 pad 11: ROTB -> ROTA
- U2 pad 13: (no net) -> LCDRS
- U2 pad 14: (no net) -> /INT2
- U2 pad 16: /INT2 -> LCDCS
- U2 pad 25: (no net) -> SPI2_CS_POTI
- U2 pad 26: (no net) -> SPI2_CLK
- U2 pad 28: (no net) -> SPI2_MOSI
- U2 pad 29: (no net) -> VBUS
- U2 pad 3: LCDRS -> (no net)
- U2 pad 38: (no net) -> Net-(J13-Pad1)
- U2 pad 39: (no net) -> Net-(J1-Pad1)
- U2 pad 4: LCDCS -> (no net)
- U2 pad 40: (no net) -> Net-(J9-Pad1)
- U2 pad 41: (no net) -> Net-(J10-Pad1)
- U2 pad 42: (no net) -> Net-(J11-Pad1)
- U2 pad 43: (no net) -> Net-(J12-Pad1)
- U4 pad 6: (no net) -> /CANL
- U4 pad 7: (no net) -> /CANH
Routing:
- net +3V3: track 8.97 -> 218.4 mm, vias 0 -> 5
- net /CANL: track 0.00 -> 96.3 mm
- net /CANH: track 0.00 -> 95.8 mm
- net /SCL: track 0.00 -> 83.6 mm, vias 0 -> 1
- net /SDA: track 0.00 -> 82.2 mm, vias 0 -> 1
- net /NRST: track 0.00 -> 79.1 mm, vias 0 -> 4
- net Net-(Z69-Pad1): track 82.5 -> 5.08 mm
- net /USB-: track 0.00 -> 67.7 mm
- net /USB+: track 0.00 -> 63.4 mm
- net VBUS: track 0.00 -> 60.7 mm, vias 0 -> 1
- net /INT1: track 31.4 -> 84.0 mm, vias 0 -> 1
- net /INT0: track 42.2 -> 91.3 mm, vias 0 -> 1
- net /INT2: track 30.5 -> 79.5 mm, vias 0 -> 1
- net +24V: track 0.00 -> 43.4 mm
- net GND: track 0.00 -> 37.9 mm, vias 0 -> 52
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- added copper zone on B.Cu, net GND
- added copper zone on F.Cu, net GND
Other:
- outline, holes or cut-outs redrawn
- net class HighVoltage added: clearance 0.3, trace_width 0.2, via_dia 0.6, via_drill 0.3
- rule trace_min: 0.0889 -> 0
- board text added: "24V"
- board text added: "3V3"
- board text added: "GND"
