File: pcb/sensactHsExt/sensactHsExt.sch (KiCad schematic (older format))
At the start: 85 parts, among them J2 LINKS1, J3 SO8, J4 SensactBusConnector, J5 PROG, J6 LINKS2, J7 SO8, J8 USB_C_Receptacle_USB2.0, SW1 Reset, SW2 SW_Push, SW3 Mitsumi_SIQ-02FVS3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

Commit message: sensactHSExt and sensactAudioExt
Parts:
- added J1: B3, TestPoint:TestPoint_Pad_2.5x2.5mm, symbol Connector_Generic:Conn_01x01
- added J10: B5, TestPoint:TestPoint_Pad_2.5x2.5mm, symbol Connector_Generic:Conn_01x01
- added J11: B6, TestPoint:TestPoint_Pad_2.5x2.5mm, symbol Connector_Generic:Conn_01x01
- added J12: B7, TestPoint:TestPoint_Pad_2.5x2.5mm, symbol Connector_Generic:Conn_01x01
- added J13: A15, TestPoint:TestPoint_Pad_2.5x2.5mm, symbol Connector_Generic:Conn_01x01
- added J14: Conn_01x04, sensact:PhoenixContact_MC_0,5_4-G-2.5_1x04_P2.50mm_Horizontal, symbol Connector_Generic:Conn_01x04
- added J15: P0A, TestPoint:TestPoint_Pad_2.5x2.5mm, symbol Connector_Generic:Conn_01x01
- added J16: P0W, TestPoint:TestPoint_Pad_2.5x2.5mm, symbol Connector_Generic:Conn_01x01
- added J17: P0B, TestPoint:TestPoint_Pad_2.5x2.5mm, symbol Connector_Generic:Conn_01x01
- added J18: P1A, TestPoint:TestPoint_Pad_2.5x2.5mm, symbol Connector_Generic:Conn_01x01
- added J19: P1W, TestPoint:TestPoint_Pad_2.5x2.5mm, symbol Connector_Generic:Conn_01x01
- added J20: P1B, TestPoint:TestPoint_Pad_2.5x2.5mm, symbol Connector_Generic:Conn_01x01
- added J9: B4, TestPoint:TestPoint_Pad_2.5x2.5mm, symbol Connector_Generic:Conn_01x01
- J6: footprint sensact:PhoenixContact_FFKDS_1x08_P2.54mm -> sensact:PhoenixContact_MC_0,5_8-G-2.5_1x08_P2.50mm_Horizontal
- JP1: renamed from JP?; footprint (none) -> Jumper:SolderJumper-2_P1.3mm_Open_Pad1.0x1.5mm
- U5: footprint (none) -> sensact:SOIC-14_3.9x8.7mm_P1.27mm_handsolder
Connections:
- net labels added: CANH, CANL, CB, FB, SPI2_CS_POTI, SW
- wire segments 90 -> 93
- no-connect marks 5 -> 9
