File: pcb/sensactAudioExt/sensactAudioExt.kicad_pcb (KiCad board)
At the start: 2 copper layers, 86.5 x 70.2 mm, 92 parts, among them J1 Conn_01x08, J11 USB_C_Receptacle_USB2.0, J12 USB_C_Receptacle_USB2.0, J2 Audio Out, J3 Conn_01x08, J6 B6, J7 B7, J8 SensactBusConnector, SW1 SW_Push, SW2 SW_Push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

Commit message: sensactHsIO RC1 and sensactAudioExt, RC1
Parts:
- moved U5 2.06 mm to (91.5, 39.0)
Routing:
- net +3V3: track 210.9 -> 215.8 mm
- net /hmi/NRST: track 39.3 -> 36.9 mm
- net SPI_CLK: track 4.37 -> 6.52 mm
- net SPI_MOSI: track 3.85 -> 5.95 mm
- net LCDRS: track 15.4 -> 17.3 mm
- net LCDCS: track 5.44 -> 6.46 mm
- net Net-(R20-Pad1): track 12.6 -> 11.7 mm
- net GND: vias 108 -> 115
- net Net-(R12-Pad2): vias 0 -> 1
