File: pcb/sensactHsIO/hmi.sch (KiCad schematic (older format))
At the start: 49 parts, among them J11 USB_C_Receptacle_USB2.0, J12 USB_C_Receptacle_USB2.0, J8 SensactBusConnector, SW5 Reset, SW6 SW_Push, SW7 Mitsumi_SIQ-02FVS3, U3 STM32F072RBTx, U4 LMR14206, U5 FP-096H09A, U6 SN65HVD230

Commit message: KiCad sensactHsIO
Connections:
- net labels added: SCL1, SCL2, SDA1, SDA2
- net labels removed: SCL, SDA, SPIB_CS
Changed lines of the file:
@@
 Text Label 2700 2150 0    50   ~ 0
 RX
-Text Label 2700 3850 0    50   ~ 0
-SCL
-Text Label 2700 3950 0    50   ~ 0
-SDA
 $Comp
 L Device:LED D1
@@
 	0    1    1    0
 $EndComp
-Text Label 1250 6750 0    50   ~ 0
-SCL
-Text Label 1250 6850 0    50   ~ 0
-SDA
 Wire Wire Line
 	1200 6750 1450 6750
@@
 Text GLabel 650  2450 3    50   Input ~ 0
 LED
-Text GLabel 1300 3850 0    50   Output ~ 0
+Text GLabel 850  4400 0    50   Output ~ 0
 LED
 Wire Wire Line
@@
 Text GLabel 2700 4350 2    50   Output ~ 0
 SPIB_MOSI
-Text GLabel 2700 4050 2    50   Output ~ 0
-SPIB_CS
 Text GLabel 10100 2750 0    50   Input ~ 0
 LCD_CLK
@@
 Connection ~ 2100 4550
 Connection ~ 2200 4550
-Text GLabel 2700 3550 2    50   Output ~ 0
-LCD_BL
 $Comp
 L sensact:FP-096H09A U5
@@
 	1    0    0    -1
 $EndComp
-Text GLabel 2700 3450 2    50   Output ~ 0
-LCD_RS
 Text GLabel 2700 4250 2    50   Input ~ 0
 SPIB_MISO
@@
 	1    0    0    -1
 $EndComp
-Text GLabel 1300 4050 0    50   Output ~ 0
-LCD_RST
 Text GLabel 10100 2450 0    50   Input ~ 0
 LCD_RST
@@
 	10100 2850 9450 2850
 Connection ~ 9450 2850
-Text GLabel 1300 2650 0    50   Input ~ 0
-S
 $Comp
 L power:GND #PWR0109
@@
 	1    0    0    -1
 $EndComp
+Text GLabel 2700 3450 2    50   BiDi ~ 0
+SCL1
+Text GLabel 2700 3550 2    50   BiDi ~ 0
+SDA1
+Text GLabel 2700 3850 2    50   BiDi ~ 0
+SCL2
+Text GLabel 2700 3950 2    50   BiDi ~ 0
+SDA2
+Text GLabel 1450 6750 2    50   BiDi ~ 0
+SCL1
+Text GLabel 1450 6850 2    50   BiDi ~ 0
+SDA1
+Text GLabel 1300 3850 0    50   Input ~ 0
+S
+Text GLabel 1300 3950 0    50   Output ~ 0
+LCD_RS
+Text GLabel 1300 4050 0    50   Output ~ 0
+LCD_RST
+Text GLabel 1300 2650 0    50   Output ~ 0
+LCD_BL
 $EndSCHEMATC

Commit message: sensactHsIO as ordered at JLCPBC (last minute changes)
Parts:
- J8: value SensactBusConnector -> SensactBus
Changed lines of the file:
@@
 P 900 7100
 F 0 "J8" H 958 7865 50  0000 C CNN
-F 1 "SensactBusConnector" H 958 7774 50  0000 C CNN
+F 1 "SensactBus" H 958 7774 50  0000 C CNN
 F 2 "Connector_IDC:IDC-Header_2x05_P2.54mm_Horizontal" H 900 7100 50  0001 C CNN
 F 3 "" H 900 7100 50  0001 C CNN
