File: pcb/sensactHsIO2/sensactHsIO2.kicad_pcb (KiCad board)
At the start: 2 copper layers, 86.5 x 71 mm, 142 parts, among them J1 SensactBus, J2 USB_C_Receptacle_USB2.0, J3 Conn_01x08, J4 Conn_01x08, J5 USB_C_Receptacle_USB2.0, J6 Conn_01x08, Q1 Q_NMOS_GSD, Q10 Q_NMOS_GSD, Q11 Q_NMOS_GSD, Q12 Q_NMOS_GSD, Q13 Q_NMOS_GSD, Q14 Q_NMOS_GSD, Q15 Q_NMOS_GSD, Q16 Q_NMOS_GSD, Q2 Q_NMOS_GSD, Q3 Q_NMOS_GSD, Q4 Q_NMOS_GSD, Q5 Q_NMOS_GSD, Q6 Q_NMOS_GSD, Q7 Q_NMOS_GSD, Q8 Q_NMOS_GSD, Q9 Q_NMOS_GSD, SW1 Reset, SW2 SW_Push, SW3 Mitsumi_SIQ-02FVS3, U1 STM32F072R8Tx, U2 SN65HVD230, U3 FP-096H09A, U4 SRV05-4, U5 SRV05-4, U6 SRV05-4, U7 SRV05-4

Commit message: updates in sensactHsIO2
Parts:
- added R16: 1k, Resistor_SMD:R_0805_2012Metric_Pad1.15x1.40mm_HandSolder, F.Cu at (132.7, 75.8)
- added R17: 1k, Resistor_SMD:R_0805_2012Metric_Pad1.15x1.40mm_HandSolder, F.Cu at (136.3, 74.8)
- added R18: 22R, Resistor_SMD:R_0805_2012Metric_Pad1.15x1.40mm_HandSolder, F.Cu at (90.7, 51.7)
- added U8: ESP-01v090, ESP8266:ESP-01, B.Cu at (113.7, 52.7)
- U1: value STM32F072R8Tx -> STM32F103R8Tx
- moved C12 15.3 mm to (96.4, 47.0), turned to 0 degrees
- moved R10 4.08 mm to (81.0, 39.2), turned to 0 degrees
- moved R11 2.69 mm to (84.7, 39.2)
Connections:
- J2 pad A5: /TX -> SWO
- J2 pad B5: /TX -> SWO
- J6 pad 1: (no net) -> DAC0
- J6 pad 2: (no net) -> DAC1
- U1 pad 20: (no net) -> DAC0
- U1 pad 21: (no net) -> DAC1
- U1 pad 42: /TX -> (no net)
Routing:
- net /TX: track 49.7 -> 0.00 mm, vias 4 -> 0
- net +3V3: track 295.2 -> 332.9 mm
- net SDA1: track 49.1 -> 67.5 mm, vias 2 -> 3
- net SCL1: track 50.1 -> 67.1 mm, vias 2 -> 3
- net SWO: track 0.00 -> 9.52 mm
- net Net-(R10-Pad2): track 7.70 -> 3.66 mm
- net I09: track 30.1 -> 33.7 mm
- net S: track 41.6 -> 38.9 mm
- net /INT2: track 46.8 -> 47.8 mm
- net LCD_MOSI: track 29.1 -> 30.0 mm
- net GND: track 46.6 -> 47.3 mm
