File: pcb/sensactHsNano/ethswitch.sch (KiCad schematic (older format))
At the start: 3 parts, among them J4 HR911105A, U2 KSZ8863RLL

Commit message: sensactHsNano & sensactHsIO3
Parts:
- added C26, C35, C38, C43: 22u, Capacitor_SMD:C_0805_2012Metric_Pad1.18x1.45mm_HandSolder, symbol Device:C
- added C27, C28, C29, C30, C31, C32, C33, C37, C39, C41, C44: u1, Capacitor_SMD:C_0805_2012Metric_Pad1.18x1.45mm_HandSolder, symbol Device:C
- added C34, C36, C45: 10u, Capacitor_SMD:C_0805_2012Metric_Pad1.18x1.45mm_HandSolder, symbol Device:C
- added C40, C42: 18p, Capacitor_SMD:C_0805_2012Metric_Pad1.18x1.45mm_HandSolder, symbol Device:C
- added D2: 1N4148W, Diode_SMD:D_SOD-123, symbol Diode:1N4148W
- added FB1, FB2: Ferrite_Bead, Inductor_SMD:L_0805_2012Metric_Pad1.15x1.40mm_HandSolder, symbol Device:Ferrite_Bead
- added R19, R20, R21, R22: 330R, Resistor_SMD:R_0805_2012Metric_Pad1.15x1.40mm_HandSolder, symbol Device:R
- added R23, R24, R25, R26, R27, R28, R29, R30: 49R9, Resistor_SMD:R_0805_2012Metric_Pad1.15x1.40mm_HandSolder, symbol Device:R
- added R31, R32, R34, R37: 1k, Resistor_SMD:R_0805_2012Metric_Pad1.15x1.40mm_HandSolder, symbol Device:R
- added R33, R35, R36, R40, R41, R42, R43: 22R, Resistor_SMD:R_0805_2012Metric_Pad1.15x1.40mm_HandSolder, symbol Device:R
- added R38, R39: 4k7, Resistor_SMD:R_0805_2012Metric_Pad1.15x1.40mm_HandSolder, symbol Device:R
- added R44: 10k, Resistor_SMD:R_0805_2012Metric_Pad1.15x1.40mm_HandSolder, symbol Device:R
- added Y1: Crystal_GND24, symbol Device:Crystal_GND24
Connections:
- net ETH_CRS_DV: now also R33.1; no longer U2.16 (SMTXEN3)
- net ETH_POWER: now also R34.1
- net ETH_REF_CLK: now also R42.1; no longer U2.23 (SMTXC3)
- net ETH_RXD0: now also R36.1; no longer U2.20 (SMTXD30)
- net ETH_RXD1: now also R35.1; no longer U2.19 (SMTXD31)
- net ETH_TXD0: now also R40.1; no longer U2.29 (SMRXD30)
- net ETH_TXD1: now also R41.1; no longer U2.28 (SMRXD31)
- net ETH_TX_EN: now also R43.1; no longer U2.25 (SMRXDV3)
- net GND: now also J4.20 (GND), J4.8 (GND), J4.SH (Shield), U2.10 (AGND), U2.21 (GND), U2.31 (GND), U2.41 (GND), C26.2, C27.2, C28.2, C29.2, C30.1, C31.1, C32.1, C33.1, C34.2, C35.2, C36.2, C37.2, C38.2, C39.2, C40.2, C41.2, C42.2, C43.2, C44.2, C45.2, R31.2, R32.2, R34.2, R37.2, Y1.2, Y1.4
- net P2LED1: now also R32.1
- net SCL1: now also R39.2
- net SDA1: now also R38.2
- net TX1P: now reaches U2.4 (TXP1)
- net TX1P: now also J4.13 (TXP), R29.2; no longer J4.1 (TXP)
- net at J4.12 (Y+): now also R20.2
- net TX2P: now reaches U2.12 (TXP2)
- net TX2P: now also J4.1 (TXP), R23.2; no longer J4.13 (TXP)
- net TX1N: now reaches J4.14 (TXN)
- net TX1N: now also U2.3 (TXM1), R30.2; no longer U2.11 (TXM2)
- net RX1P: now reaches J4.15 (RXP)
- net RX1P: now also U2.2 (RXP1), R27.2; no longer U2.9 (RXP2)
- net +3.3VA: now reaches J4.16 (TXC)
- net +3.3VA: now also J4.17 (RXC), J4.4 (TXC), J4.5 (RXC), U2.5 (VDDA_3.3), C34.1, C36.1, C43.1, C44.1, FB2.1
- net RX1N: now reaches J4.18 (RXN)
- net RX1N: now also U2.1 (RXM1), R28.2; no longer U2.8 (RXM2)
- net TX2N: now reaches J4.2 (TXN)
- net TX2N: now also U2.11 (TXM2), R24.2; no longer U2.3 (TXM1)
- net at J4.21 (G+): now also R21.2
- net at J4.24 (Y+): now also R22.2
- net RX2P: now reaches J4.3 (RXP)
- net RX2P: now also U2.9 (RXP2), R25.2; no longer U2.2 (RXP1)
- net RX2N: now reaches J4.6 (RXN)
- net RX2N: now also U2.8 (RXM2), R26.2; no longer U2.1 (RXM1)
- net at J4.9 (G+): now also R19.2
- net at U2.14 (X1): now also C40.1, Y1.1
- net at U2.15 (X2): now also C42.1, Y1.3
- net +3V3: now reaches U2.22 (VDDIO)
- net +3V3: now also U2.40 (VDDIO), C38.1, C39.1, C41.1, D2.1 (K), FB2.2, R19.1, R20.1, R21.1, R22.1, R38.1, R39.1, R44.1
- net at U2.26 (SMRXD33): now also R42.2
- net +1V8: now reaches U2.32 (VDDC_1.8)
- net +1V8: now also U2.42 (VDDCO), C26.1, C27.1, C28.1, C29.1, FB1.2
- net RSTN: now reaches U2.47 (~RSTN)
- net RSTN: now also C45.1, D2.2 (A), R44.2
- net at U2.48 (FXSD1): now also R31.1
- net +1V5: now reaches U2.7 (VDDA_1.8)
- net +1V5: now also C35.1, C37.1, FB1.1
- new net: R33.2, U2.16 (SMTXEN3)
- new net: R35.2, U2.19 (SMTXD31)
- new net: R36.2, U2.20 (SMTXD30)
- new net: R37.1, U2.23 (SMTXC3)
- new net: R43.2, U2.25 (SMRXDV3)
- new net: R41.2, U2.28 (SMRXD31)
- new net: R40.2, U2.29 (SMRXD30)
- new net: C30.2, R23.1, R24.1
- new net: C31.2, R25.1, R26.1
- new net: C32.2, R27.1, R28.1
- new net: C33.2, R29.1, R30.1
- no-connect marks 5 -> 10
Other:
- note added: "Center"
- note added: "STRAPPING CLOCK MODE 5"
- note added: "STRAPPING CLOCK OUT DISABLE On STARTUP\n"
- note added: "STRAPPING I2C Slave"
- moved on the sheet: R5, U2
