File: pcb/sensactHsNano/sensactHsNano.kicad_pcb (KiCad board)
At the start: 2 copper layers, 90 x 94.8 mm, 67 parts, among them J1 Conn_01x08, J2 SensactBusConnector, J3 Conn_01x04, J4 HR911105A, J6 LEFT, J7 RIGHT, J8 Conn_01x08, J9 Conn_01x08, Q1 BC847, Q2 BC847, SW1 TERM, SW2 SW_Push, SW3 SW_Push, SW4 SW_Push, SW5 SW_Push, U1 TAS5805M, U2 KSZ8863RLL, U3 ESP32-WROOM-32U, U4 DS2482, U5 SN65HVD230, U6 FP-096H09A

Commit message: Initial Layout Top board
Parts:
- added R17: 10k, Resistor_SMD:R_0805_2012Metric_Pad1.15x1.40mm_HandSolder, B.Cu at (160.5, 65.5)
- added R18: 10k, Resistor_SMD:R_0805_2012Metric_Pad1.15x1.40mm_HandSolder, B.Cu at (139.1, 62.5)
- Q1: value BC847 -> IRLML6344TRPBF; moved to B.Cu
- Q2: value BC847 -> IRLML5203
- R13, R14: moved to B.Cu
- moved C23 24.9 mm to (168.8, 64.6), turned to 180 degrees
- moved Q1 18.4 mm to (160.4, 69.2), turned to 270 degrees
- moved R14 14.8 mm to (143.1, 72.0)
- moved R13 11.1 mm to (160.5, 63.6)
- moved R10 8.46 mm to (165.0, 64.6)
- moved R9 5.06 mm to (143.1, 73.9), turned to 180 degrees
- moved C24 1.84 mm to (138.4, 72.4)
- moved C25 1.84 mm to (140.3, 72.4)
- moved R12 1.65 mm to (162.2, 61.6)
- moved R16 1.54 mm to (147.5, 61.6)
- moved Q2 1.52 mm to (142.7, 62.5)
- moved C21 1.40 mm to (131.3, 73.4)
- moved R15 0.28 mm to (137.2, 62.5)
- moved D1 0.23 mm to (160.4, 71.8)
- moved R8 0.06 mm to (136.5, 72.4)
Connections:
- Q2 pad 2: GND1 -> +3V3
Routing:
- net +3V3: track 86.7 -> 102.9 mm, vias 2 -> 4
- net HMI_SW: track 17.4 -> 32.9 mm
- net Net-(D1-Pad2): track 0.00 -> 11.1 mm, vias 0 -> 1
- net Net-(R10-Pad1): track 19.8 -> 26.7 mm, vias 2 -> 3
- net GND1: track 8.18 -> 3.23 mm
- net Net-(Q1-Pad1): track 0.00 -> 4.11 mm
- net Net-(D1-Pad1): track 0.00 -> 3.84 mm, vias 0 -> 1
- net HMI_RS_LCD: track 36.0 -> 33.3 mm
- net HMI_SDA_LCD: track 37.1 -> 35.0 mm
- net Net-(Q2-Pad1): track 2.39 -> 4.12 mm
- net HMI_SCL_LCD: track 38.1 -> 36.4 mm
- net Net-(R16-Pad1): track 11.5 -> 13.1 mm
- net HMI_RESET_SW: track 14.8 -> 16.2 mm
- net Net-(R11-Pad1): track 17.3 -> 16.0 mm

Commit message: sensactHsNano & sensactHsIO3
Parts:
- moved R11 0.08 mm to (168.8, 61.6)
Routing:
- net HMI_LED: track 0.00 -> 35.3 mm, vias 0 -> 2
- net Net-(R11-Pad1): track 16.0 -> 18.7 mm, vias 2 -> 1
- net Net-(R16-Pad1): track 13.1 -> 14.3 mm
- net Net-(R10-Pad1): track 26.7 -> 27.7 mm
- net HMI_RESET_SW: track 16.2 -> 15.4 mm
- net HMI_SDA_LCD: track 35.0 -> 35.6 mm
- net HMI_RS_LCD: track 33.3 -> 33.8 mm
- net HMI_SCL_LCD: track 36.4 -> 37.0 mm
- net GND1: vias 0 -> 30
- added copper zone on F.Cu, net GND1

Commit message: Various PCB Updates
Parts:
- removed D1: LED, LED_SMD:LED_PLCC_2835_Handsoldering
- removed J1: Conn_01x08, sensact:PhoenixContact_MC_0,5_8-G-2.5_1x08_P2.50mm_Horizontal
- removed J6: LEFT, Connector_PinSocket_1.27mm:PinSocket_2x04_P1.27mm_Vertical_SMD
- removed J7: RIGHT, Connector_PinSocket_1.27mm:PinSocket_2x04_P1.27mm_Vertical_SMD
- removed J8, J9: Conn_01x08, Connector_PinHeader_1.27mm:PinHeader_2x04_P1.27mm_Horizontal
- removed Q1: IRLML6344TRPBF, Package_TO_SOT_SMD:SOT-23_Handsoldering
- removed Q2: IRLML5203, Package_TO_SOT_SMD:SOT-23_Handsoldering
- removed SW2: SW_Push, sensact:SW_SPST_2x4x3,5
- removed SW3, SW4, SW5: SW_Push, Button_Switch_SMD:SW_SPST_SKQG_WithStem
- removed U6: FP-096H09A, smopla:FP-96H09A
- added C26: 2u2, Capacitor_SMD:C_0805_2012Metric_Pad1.18x1.45mm_HandSolder, F.Cu at (141.7, 69.2)
- added C27: u1, Capacitor_SMD:C_0805_2012Metric_Pad1.18x1.45mm_HandSolder, F.Cu at (146.5, 66.2)
- added C28: u1, Capacitor_SMD:C_0805_2012Metric_Pad1.18x1.45mm_HandSolder, F.Cu at (141.7, 72.2)
- added C29: 2u2, Capacitor_SMD:C_0805_2012Metric_Pad1.18x1.45mm_HandSolder, F.Cu at (146.5, 69.2)
- added C30: 10n, Capacitor_SMD:C_0805_2012Metric_Pad1.18x1.45mm_HandSolder, F.Cu at (151.3, 66.2)
- added C31: 10n, Capacitor_SMD:C_0805_2012Metric_Pad1.18x1.45mm_HandSolder, F.Cu at (146.5, 72.2)
- added C32: u1, Capacitor_SMD:C_0805_2012Metric_Pad1.18x1.45mm_HandSolder, F.Cu at (170.1, 66.2)
- added C33: 22u, Capacitor_SMD:C_1206_3216Metric_Pad1.33x1.80mm_HandSolder, F.Cu at (159.9, 66.4)
- added FB1: Ferrite_Bead_Small, Inductor_SMD:L_0805_2012Metric_Pad1.15x1.40mm_HandSolder, F.Cu at (313.4, 96.0)
- added J5: Conn_01x04, Connector_Phoenix_MC:PhoenixContact_MC_1,5_4-G-3.5_1x04_P3.50mm_Horizontal, B.Cu at (113.4, 141.5)
- added R19: 49R, Resistor_SMD:R_0805_2012Metric_Pad1.20x1.40mm_HandSolder, F.Cu at (274.8, 243.6)
- added R20: K33, Resistor_SMD:R_0805_2012Metric_Pad1.20x1.40mm_HandSolder, F.Cu at (270.0, 246.6)
- added R21: K33, Resistor_SMD:R_0805_2012Metric_Pad1.20x1.40mm_HandSolder, F.Cu at (270.0, 243.6)
- added U7: TPS5430DDA, Package_SO:TI_SO-PowerPAD-8_ThermalVias, F.Cu at (281.9, 137.2)
- added X1: XO32, Oscillator:Oscillator_SMD_EuroQuartz_XO32-4Pin_3.2x2.5mm_HandSoldering, F.Cu at (307.1, 103.6)
- C10, C21, C23, C4, C5, C6, C7: footprint Capacitor_SMD:C_0805_2012Metric_Pad1.15x1.40mm_HandSolder -> Capacitor_SMD:C_0805_2012Metric_Pad1.18x1.45mm_HandSolder; moved to F.Cu
- C11, C12, C13, C14, C19, C2, C20, C22: footprint Capacitor_SMD:C_0805_2012Metric_Pad1.15x1.40mm_HandSolder -> Capacitor_SMD:C_0805_2012Metric_Pad1.18x1.45mm_HandSolder
- C15, C16, C18: footprint Capacitor_SMD:C_0805_2012Metric_Pad1.15x1.40mm_HandSolder -> Capacitor_SMD:C_1206_3216Metric_Pad1.33x1.80mm_HandSolder; moved to F.Cu
- C17: footprint Capacitor_SMD:C_0805_2012Metric_Pad1.15x1.40mm_HandSolder -> Capacitor_SMD:C_1206_3216Metric_Pad1.33x1.80mm_HandSolder
- C24: value u1 -> 2u2; footprint Capacitor_SMD:C_0805_2012Metric_Pad1.15x1.40mm_HandSolder -> Capacitor_SMD:C_0805_2012Metric_Pad1.18x1.45mm_HandSolder; moved to F.Cu
- C25: value 2u2 -> u1; footprint Capacitor_SMD:C_0805_2012Metric_Pad1.15x1.40mm_HandSolder -> Capacitor_SMD:C_0805_2012Metric_Pad1.18x1.45mm_HandSolder; moved to F.Cu
- C3, C9: value 1u -> 22u; footprint Capacitor_SMD:C_0805_2012Metric_Pad1.15x1.40mm_HandSolder -> Capacitor_SMD:C_1210_3225Metric_Pad1.33x2.70mm_HandSolder; moved to F.Cu
- J3: footprint sensact:PhoenixContact_MC_0,5_4-G-2.5_1x04_P2.50mm_Horizontal -> Connector_Phoenix_MC:PhoenixContact_MC_1,5_4-G-3.5_1x04_P3.50mm_Horizontal
- J4: footprint smopla:RJ45_Hanrun_HR911105Ax2 -> liebler_CONN:HANRUN_HR911105A
- L1, L2: value 4u7 -> 10u/23mR; footprint smopla:L_0630 -> Inductor_SMD:L_Taiyo-Yuden_NR-10050_9.8x10.0mm_HandSoldering
- L3, L4: value 4u7 -> 10u; footprint smopla:L_0630 -> Inductor_SMD:L_Taiyo-Yuden_NR-10050_9.8x10.0mm_HandSoldering
- R1, R3, R4, R6: footprint Resistor_SMD:R_0805_2012Metric_Pad1.15x1.40mm_HandSolder -> Resistor_SMD:R_0805_2012Metric_Pad1.20x1.40mm_HandSolder
- R10: value 4k7 -> 33R; footprint Resistor_SMD:R_0805_2012Metric_Pad1.15x1.40mm_HandSolder -> Resistor_SMD:R_0805_2012Metric_Pad1.20x1.40mm_HandSolder; moved to F.Cu
- R11: value 2k2 -> 33R; footprint Resistor_SMD:R_0805_2012Metric_Pad1.15x1.40mm_HandSolder -> Resistor_SMD:R_0805_2012Metric_Pad1.20x1.40mm_HandSolder; moved to F.Cu
- R12, R13, R8: value 1k -> 33R; footprint Resistor_SMD:R_0805_2012Metric_Pad1.15x1.40mm_HandSolder -> Resistor_SMD:R_0805_2012Metric_Pad1.20x1.40mm_HandSolder; moved to F.Cu
- R14: value K22 -> 33R; footprint Resistor_SMD:R_0805_2012Metric_Pad1.15x1.40mm_HandSolder -> Resistor_SMD:R_0805_2012Metric_Pad1.20x1.40mm_HandSolder; moved to F.Cu
- R15: value 1k -> 49R; footprint Resistor_SMD:R_0805_2012Metric_Pad1.15x1.40mm_HandSolder -> Resistor_SMD:R_0805_2012Metric_Pad1.20x1.40mm_HandSolder; moved to F.Cu
- R16: value 100R -> 12K1; footprint Resistor_SMD:R_0805_2012Metric_Pad1.15x1.40mm_HandSolder -> Resistor_SMD:R_0805_2012Metric_Pad1.20x1.40mm_HandSolder; moved to F.Cu
- R17, R18: value 10k -> 49R; footprint Resistor_SMD:R_0805_2012Metric_Pad1.15x1.40mm_HandSolder -> Resistor_SMD:R_0805_2012Metric_Pad1.20x1.40mm_HandSolder; moved to F.Cu
- R2: footprint Resistor_SMD:R_0805_2012Metric_Pad1.15x1.40mm_HandSolder -> Resistor_SMD:R_0805_2012Metric_Pad1.20x1.40mm_HandSolder; moved to F.Cu
- R5: value 11K8 -> 1K5; footprint Resistor_SMD:R_0805_2012Metric_Pad1.15x1.40mm_HandSolder -> Resistor_SMD:R_0805_2012Metric_Pad1.20x1.40mm_HandSolder
- R7: footprint Resistor_SMD:R_1206_3216Metric_Pad1.42x1.75mm_HandSolder -> Resistor_SMD:R_1206_3216Metric_Pad1.30x1.75mm_HandSolder
- R9: value 22k -> 33R; footprint Resistor_SMD:R_0805_2012Metric_Pad1.15x1.40mm_HandSolder -> Resistor_SMD:R_0805_2012Metric_Pad1.20x1.40mm_HandSolder; moved to F.Cu
- U2: value KSZ8863RLL -> LAN8720A; footprint sensact:LQFP-48_7x7mm_P0.5mm_handsolder -> sensact:QFN-24-1EP_4x4mm_P0.5mm_EP2.6x2.6mm_handsolder; moved to F.Cu
- U3: footprint RF_Module:ESP32-WROOM-32U -> smopla:ESP32-WROOM-32_HANDSOLDER; moved to F.Cu
- U5: moved to B.Cu
- moved R15 231.8 mm to (270.0, 252.5), turned to 0 degrees
- moved R18 228.3 mm to (270.0, 249.5), turned to 0 degrees
- moved R16 224.9 mm to (279.5, 243.6), turned to 0 degrees
- moved R9 223.0 mm to (284.3, 246.6), turned to 0 degrees
- moved R14 221.0 mm to (274.8, 249.5)
- moved R12 219.2 mm to (284.3, 243.6)
- moved R11 218.3 mm to (274.8, 252.5)
- moved R13 218.2 mm to (279.5, 246.6)
- moved R10 217.5 mm to (279.5, 249.5)
- moved R17 214.1 mm to (274.8, 246.6)
- moved C10 207.1 mm to (295.7, 246.6), turned to 0 degrees
- moved R4 201.7 mm to (305.3, 243.6), turned to 0 degrees
- moved R5 199.8 mm to (279.5, 252.5), turned to 0 degrees
- moved C5 196.5 mm to (295.7, 243.6), turned to 0 degrees
- moved R2 193.6 mm to (300.5, 246.6), turned to 0 degrees
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Connections:
- net Net-(U2-Pad13) renamed ETH_MDC
- net Net-(U2-Pad15) renamed NRST
- net Net-(U2-Pad18) renamed ETH_TX1
- C21 pad 1: GND1 -> +3V3
- C21 pad 2: HMI_RESET_SW -> GND
- C23 pad 1: GND1 -> Net-(C23-Pad1)
- C23 pad 2: HMI_SW -> GND
- C24 pad 1: +3V3 -> Net-(C23-Pad1)
- C24 pad 2: GND1 -> GND
- C25 pad 2: GND1 -> GND
- J3 pad 1: Net-(J3-Pad1) -> GND
- J3 pad 2: Net-(J3-Pad2) -> +24V
- J3 pad 3: Net-(J3-Pad3) -> CANL
- J3 pad 4: Net-(J3-Pad4) -> CANH
- J4 pad 1: Net-(J4-Pad1) -> /Sheet60E30B79/TX_P
- J4 pad 10: /ethswitch/P1LED0 -> Net-(J4-Pad10)
- J4 pad 11: /ethswitch/P1LED1 -> Net-(J4-Pad11)
- J4 pad 12: Net-(J4-Pad12) -> +3V3
- J4 pad 15: Net-(J4-Pad15) -> GND
- J4 pad 16: Net-(J4-Pad16) -> GND
- J4 pad 2: Net-(J4-Pad2) -> /Sheet60E30B79/TX_N
- J4 pad 3: Net-(J4-Pad3) -> /Sheet60E30B79/RX_P
- J4 pad 4: Net-(J4-Pad4) -> /Sheet60E30B79/VDD2A
- J4 pad 5: Net-(J4-Pad5) -> /Sheet60E30B79/VDD2A
- J4 pad 6: Net-(J4-Pad6) -> /Sheet60E30B79/RX_N
- J4 pad 7: Net-(J4-Pad7) -> (no net)
- J4 pad 8: Net-(J4-Pad8) -> GND
- J4 pad 9: Net-(J4-Pad9) -> +3V3
- R10 pad 1: Net-(R10-Pad1) -> ETH_RX1
- R10 pad 2: HMI_SW -> Net-(R10-Pad2)
- R11 pad 1: Net-(R11-Pad1) -> ETH_RXER
- R11 pad 2: Net-(R10-Pad1) -> Net-(R11-Pad2)
- R12 pad 1: GND1 -> ETH_CRS
- R12 pad 2: Net-(R11-Pad1) -> Net-(R12-Pad2)
- R13 pad 1: Net-(Q1-Pad1) -> ETH_CLK
- R13 pad 2: HMI_LED -> Net-(R13-Pad2)
- R14 pad 1: +3V3 -> Net-(R14-Pad1)
- R14 pad 2: Net-(D1-Pad2) -> Net-(R14-Pad2)
- R15 pad 1: Net-(Q2-Pad1) -> /Sheet60E30B79/VDD2A
- R15 pad 2: HMI_BL_LCD -> /Sheet60E30B79/TX_P
- R16 pad 1: Net-(R16-Pad1) -> GND
- R16 pad 2: Net-(Q2-Pad3) -> Net-(R16-Pad2)
- R17 pad 1: Net-(Q1-Pad1) -> /Sheet60E30B79/VDD2A
- R17 pad 2: GND1 -> /Sheet60E30B79/TX_N
- R18 pad 1: Net-(Q2-Pad1) -> /Sheet60E30B79/VDD2A
- R18 pad 2: +3V3 -> /Sheet60E30B79/RX_P
- R5 pad 1: Net-(R5-Pad1) -> ETH_MDIO
- R5 pad 2: GND -> +3V3
- R8 pad 1: HMI_RESET_SW -> ETH_CLK
- R8 pad 2: +3V3 -> Net-(R14-Pad1)
- R9 pad 1: HMI_SW -> Net-(R9-Pad1)
- R9 pad 2: +3V3 -> ETH_RX0
- U2 pad 1: Net-(J4-Pad6) -> /Sheet60E30B79/VDD2A
- U2 pad 10: Net-(U2-Pad10) -> Net-(R11-Pad2)
- U2 pad 11: Net-(J4-Pad14) -> Net-(R12-Pad2)
- U2 pad 12: Net-(J4-Pad13) -> ETH_MDIO
- U2 pad 14: Net-(U2-Pad14) -> Net-(R13-Pad2)
- U2 pad 16: ETH_CRS_DV -> ETH_TXEN
- U2 pad 17: ETH_POWER -> ETH_TX0
- U2 pad 19: ETH_RXD1 -> /Sheet60E30B79/VDD2A
- U2 pad 2: Net-(J4-Pad3) -> /Sheet60E30B79/LED2
- U2 pad 20: ETH_RXD0 -> /Sheet60E30B79/TX_N
- U2 pad 21: Net-(U2-Pad21) -> /Sheet60E30B79/TX_P
- U2 pad 22: Net-(U2-Pad22) -> /Sheet60E30B79/RX_N
- U2 pad 23: ETH_REF_CLK -> /Sheet60E30B79/RX_P
- U2 pad 24: ETH_RX_ERR -> Net-(R16-Pad2)
- U2 pad 25: ETH_TX_EN -> GND
- U2 pad 3: Net-(J4-Pad2) -> /Sheet60E30B79/LED1
- U2 pad 4: Net-(J4-Pad1) -> Net-(U2-Pad4)
- U2 pad 5: Net-(U2-Pad5) -> Net-(R14-Pad2)
- U2 pad 6: Net-(R5-Pad1) -> Net-(C23-Pad1)
- U2 pad 7: Net-(U2-Pad7) -> Net-(R10-Pad2)
- U2 pad 8: Net-(J4-Pad18) -> Net-(R9-Pad1)
- U2 pad 9: Net-(J4-Pad15) -> +3V3
Routing:
- net SDA1: track 122.8 -> 0.00 mm, vias 2 -> 0
- net SCL1: track 111.0 -> 0.00 mm, vias 2 -> 0
- net +3V3: track 102.7 -> 0.00 mm, vias 4 -> 0
- net LRCLK: track 44.8 -> 0.00 mm, vias 2 -> 0
- net CAN_RX: track 42.0 -> 0.00 mm, vias 1 -> 0
- net SCLK: track 39.0 -> 0.00 mm
- net SDIN: track 38.4 -> 0.00 mm
- net HMI_SCL_LCD: track 37.0 -> 0.00 mm
- net CAN_TX: track 36.3 -> 0.00 mm, vias 1 -> 0
- net HMI_SDA_LCD: track 35.6 -> 0.00 mm
- net HMI_LED: track 35.3 -> 0.00 mm, vias 2 -> 0
- net HMI_RS_LCD: track 33.8 -> 0.00 mm
- net HMI_SW: track 33.3 -> 0.00 mm, vias 1 -> 0
- net ETH_REF_CLK: track 32.0 -> 0.00 mm
- net ETH_POWER: track 31.3 -> 0.00 mm, vias 2 -> 0
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- removed copper zone on B.Cu, net GND1
- removed copper zone on F.Cu, net GND1
Other:
- board size 90 x 94.8 mm -> 90 x 58.5 mm
- net class Default: clearance 0.2 -> 0.19
- net class HigherVoltage added: clearance 0.3, trace_width 0.2, via_dia 0.6, via_drill 0.3
- rule pad_to_mask_clearance: 0.05 -> 0
- rule trace_clearance: 0.2 -> 0.19
- rule trace_min: 0.2 -> 0
- board text added: "CH CL CL CH"
- board text added: "GN 24"
- board text added: "IN0-3 IO4-7"
- board text added: "IO8...15"
- board text added: "OUT3-0"
- board text added: "RED: POWER GREEN:INFO"

Commit message: Updated sensactHsNano
Parts:
- added C34: 10u, Capacitor_SMD:C_1210_3225Metric_Pad1.33x2.70mm_HandSolder, B.Cu at (121.8, 145.9)
- added C35: 10n, Capacitor_SMD:C_0805_2012Metric_Pad1.18x1.45mm_HandSolder, B.Cu at (131.8, 141.5)
- added C36: m1, Capacitor_SMD:C_1210_3225Metric_Pad1.33x2.70mm_HandSolder, B.Cu at (139.2, 132.7)
- added C37: m1, Capacitor_SMD:C_1210_3225Metric_Pad1.33x2.70mm_HandSolder, B.Cu at (139.2, 142.6)
- added C38: m1, Capacitor_SMD:C_1210_3225Metric_Pad1.33x2.70mm_HandSolder, B.Cu at (139.2, 139.3)
- added C39: m1, Capacitor_SMD:C_1210_3225Metric_Pad1.33x2.70mm_HandSolder, B.Cu at (139.2, 136.0)
- added C40: u1, Capacitor_SMD:C_0805_2012Metric_Pad1.18x1.45mm_HandSolder, F.Cu at (154.9, 107.1)
- added D1: Rpower_Ginfo, liebler_SEMICONDUCTORS:Dialight-5530123F-0, B.Cu at (131.6, 101.0)
- added D2: 2A, Diode_SMD:D_SMB_Handsoldering, B.Cu at (125.7, 144.7)
- added D3: NUP2105, Package_TO_SOT_SMD:SOT-23_Handsoldering, F.Cu at (191.6, 112.1)
- added J1: PROG, liebler_CONN:IDC_2x03_P1.27mm_Vertical, B.Cu at (139.4, 127.3)
- added J6: 1wire, Connector_JST:JST_XH_B4B-XH-AM_1x04_P2.50mm_Vertical, B.Cu at (115.4, 129.3)
- added L5: 22u, Inductor_SMD:L_Taiyo-Yuden_NR-80xx_HandSoldering, B.Cu at (132.3, 135.1)
- added R22: 10k, Resistor_SMD:R_0805_2012Metric_Pad1.20x1.40mm_HandSolder, B.Cu at (137.5, 146.2)
- added R23: 4k7, Resistor_SMD:R_0805_2012Metric_Pad1.20x1.40mm_HandSolder, B.Cu at (139.6, 146.2)
- added R24: 1k, Resistor_SMD:R_0805_2012Metric_Pad1.20x1.40mm_HandSolder, B.Cu at (141.6, 146.2)
- added R25: 10k, Resistor_SMD:R_0805_2012Metric_Pad1.20x1.40mm_HandSolder, F.Cu at (139.3, 125.1)
- added R26: k22, Resistor_SMD:R_0805_2012Metric_Pad1.20x1.40mm_HandSolder, F.Cu at (133.7, 105.7)
- added R27: k22, Resistor_SMD:R_0805_2012Metric_Pad1.20x1.40mm_HandSolder, F.Cu at (132.8, 108.6)
- added R28: 4k7, Resistor_SMD:R_0805_2012Metric_Pad1.20x1.40mm_HandSolder, F.Cu at (151.5, 131.8)
- added R29: 4k7, Resistor_SMD:R_0805_2012Metric_Pad1.20x1.40mm_HandSolder, F.Cu at (145.5, 131.8)
- added SW2: Prog, Button_Switch_THT:SW_Tactile_SPST_Angled_PTS645Vx58-2LFS, B.Cu at (168.0, 99.5)
- added SW3: Reset, sensact:SW_SPST_2x4x3,5, F.Cu at (180.0, 108.8)
- C1, C8: footprint Capacitor_SMD:CP_Elec_10x10.5 -> Capacitor_THT:CP_Radial_D10.0mm_P3.50mm
- C19, C20, C22, C23, C24, C25, C27, C28, C32, C33, C4, C6, C7, R1, R3, R4, U2, U4: moved to B.Cu
- C2: moved to F.Cu
- C3, C9: footprint Capacitor_SMD:C_1210_3225Metric_Pad1.33x2.70mm_HandSolder -> Capacitor_SMD:C_1206_3216Metric_Pad1.33x1.80mm_HandSolder; moved to B.Cu
- FB1: value Ferrite_Bead_Small -> Bead
- J2: value SensactBusConnector -> SensactBus
- J3: value Conn_01x04 -> CAN+24V
- J5: value Conn_01x04 -> Audio
- L1, L2: value 10u/23mR -> 10u; footprint Inductor_SMD:L_Taiyo-Yuden_NR-10050_9.8x10.0mm_HandSoldering -> liebler_PASSIVES:Inductor_CDRH104_handsolder
- L3, L4: footprint Inductor_SMD:L_Taiyo-Yuden_NR-10050_9.8x10.0mm_HandSoldering -> liebler_PASSIVES:Inductor_CDRH104_handsolder
- R11, R13: value 33R -> 1k
- R14, R8: value 33R -> k1
- U3: value ESP32-WROOM-32U -> ESP32; moved to B.Cu
- U7: footprint Package_SO:TI_SO-PowerPAD-8_ThermalVias -> sensact:SOIC-8_3.9x4.9mm_Pitch1.27mm_pad_handsolder; moved to B.Cu
- X1: value XO32 -> 50MHz
- moved R6 219.5 mm to (117.6, 136.8), turned to 180 degrees
- moved R1 210.7 mm to (121.2, 140.3), turned to 270 degrees
- moved R16 206.9 mm to (119.7, 112.2)
- moved R21 205.7 mm to (109.6, 114.9), turned to 180 degrees
- moved R19 203.5 mm to (117.2, 114.9)
- moved R5 202.2 mm to (132.3, 113.8), turned to 180 degrees
- moved R20 202.1 mm to (110.5, 122.6), turned to 90 degrees
- moved R17 201.7 mm to (117.2, 120.7)
- moved FB1 201.3 mm to (113.4, 118.8), turned to 180 degrees
- moved R18 201.1 mm to (117.2, 118.8)
- moved R15 200.5 mm to (117.2, 122.6)
- moved R9 199.3 mm to (132.3, 117.7)
- moved R10 198.9 mm to (132.3, 115.8), turned to 180 degrees
- moved R12 196.2 mm to (132.3, 119.6), turned to 180 degrees
- moved R14 193.9 mm to (129.5, 121.1), turned to 90 degrees
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Connections:
- net /Sheet60E30B79/LED1 renamed /eth/LED1
- net /Sheet60E30B79/LED2 renamed /eth/LED2
- net /Sheet60E30B79/RX_N renamed /eth/RX_N
- net /Sheet60E30B79/RX_P renamed /eth/RX_P
- net /Sheet60E30B79/TX_N renamed /eth/TX_N
- net /Sheet60E30B79/TX_P renamed /eth/TX_P
- net Net-(R10-Pad2) renamed /eth/RX1
- net Net-(R12-Pad2) renamed /eth/CRS
- net Net-(R9-Pad1) renamed /eth/RX0
- C27 pad 1: /Sheet60E30B79/VDD2A -> /eth/VDD2A
- C28 pad 1: /Sheet60E30B79/VDD2A -> /eth/VDD2A
- C29 pad 1: /Sheet60E30B79/VDD2A -> /eth/VDD2A
- C30 pad 1: /Sheet60E30B79/VDD2A -> /eth/VDD2A
- C31 pad 1: /Sheet60E30B79/VDD2A -> /eth/VDD2A
- FB1 pad 1: /Sheet60E30B79/VDD2A -> /eth/VDD2A
- J2 pad 1: Net-(J2-Pad1) -> +3V3
- J2 pad 10: Net-(J2-Pad10) -> GND
- J2 pad 2: Net-(J2-Pad2) -> SCL1
- J2 pad 3: Net-(J2-Pad3) -> SDA1
- J2 pad 4: Net-(J2-Pad4) -> INT0
- J2 pad 5: Net-(J2-Pad5) -> INT1
- J2 pad 7: Net-(J2-Pad7) -> +24V
- J2 pad 8: Net-(J2-Pad8) -> +24V
- J2 pad 9: Net-(J2-Pad9) -> GND
- J4 pad 10: Net-(J4-Pad10) -> GND
- J4 pad 12: +3V3 -> /eth/VDD2A
- J4 pad 4: /Sheet60E30B79/VDD2A -> /eth/VDD2A
- J4 pad 5: /Sheet60E30B79/VDD2A -> /eth/VDD2A
- J4 pad 9: +3V3 -> Net-(J4-Pad9)
- R11 pad 1: ETH_RXER -> +3V3
- R11 pad 2: Net-(R11-Pad2) -> EN
- R13 pad 1: ETH_CLK -> +3V3
- R15 pad 1: /Sheet60E30B79/VDD2A -> /eth/VDD2A
- R17 pad 1: /Sheet60E30B79/VDD2A -> /eth/VDD2A
- R18 pad 1: /Sheet60E30B79/VDD2A -> /eth/VDD2A
- R19 pad 1: /Sheet60E30B79/VDD2A -> /eth/VDD2A
- R2 pad 2: /audioamplifier/PDN -> AMP_PDN
- R20 pad 1: Net-(J4-Pad10) -> Net-(J4-Pad9)
- U1 pad 10: SDA1 -> SDA2
- U1 pad 11: SCL1 -> SCL2
- U1 pad 12: /audioamplifier/PDN -> AMP_PDN
- U2 pad 1: /Sheet60E30B79/VDD2A -> /eth/VDD2A
- U2 pad 10: Net-(R11-Pad2) -> Net-(U2-Pad10)
- U2 pad 14: Net-(R13-Pad2) -> Net-(U2-Pad14)
- U2 pad 15: NRST -> EN
- U2 pad 19: /Sheet60E30B79/VDD2A -> /eth/VDD2A
- U3 pad 10: ETH_RXD0 -> ETH_RX0
- U3 pad 11: ETH_RXD1 -> ETH_RX1
- U3 pad 12: ETH_CRS_DV -> ETH_CRS
- U3 pad 24: Net-(U3-Pad24) -> SDA2
- U3 pad 25: ETH_REF_CLK -> ETH_CLK
- U3 pad 29: Net-(U3-Pad29) -> SCL2
- U3 pad 3: Net-(U3-Pad3) -> EN
- U3 pad 30: Net-(U3-Pad30) -> ETH_MDIO
- U3 pad 31: ETH_TXD0 -> ETH_TX0
- U3 pad 33: ETH_TX_EN -> ETH_TXEN
- U3 pad 34: Net-(U3-Pad34) -> PROG_RX
- U3 pad 35: Net-(U3-Pad35) -> PROG_TX
- U3 pad 36: ETH_TXD1 -> ETH_TX1
- U3 pad 37: Net-(U3-Pad37) -> ETH_MDC
- U3 pad 4: Net-(U3-Pad4) -> Net-(R13-Pad2)
- U3 pad 5: Net-(U3-Pad5) -> INT0
- U3 pad 6: Net-(U3-Pad6) -> INT1
- U3 pad 9: Net-(U3-Pad9) -> AMP_PDN
- U4 pad 4: SCL1 -> SCL2
- U4 pad 5: SDA1 -> SDA2
- U7 pad 4: Net-(U7-Pad4) -> /psu/VSENSE
- U7 pad 5: Net-(U7-Pad5) -> +24V
- U7 pad 6: Net-(U7-Pad6) -> GND
- U7 pad 7: Net-(U7-Pad7) -> +24V
- U7 pad 8: Net-(U7-Pad8) -> /psu/SW
- U7 pad 9: Net-(U7-Pad9) -> GND
- X1 pad 1: Net-(X1-Pad1) -> ETH_POWER
Routing:
- net +3V3: track 0.00 -> 226.3 mm, vias 0 -> 10
- net +24V: track 0.00 -> 152.7 mm, vias 0 -> 1
- net EN: track 0.00 -> 94.5 mm, vias 0 -> 5
- net INT0: track 0.00 -> 67.0 mm, vias 0 -> 2
- net INT1: track 0.00 -> 64.4 mm, vias 0 -> 2
- net /eth/VDD2A: track 0.00 -> 40.0 mm, vias 0 -> 2
- net CANH: track 0.00 -> 39.2 mm
- net SCL1: track 0.00 -> 37.7 mm
- net GND: track 0.00 -> 37.6 mm, vias 0 -> 29
- net OneWire: track 0.00 -> 34.5 mm, vias 0 -> 1
- net SCL2: track 0.00 -> 33.6 mm, vias 0 -> 3
- net SDA1: track 0.00 -> 32.3 mm
- net /eth/LED1: track 0.00 -> 31.1 mm, vias 0 -> 1
- net CANL: track 0.00 -> 30.4 mm
- net ETH_TX1: track 0.00 -> 26.0 mm, vias 0 -> 2
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- added copper zone on B.Cu, net /psu/SW
- added copper zone on B.Cu, net GND
- added copper zone on F.Cu, net GND
Other:
- net class HigherVoltage: clearance 0.3 -> 0.25
- rule via_min_size: 0.4 -> 0.6
- board text removed: "CH CL CL CH"
- board text removed: "GN 24"
- board text removed: "IN0-3 IO4-7"
- board text removed: "IO8...15"
- board text removed: "OUT3-0"

Commit message: Complete reorganisation
Parts:
- added C41: 10u, Capacitor_SMD:C_1206_3216Metric_Pad1.33x1.80mm_HandSolder, F.Cu at (188.6, 124.8)
- added C42: 10u, Capacitor_SMD:C_1206_3216Metric_Pad1.33x1.80mm_HandSolder, F.Cu at (192.3, 130.9)
- added C43: u1, Capacitor_SMD:C_0805_2012Metric_Pad1.18x1.45mm_HandSolder, F.Cu at (192.3, 128.7)
- added D10: 1N4007, liebler_SEMICONDUCTORS:D_SOD-123_handsolder, F.Cu at (191.1, 141.3)
- added D11: 1N4007, liebler_SEMICONDUCTORS:D_SOD-123_handsolder, F.Cu at (191.8, 139.0)
- added D4: 2A, Diode_SMD:D_SMB_Handsoldering, F.Cu at (180.3, 113.6)
- added D5: ebus-RX, Diode_SMD:D_0805_2012Metric_Pad1.15x1.40mm_HandSolder, F.Cu at (145.4, 135.6)
- added D6: ebus-TX, Diode_SMD:D_0805_2012Metric_Pad1.15x1.40mm_HandSolder, F.Cu at (143.2, 146.4)
- added D7: 9,1V/1,3W, Diode_THT:D_DO-41_SOD81_P10.16mm_Horizontal, B.Cu at (192.8, 151.1)
- added D8: 1N4007, liebler_SEMICONDUCTORS:D_SOD-123_handsolder, F.Cu at (191.8, 136.7)
- added D9: 1N4007, liebler_SEMICONDUCTORS:D_SOD-123_handsolder, F.Cu at (191.1, 134.3)
- added Q1: BC817, Package_TO_SOT_SMD:SOT-23_Handsoldering, F.Cu at (171.5, 146.4)
- added R30: k22, Resistor_SMD:R_0805_2012Metric_Pad1.20x1.40mm_HandSolder, F.Cu at (147.4, 136.3)
- added R31: k22, Resistor_SMD:R_0805_2012Metric_Pad1.20x1.40mm_HandSolder, F.Cu at (151.3, 135.6)
- added R32: 1k, Resistor_SMD:R_0805_2012Metric_Pad1.20x1.40mm_HandSolder, F.Cu at (149.3, 135.6)
- added R33: k47, Resistor_SMD:R_0805_2012Metric_Pad1.20x1.40mm_HandSolder, F.Cu at (147.4, 146.4)
- added R34: k47, Resistor_SMD:R_0805_2012Metric_Pad1.20x1.40mm_HandSolder, F.Cu at (144.4, 143.5)
- added R35: 10k, Resistor_SMD:R_0805_2012Metric_Pad1.20x1.40mm_HandSolder, B.Cu at (153.6, 146.1)
- added R36: m22, Resistor_SMD:R_0805_2012Metric_Pad1.20x1.40mm_HandSolder, F.Cu at (162.0, 146.3)
- added R37: 18k, Resistor_SMD:R_0805_2012Metric_Pad1.20x1.40mm_HandSolder, F.Cu at (145.4, 146.4)
- added R38: 15k, Resistor_SMD:R_0805_2012Metric_Pad1.20x1.40mm_HandSolder, F.Cu at (163.9, 146.3)
- added R39: m1, Resistor_SMD:R_0805_2012Metric_Pad1.20x1.40mm_HandSolder, F.Cu at (176.1, 146.5)
- added R40: 22k, Resistor_SMD:R_0805_2012Metric_Pad1.20x1.40mm_HandSolder, F.Cu at (165.9, 146.3)
- added R41: k22, Resistor_SMD:R_0805_2012Metric_Pad1.20x1.40mm_HandSolder, F.Cu at (167.8, 146.3)
- added R42: 10k, Resistor_SMD:R_0805_2012Metric_Pad1.20x1.40mm_HandSolder, F.Cu at (126.2, 128.0)
- added U10: HT75xx-1-SOT89, Package_TO_SOT_SMD:SOT-89-3_Handsoldering, F.Cu at (192.3, 124.1)
- added U6: EL817, liebler_SEMICONDUCTORS:SO-4_7.6x3.6mm_P2.54mm_handsolder, B.Cu at (146.0, 141.2)
- added U8: EL817, liebler_SEMICONDUCTORS:SO-4_7.6x3.6mm_P2.54mm_handsolder, B.Cu at (150.5, 141.2)
- added U9: LM393, sensact:SOIC-8_3.9x4.9mm_Pitch1.27mm_handsolder, F.Cu at (152.6, 145.5)
- L5: footprint Inductor_SMD:L_Taiyo-Yuden_NR-80xx_HandSoldering -> liebler_PASSIVES:Inductor_CDRH104_handsolder
- R1: moved to F.Cu
- moved C16 8.64 mm to (182.9, 132.4), turned to 0 degrees
- moved C17 8.64 mm to (182.9, 139.4), turned to 0 degrees
- moved C15 8.64 mm to (182.9, 136.0), turned to 0 degrees
- moved C18 8.64 mm to (182.9, 128.9), turned to 0 degrees
- moved L5 3.52 mm to (128.8, 135.4), turned to 180 degrees
- moved SW1 3.43 mm to (192.7, 116.0)
- moved C36 3.28 mm to (136.0, 132.0)
- moved C38 3.28 mm to (136.0, 138.6)
- moved C39 3.28 mm to (136.0, 135.3)
- moved R1 2.57 mm to (120.8, 137.8)
- moved D3 2.47 mm to (191.8, 109.7), turned to 180 degrees
- moved C20 2.10 mm to (142.7, 133.9), turned to 90 degrees
- moved R7 1.83 mm to (185.0, 124.2), turned to 90 degrees
- moved C19 0.90 mm to (142.7, 137.7), turned to 270 degrees
- moved C37 0.79 mm to (139.1, 141.8)
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Connections:
- net /audioamplifier/OUT_A+ renamed OUT_A+
- net /audioamplifier/OUT_A- renamed OUT_A-
- net /audioamplifier/OUT_B+ renamed OUT_B+
- net /audioamplifier/OUT_B- renamed OUT_B-
- net LRCLK renamed EB_TX
- net SDIN renamed EB_RX
- D3 pad 1: CANH -> CANL
- D3 pad 2: CANL -> CANH
- J3 pad 2: +24V -> Net-(D4-Pad2)
Routing:
- net GND1: track 0.00 -> 86.9 mm
- net +5VA: track 0.00 -> 82.3 mm, vias 0 -> 2
- net Net-(C41-Pad1): track 0.00 -> 51.4 mm
- net GND: track 37.6 -> 61.3 mm, vias 29 -> 25
- net Net-(R36-Pad1): track 0.00 -> 22.0 mm
- net Net-(R39-Pad2): track 0.00 -> 21.9 mm
- net Net-(Q1-Pad1): track 0.00 -> 19.5 mm, vias 0 -> 1
- net /psu/SW: track 19.1 -> 0.00 mm, vias 2 -> 0
- net EB_RX: track 19.0 -> 35.7 mm, vias 0 -> 3
- net Net-(R35-Pad2): track 0.00 -> 13.9 mm, vias 0 -> 1
- net OUT_B+: track 14.4 -> 27.8 mm
- net Net-(D7-Pad2): track 0.00 -> 11.8 mm, vias 0 -> 1
- net OUT_A+: track 12.5 -> 21.4 mm
- net Net-(R7-Pad1): track 5.85 -> 13.7 mm, vias 0 -> 2
- net +3V3: track 226.3 -> 234.0 mm
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Other:
- board text added: "B+ B- ebus/A- ebus/A+"
- board text added: "GN 3V OW GN"
- board text added: "SCL 3V3 IN1 SDA NC IN2 24V 24V GND GND"
- board text added: "TERM ON TERM OFF"

Commit message: sensactUP2, sensactHsNano sensactHsLED sensactOutdoor as ordered at JLCPCB
Parts:
- added JP1: INT0, Jumper:SolderJumper-2_P1.3mm_Open_RoundedPad1.0x1.5mm, F.Cu at (153.8, 110.9)
- added JP2: SUP_MON, Jumper:SolderJumper-2_P1.3mm_Open_RoundedPad1.0x1.5mm, B.Cu at (179.1, 111.6)
- added NT1: Net-Tie_2, NetTie:NetTie-2_SMD_Pad2.0mm, B.Cu at (164.3, 115.4)
- added R43: 1k, Resistor_SMD:R_0805_2012Metric_Pad1.20x1.40mm_HandSolder, F.Cu at (157.4, 113.0)
- added R44: 10k, Resistor_SMD:R_0805_2012Metric_Pad1.20x1.40mm_HandSolder, B.Cu at (182.6, 112.6)
- added R45: 1k, Resistor_SMD:R_0805_2012Metric_Pad1.20x1.40mm_HandSolder, B.Cu at (182.6, 110.6)
- added R46: 1k, Resistor_SMD:R_0805_2012Metric_Pad1.20x1.40mm_HandSolder, F.Cu at (157.4, 111.1)
- R15, R17, R18, R19: value 49R -> 49R9
- R3: moved to F.Cu
- SW1: footprint Button_Switch_SMD:SW_SPDT_PCM12 -> liebler_MECH:SW_SPDT_PCM12_handsolder
- moved D3 20.1 mm to (172.1, 113.4), turned to 0 degrees
- moved R11 4.45 mm to (157.4, 107.3), turned to 180 degrees
- moved R3 3.42 mm to (167.5, 114.4), turned to 90 degrees
- moved R13 2.26 mm to (157.4, 109.2), turned to 180 degrees
- moved C40 2.03 mm to (153.5, 108.6), turned to 180 degrees
- moved C10 1.45 mm to (166.8, 128.8), turned to 0 degrees
- moved C5 1.44 mm to (166.8, 136.7), turned to 0 degrees
- moved R2 1.14 mm to (157.4, 114.9)
- moved C43 0.89 mm to (192.3, 129.6)
- moved U10 0.89 mm to (192.3, 125.0)
- moved C42 0.89 mm to (192.3, 131.7)
- moved C41 0.51 mm to (188.6, 125.3)
Connections:
- C1 pad 2: GND -> GNDA
- C10 pad 2: GND -> GNDA
- C15 pad 1: GND -> GNDA
- C16 pad 1: GND -> GNDA
- C17 pad 1: GND -> GNDA
- C18 pad 1: GND -> GNDA
- C3 pad 2: GND -> GNDA
- C5 pad 2: GND -> GNDA
- C8 pad 2: GND -> GNDA
- C9 pad 2: GND -> GNDA
- U1 pad 14: GND -> GNDA
- U1 pad 19: GND -> GNDA
- U1 pad 24: GND -> GNDA
- U1 pad 29: GND -> GNDA
- U3 pad 5: INT0 -> SENSOR_VN
Routing:
- net GNDA: track 0.00 -> 77.0 mm, vias 0 -> 20
- net SENSOR_VN: track 0.00 -> 26.3 mm, vias 0 -> 3
- net +24V: track 157.1 -> 139.7 mm
- net SUPPLY_MONITOR: track 0.00 -> 3.94 mm
- net Net-(D4-Pad2): track 4.13 -> 7.95 mm
- net +3V3: track 234.0 -> 230.6 mm, vias 10 -> 9
- net Net-(R13-Pad2): track 17.2 -> 14.6 mm
- net Net-(R3-Pad1): track 2.38 -> 0.00 mm, vias 0 -> 1
- net AMP_PDN: track 19.3 -> 20.6 mm
- net Net-(R26-Pad2): track 22.6 -> 24.0 mm
- net EN: track 94.8 -> 96.1 mm
- net GND1: track 86.9 -> 85.6 mm
- net INT1: track 67.2 -> 68.4 mm, vias 2 -> 3
- net CANH: track 42.9 -> 44.1 mm, vias 1 -> 2
- net Net-(C41-Pad1): track 51.4 -> 52.5 mm
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- added copper zone on B.Cu, net GNDA
- added copper zone on F.Cu, net GNDA
