File: pcb/sensactHsIO4/io4.sch (KiCad schematic (older format))
At the start: 25 parts, among them Q1 IRLML6344, Q2 IRLML6344, Q5 IRLML6344, Q6 IRLML6344, U4 SRV05

Commit message: Improvements in pcb design of sensactOutdoor and sensactHsIO4
Changed lines of the file:
@@
 AR Path="/60587002/5E28AF71" Ref="Q2"  Part="1"
 AR Path="/60587D6B/5E28AF71" Ref="Q6"  Part="1"
-F 0 "Q6" H 2755 3396 50  0000 L CNN
+F 0 "Q10" H 2755 3396 50  0000 L CNN
 F 1 "IRLML6344" H 2755 3305 50  0000 L CNN
 F 2 "Package_TO_SOT_SMD:SOT-23_Handsoldering" H 2750 3450 50  0001 C CNN
@@
 AR Path="/60587002/5E28E1B5" Ref="R32"  Part="1"
 AR Path="/60587D6B/5E28E1B5" Ref="R48"  Part="1"
-F 0 "R48" V 2800 3350 50  0000 C CNN
+F 0 "R64" V 2800 3350 50  0000 C CNN
 F 1 "1k" V 2900 3350 50  0000 C CNN
 F 2 "Resistor_SMD:R_0805_2012Metric_Pad1.20x1.40mm_HandSolder" V 2830 3350 50  0001 C CNN
@@
 AR Path="/60587002/5E28E848" Ref="R28"  Part="1"
 AR Path="/60587D6B/5E28E848" Ref="R44"  Part="1"
-F 0 "R44" V 2650 3550 50  0000 R CNN
+F 0 "R60" V 2650 3550 50  0000 R CNN
 F 1 "10k" V 2750 3500 50  0000 C CNN
 F 2 "Resistor_SMD:R_0805_2012Metric_Pad1.20x1.40mm_HandSolder" V 2680 3500 50  0001 C CNN
@@
 AR Path="/60587002/5E28F71C" Ref="C15"  Part="1"
 AR Path="/60587D6B/5E28F71C" Ref="C19"  Part="1"
-F 0 "C19" H 3165 3546 50  0000 L CNN
+F 0 "C23" H 3165 3546 50  0000 L CNN
 F 1 "u1" H 3165 3455 50  0000 L CNN
 F 2 "Capacitor_SMD:C_0805_2012Metric_Pad1.18x1.45mm_HandSolder" H 3088 3350 50  0001 C CNN
@@
 AR Path="/60587002/5E292C13" Ref="R24"  Part="1"
 AR Path="/60587D6B/5E292C13" Ref="R40"  Part="1"
-F 0 "R40" V 2500 3100 50  0000 R CNN
+F 0 "R56" V 2500 3100 50  0000 R CNN
 F 1 "10R" V 2600 3050 50  0000 C CNN
 F 2 "Resistor_SMD:R_0805_2012Metric_Pad1.20x1.40mm_HandSolder" V 2530 3050 50  0001 C CNN
@@
 AR Path="/60587002/5E294612" Ref="R36"  Part="1"
 AR Path="/60587D6B/5E294612" Ref="R52"  Part="1"
-F 0 "R52" V 2950 3200 50  0000 C CNN
+F 0 "R68" V 2950 3200 50  0000 C CNN
 F 1 "10k" V 3050 3200 50  0000 C CNN
 F 2 "Resistor_SMD:R_0805_2012Metric_Pad1.20x1.40mm_HandSolder" V 2980 3200 50  0001 C CNN
@@
 AR Path="/60587002/5E29E0A6" Ref="Q1"  Part="1"
 AR Path="/60587D6B/5E29E0A6" Ref="Q5"  Part="1"
-F 0 "Q5" H 2755 2196 50  0000 L CNN
+F 0 "Q9" H 2755 2196 50  0000 L CNN
 F 1 "IRLML6344" H 2755 2105 50  0000 L CNN
 F 2 "Package_TO_SOT_SMD:SOT-23_Handsoldering" H 2750 2250 50  0001 C CNN
@@
 AR Path="/60587002/5E29E0C5" Ref="R27"  Part="1"
 AR Path="/60587D6B/5E29E0C5" Ref="R43"  Part="1"
-F 0 "R43" V 2650 2350 50  0000 R CNN
+F 0 "R59" V 2650 2350 50  0000 R CNN
 F 1 "10k" V 2750 2300 50  0000 C CNN
 F 2 "Resistor_SMD:R_0805_2012Metric_Pad1.20x1.40mm_HandSolder" V 2680 2300 50  0001 C CNN
@@
 AR Path="/60587002/605F93F4" Ref="C14"  Part="1"
 AR Path="/60587D6B/605F93F4" Ref="C18"  Part="1"
-F 0 "C18" H 3165 2346 50  0000 L CNN
+F 0 "C22" H 3165 2346 50  0000 L CNN
 F 1 "u1" H 3165 2255 50  0000 L CNN
 F 2 "Capacitor_SMD:C_0805_2012Metric_Pad1.18x1.45mm_HandSolder" H 3088 2150 50  0001 C CNN
@@
 AR Path="/60587002/605F93F6" Ref="R35"  Part="1"
 AR Path="/60587D6B/605F93F6" Ref="R51"  Part="1"
-F 0 "R51" V 2950 2000 50  0000 C CNN
+F 0 "R67" V 2950 2000 50  0000 C CNN
 F 1 "10k" V 3050 2000 50  0000 C CNN
 F 2 "Resistor_SMD:R_0805_2012Metric_Pad1.20x1.40mm_HandSolder" V 2980 2000 50  0001 C CNN
@@
 AR Path="/60587002/5FF3463A" Ref="R23"  Part="1"
 AR Path="/60587D6B/5FF3463A" Ref="R39"  Part="1"
-F 0 "R39" V 2500 1850 50  0000 C CNN
+F 0 "R55" V 2500 1850 50  0000 C CNN
 F 1 "10R" V 2600 1850 50  0000 C CNN
 F 2 "Resistor_SMD:R_0805_2012Metric_Pad1.20x1.40mm_HandSolder" V 2530 1850 50  0001 C CNN
@@
 AR Path="/60587002/5FF48F46" Ref="Q3"  Part="1"
 AR Path="/60587D6B/5FF48F46" Ref="Q7"  Part="1"
-F 0 "Q7" H 2755 4896 50  0000 L CNN
+F 0 "Q11" H 2755 4896 50  0000 L CNN
 F 1 "IRLML6344" H 2755 4805 50  0000 L CNN
 F 2 "Package_TO_SOT_SMD:SOT-23_Handsoldering" H 2750 4950 50  0001 C CNN
@@
 AR Path="/60587002/5FF49149" Ref="R33"  Part="1"
 AR Path="/60587D6B/5FF49149" Ref="R49"  Part="1"
-F 0 "R49" V 2800 4850 50  0000 C CNN
+F 0 "R65" V 2800 4850 50  0000 C CNN
 F 1 "1k" V 2900 4850 50  0000 C CNN
 F 2 "Resistor_SMD:R_0805_2012Metric_Pad1.20x1.40mm_HandSolder" V 2830 4850 50  0001 C CNN
@@
 AR Path="/60587002/5FF49153" Ref="R29"  Part="1"
 AR Path="/60587D6B/5FF49153" Ref="R45"  Part="1"
-F 0 "R45" V 2650 5050 50  0000 R CNN
+F 0 "R61" V 2650 5050 50  0000 R CNN
 F 1 "10k" V 2750 5000 50  0000 C CNN
 F 2 "Resistor_SMD:R_0805_2012Metric_Pad1.20x1.40mm_HandSolder" V 2680 5000 50  0001 C CNN
@@
 AR Path="/60587002/605F93FA" Ref="C16"  Part="1"
 AR Path="/60587D6B/605F93FA" Ref="C20"  Part="1"
-F 0 "C20" H 3165 5046 50  0000 L CNN
+F 0 "C24" H 3165 5046 50  0000 L CNN
 F 1 "u1" H 3165 4955 50  0000 L CNN
 F 2 "Capacitor_SMD:C_0805_2012Metric_Pad1.18x1.45mm_HandSolder" H 3088 4850 50  0001 C CNN
@@
 AR Path="/60587002/5FF4916B" Ref="R25"  Part="1"
 AR Path="/60587D6B/5FF4916B" Ref="R41"  Part="1"
-F 0 "R41" V 2500 4600 50  0000 R CNN
+F 0 "R57" V 2500 4600 50  0000 R CNN
 F 1 "10R" V 2600 4550 50  0000 C CNN
 F 2 "Resistor_SMD:R_0805_2012Metric_Pad1.20x1.40mm_HandSolder" V 2530 4550 50  0001 C CNN
@@
 AR Path="/60587002/5FF4917F" Ref="R37"  Part="1"
 AR Path="/60587D6B/5FF4917F" Ref="R53"  Part="1"
-F 0 "R53" V 2950 4700 50  0000 C CNN
+F 0 "R69" V 2950 4700 50  0000 C CNN
 F 1 "10k" V 3050 4700 50  0000 C CNN
 F 2 "Resistor_SMD:R_0805_2012Metric_Pad1.20x1.40mm_HandSolder" V 2980 4700 50  0001 C CNN
@@
 AR Path="/60587002/5FF4D6A5" Ref="R38"  Part="1"
 AR Path="/60587D6B/5FF4D6A5" Ref="R54"  Part="1"
-F 0 "R54" V 2950 5850 50  0000 C CNN
+F 0 "R70" V 2950 5850 50  0000 C CNN
 F 1 "10k" V 3050 5850 50  0000 C CNN
 F 2 "Resistor_SMD:R_0805_2012Metric_Pad1.20x1.40mm_HandSolder" V 2980 5850 50  0001 C CNN
@@
 AR Path="/60587002/5FF4D691" Ref="R26"  Part="1"
 AR Path="/60587D6B/5FF4D691" Ref="R42"  Part="1"
-F 0 "R42" V 2500 5750 50  0000 R CNN
+F 0 "R58" V 2500 5750 50  0000 R CNN
 F 1 "10R" V 2600 5700 50  0000 C CNN
 F 2 "Resistor_SMD:R_0805_2012Metric_Pad1.20x1.40mm_HandSolder" V 2530 5700 50  0001 C CNN
@@
 AR Path="/60587002/605F93FF" Ref="C17"  Part="1"
 AR Path="/60587D6B/605F93FF" Ref="C21"  Part="1"
-F 0 "C21" H 3165 6196 50  0000 L CNN
+F 0 "C25" H 3165 6196 50  0000 L CNN
 F 1 "u1" H 3165 6105 50  0000 L CNN
 F 2 "Capacitor_SMD:C_0805_2012Metric_Pad1.18x1.45mm_HandSolder" H 3088 6000 50  0001 C CNN
@@
 AR Path="/60587002/5FF4D679" Ref="R30"  Part="1"
 AR Path="/60587D6B/5FF4D679" Ref="R46"  Part="1"
-F 0 "R46" V 2650 6200 50  0000 R CNN
+F 0 "R62" V 2650 6200 50  0000 R CNN
 F 1 "10k" V 2750 6150 50  0000 C CNN
 F 2 "Resistor_SMD:R_0805_2012Metric_Pad1.20x1.40mm_HandSolder" V 2680 6150 50  0001 C CNN
@@
 AR Path="/60587002/605F93FE" Ref="R34"  Part="1"
 AR Path="/60587D6B/605F93FE" Ref="R50"  Part="1"
-F 0 "R50" V 2800 6000 50  0000 C CNN
+F 0 "R66" V 2800 6000 50  0000 C CNN
 F 1 "1k" V 2900 6000 50  0000 C CNN
 F 2 "Resistor_SMD:R_0805_2012Metric_Pad1.20x1.40mm_HandSolder" V 2830 6000 50  0001 C CNN
@@
 AR Path="/60587002/5FF4D65A" Ref="Q4"  Part="1"
 AR Path="/60587D6B/5FF4D65A" Ref="Q8"  Part="1"
-F 0 "Q8" H 2755 6046 50  0000 L CNN
+F 0 "Q12" H 2755 6046 50  0000 L CNN
 F 1 "IRLML6344" H 2755 5955 50  0000 L CNN
 F 2 "Package_TO_SOT_SMD:SOT-23_Handsoldering" H 2750 6100 50  0001 C CNN
@@
 AR Path="/60587002/5E29E0BB" Ref="R31"  Part="1"
 AR Path="/60587D6B/5E29E0BB" Ref="R47"  Part="1"
-F 0 "R47" V 2800 2150 50  0000 C CNN
+F 0 "R63" V 2800 2150 50  0000 C CNN
 F 1 "1k" V 2900 2150 50  0000 C CNN
 F 2 "Resistor_SMD:R_0805_2012Metric_Pad1.20x1.40mm_HandSolder" V 2830 2150 50  0001 C CNN
@@
 AR Path="/60587002/5E2887A7" Ref="U10"  Part="1"
 AR Path="/60587D6B/5E2887A7" Ref="U11"  Part="1"
-F 0 "U11" V 4400 3850 50  0000 C CNN
+F 0 "U12" V 4400 3850 50  0000 C CNN
 F 1 "SRV05" V 4300 3850 50  0000 C CNN
 F 2 "Package_TO_SOT_SMD:SOT-23-6_Handsoldering" H 5250 2800 50  0001 C CNN
