File: pcb/sensactHsIO4/sensactHsIO4.kicad_pcb (KiCad board)
At the start: 2 copper layers, 90 x 74.6 mm, 183 parts, among them J1 BUS, J2 Bus, J3 24V, J4 PROG, J5 IN0-3 IO4-7, J6 IO8-15, J7 HMI, J8 Conn_01x10, J9 AOUT, Q1 AO3400A, Q2 AO3400A, SW2 TERM ON, SW3 Reset, SW4 R, SW5 L, SW6 OK, U1 ESP32-WROOM-32, U10 EUP3458, U11 LM317_TO-252, U12 SP3485EN, U13 SRV05-4, U14 SRV05-4, U15 SRV05-4, U16 SRV05-4, U2 SN65HVD230, U3 ULN2003, U4 ULN2003, U5 LM358, U6 SRV05-4, U7 SRV05-4, U8 SRV05-4, U9 SRV05-4, X1 LH114

Commit message: Various changes (does not compile)
Parts:
- removed J4: PROG, liebler_CONN:IDC_2x03_P1.27mm_Vertical
- added C28: 4u7, Capacitor_SMD:C_0603_1608Metric, B.Cu at (183.5, 119.3)
- added C29: 1u, Capacitor_SMD:C_0603_1608Metric, B.Cu at (185.2, 119.3)
- added C30: 4u7, Capacitor_SMD:C_0805_2012Metric_Pad1.18x1.45mm_HandSolder, F.Cu at (187.6, 130.3)
- added C31: 1u, Capacitor_SMD:C_0805_2012Metric_Pad1.18x1.45mm_HandSolder, F.Cu at (189.6, 130.3)
- added C32: u1, Capacitor_SMD:C_0402_1005Metric, B.Cu at (173.8, 114.9)
- added C33: u1, Capacitor_SMD:C_0402_1005Metric, B.Cu at (170.0, 120.1)
- added J10: PROG, liebler_CONN:USB-C-HANBO-MC-307_C961709, B.Cu at (179.8, 109.5)
- added Q3: BC817, Package_TO_SOT_SMD:SOT-23, B.Cu at (178.2, 125.0)
- added Q4: BC817, Package_TO_SOT_SMD:SOT-23, B.Cu at (171.4, 125.0)
- added R80: 5k1, Resistor_SMD:R_0603_1608Metric, B.Cu at (172.2, 112.3)
- added R81: 5k1, Resistor_SMD:R_0603_1608Metric, B.Cu at (181.8, 117.4)
- added R82: 10k, Resistor_SMD:R_0603_1608Metric, B.Cu at (174.8, 125.6)
- added R83: 10k, Resistor_SMD:R_0603_1608Metric, B.Cu at (174.8, 124.1)
- added SW1: USB 3V INT, liebler_MECH:SW_SPDT_PCM12_handsolder, F.Cu at (179.8, 109.9)
- added U17: AMS1117, liebler_SEMICONDUCTORS:SOT-223-3_TabPin2_HANDSOLDER, F.Cu at (188.8, 123.4)
- added U18: CH340C, Package_SO:SOIC-16_3.9x9.9mm_P1.27mm, B.Cu at (175.8, 119.6)
- J2: footprint Connector_IDC:IDC-Header_2x05_P2.54mm_Horizontal -> liebler_CONN:IDC-Header_2x05_P2.54mm_Horizontal_tightCrtYd
- JP13: value OUT_IN0 -> IO01
- JP14: value OUT_IN0 -> IO03
- JP15: value OUT_IN0 -> IO05
- JP16: value OUT_IN0 -> IO07
- JP20: value OUT_IN0 -> IO08
- JP21: value OUT_IN0 -> IO10
- JP22: value OUT_IN0 -> IO12
- JP26: value OUT_IN0 -> IO09
- JP27: value OUT_IN0 -> IO11
- JP28: value OUT_IN0 -> IO13
- JP31: value IO12 -> 485 IO12 BUZZER
- JP32: value BUST -> BUSTX
- JP33: value BUSR -> BUSRX
- JP34: value BUST -> BUS1
- JP35: value BUSR -> BUS2
- JP5: value OUT_IN0 -> IO00
- JP6: value OUT_IN0 -> IO02
- JP7: value OUT_IN0 -> IO04
- JP8: value OUT_IN0 -> IO06
- R3: footprint Resistor_SMD:R_0603_1608Metric -> Resistor_SMD:R_0402_1005Metric_Pad0.72x0.64mm_HandSolder
- R7: footprint Resistor_SMD:R_0402_1005Metric -> Resistor_SMD:R_0603_1608Metric
- SW2: value TERM ON -> OFF TERM ON
- moved J3 20.7 mm to (187.3, 110.5)
- moved C24 16.5 mm to (165.3, 128.9)
- moved C21 16.3 mm to (179.8, 132.1)
- moved R54 16.3 mm to (179.4, 127.5)
- moved R55 16.3 mm to (179.4, 129.0)
- moved L1 15.8 mm to (170.8, 130.3)
- moved U10 15.8 mm to (176.9, 131.8)
- moved C23 15.8 mm to (175.9, 128.2)
- moved C22 15.8 mm to (177.8, 135.4)
- moved D4 14.1 mm to (173.6, 135.7), turned to 180 degrees
- moved C25 11.4 mm to (156.3, 147.6), turned to 0 degrees
- moved J2 8.91 mm to (182.0, 132.1)
- moved C26 7.48 mm to (158.4, 147.6), turned to 180 degrees
- moved R65 5.83 mm to (163.3, 145.7), turned to 90 degrees
- moved JP32 5.57 mm to (170.3, 145.0), turned to 90 degrees
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Connections:
- C24 pad 1: +3V3 -> +3.3VA
- L1 pad 1: +3V3 -> +3.3VA
- R54 pad 1: +3V3 -> +3.3VA
Routing:
- net +3.3VA: track 0.00 -> 79.9 mm, vias 0 -> 3
- net Net-(C30-Pad2): track 0.00 -> 35.4 mm
- net +5P: track 0.00 -> 32.7 mm, vias 0 -> 1
- net PROG_EN: track 38.3 -> 23.6 mm, vias 1 -> 2
- net +15V: track 15.1 -> 29.1 mm
- net /UD+: track 0.00 -> 13.3 mm
- net PROG_RX: track 21.2 -> 34.1 mm, vias 0 -> 2
- net BACKLIGHT: track 36.9 -> 47.5 mm, vias 2 -> 4
- net 485_RO: track 16.5 -> 7.06 mm
- net BUS_RX: track 21.9 -> 31.2 mm
- net PROG_TX: track 23.1 -> 31.7 mm, vias 0 -> 2
- net Net-(J10-PadA5): track 0.00 -> 7.92 mm
- net GND: track 34.0 -> 26.1 mm, vias 30 -> 40
- net /UD-: track 0.00 -> 7.02 mm
- net BUS_TX: track 40.3 -> 45.8 mm
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Other:
- board text added: "0-10V GND 15V 24V"
- board text added: "CANL/B CANH/A CANH/A CANL/B"
- board text added: "DIREKT : Li:12, Re:offen INPUT : Li:23, Re:23 OUTPUT: Li:offen, Re:12"
- board text added: "GND 24V"
- board text added: "OBEN CAN UNTEN RS485"
