File: pcb/sensactHsIO4/sensactHsIO4.kicad_sch (KiCad schematic)
At the start: 154 parts, among them J1 BUS, J2 Bus, J3 24V, J4 PROG, J5 IN0-3 IO4-7, J6 IO8-15, J7 HMI, J9 AOUT, SW2 TERM ON, U1 ESP32-WROOM-32, U11 LM317_TO-252, U12 SP3485EN, U13 SRV05-4, U14 SRV05-4, U15 SRV05-4, U16 SRV05-4, U2 SN65HVD230, U3 ULN2003, U4 ULN2003, U5 LM358, U6 SRV05-4, U7 SRV05-4, U8 SRV05-4, U9 SRV05-4

Commit message: Various changes (does not compile)
Parts:
- removed J4: PROG, liebler_CONN:IDC_2x03_P1.27mm_Vertical, symbol Connector_Generic:Conn_02x03_Odd_Even
- removed SW2: TERM ON, liebler_MECH:SW_SPDT_PCM12_handsolder, symbol Switch:SW_SPDT
- added C28: 4u7, Capacitor_SMD:C_0603_1608Metric, symbol Device:C
- added C29: 1u, Capacitor_SMD:C_0603_1608Metric, symbol Device:C
- added C30: 4u7, Capacitor_SMD:C_0805_2012Metric_Pad1.18x1.45mm_HandSolder, symbol Device:C
- added C31: 1u, Capacitor_SMD:C_0805_2012Metric_Pad1.18x1.45mm_HandSolder, symbol Device:C
- added C32, C33: u1, Capacitor_SMD:C_0402_1005Metric, symbol Device:C
- added J10: PROG, liebler_CONN:USB-C-HANBO-MC-307_C961709, symbol Connector:USB_C_Receptacle_USB2.0
- added Q3, Q4: BC817, Package_TO_SOT_SMD:SOT-23, symbol Transistor_BJT:BC817
- added R80, R81: 5k1, Resistor_SMD:R_0603_1608Metric, symbol Device:R
- added R82, R83: 10k, Resistor_SMD:R_0603_1608Metric, symbol Device:R
- added SW1: USB 3V INT, liebler_MECH:SW_SPDT_PCM12_handsolder, symbol liebler_MECH:SW_SPDT_with_Case
- added SW2: OFF TERM ON, liebler_MECH:SW_SPDT_PCM12_handsolder, symbol liebler_MECH:SW_SPDT_with_Case
- added U17: AMS1117, liebler_SEMICONDUCTORS:SOT-223-3_TabPin2_HANDSOLDER, symbol Regulator_Linear:AMS1117-3.3
- added U18: CH340C, Package_SO:SOIC-16_3.9x9.9mm_P1.27mm, symbol Interface_USB:CH340C
- J2: footprint Connector_IDC:IDC-Header_2x05_P2.54mm_Horizontal -> liebler_CONN:IDC-Header_2x05_P2.54mm_Horizontal_tightCrtYd
- JP13: value OUT_IN0 -> IO01
- JP14: value OUT_IN0 -> IO03
- JP15: value OUT_IN0 -> IO05
- JP16: value OUT_IN0 -> IO07
- JP20: value OUT_IN0 -> IO08
- JP21: value OUT_IN0 -> IO10
- JP22: value OUT_IN0 -> IO12
- JP26: value OUT_IN0 -> IO09
- JP27: value OUT_IN0 -> IO11
- JP28: value OUT_IN0 -> IO13
- JP31: value IO12 -> 485 IO12 BUZZER
- JP32: value BUST -> BUSTX
- JP33: value BUSR -> BUSRX
- JP34: value BUST -> BUS1
- JP35: value BUSR -> BUS2
- JP5: value OUT_IN0 -> IO00
- JP6: value OUT_IN0 -> IO02
- JP7: value OUT_IN0 -> IO04
- JP8: value OUT_IN0 -> IO06
- R3: footprint Resistor_SMD:R_0603_1608Metric -> Resistor_SMD:R_0402_1005Metric_Pad0.72x0.64mm_HandSolder
- R7: footprint Resistor_SMD:R_0402_1005Metric -> Resistor_SMD:R_0603_1608Metric
Connections:
- net +3V3: now also SW1.2 (B)
- net BACKLIGHT: now also Q3.3 (C)
- net BUS_1: now also SW2.2 (B)
- net GND: now also C28.1, C29.2, C30.1, C31.2, C32.2, C33.2, J10.A1 (GND), J10.A12 (GND), J10.B1 (GND), J10.B12 (GND), J10.S1 (SHIELD), R80.1, R81.1, SW1.CASE, SW2.CASE, U17.1 (GND), U18.1 (GND)
- net PROG_EN: now also Q4.3 (C)
- net PROG_RX: now also U18.3 (RXD)
- net PROG_TX: now also U18.2 (TXD)
- net at R9.2: now also SW2.3 (C)
- new net: Q4.1 (B), R83.1
- new net: C30.2, C31.1, SW1.3 (C), U17.2 (VO)
- new net: Q3.1 (B), R82.1
- new net: C32.1, U18.4 (V3)
- new net: J10.B5 (CC2), R81.2
- new net: J10.A5 (CC1), R80.2
- new net +3.3VA: SW1.1 (A)
- new net +5P: C28.2, C29.1, C33.1, J10.A4 (VBUS), J10.A9 (VBUS), J10.B4 (VBUS), J10.B9 (VBUS), U17.3 (VI), U18.16 (VCC)
- new net DTR: Q3.2 (E), R83.2, U18.13 (~{DTR})
- new net RTS: Q4.2 (E), R82.2, U18.14 (~{RTS})
- new net UD+: J10.A6 (D+), J10.B6 (D+), U18.5 (UD+)
- new net UD-: J10.A7 (D-), J10.B7 (D-), U18.6 (UD-)
- no-connect marks 14 -> 21
Other:
- note added: "5V->3V3"
