File: pcb/sensactHsNano2/eth.kicad_sch (KiCad schematic)
At the start: 30 parts, among them J4 HR911105A, U2 LAN8720A, X1 50MHz

Commit message: DIn-schiene-seitenwand + sensactHsNano2
Parts:
- removed JP3: ETH_RST, Jumper:SolderJumper-2_P1.3mm_Open_RoundedPad1.0x1.5mm, symbol Device:Jumper_NO_Small
- removed R42: 10k, Resistor_SMD:R_0805_2012Metric_Pad1.20x1.40mm_HandSolder, symbol Device:R
- C21: footprint Capacitor_SMD:C_0603_1608Metric -> Capacitor_SMD:C_0805_2012Metric_Pad1.18x1.45mm_HandSolder
- C23, C24, C25, C26, C27, C28: footprint Capacitor_SMD:C_0603_1608Metric -> Capacitor_SMD:C_0402_1005Metric
- C29, C45: footprint Capacitor_SMD:C_0805_2012Metric_Pad1.18x1.45mm_HandSolder -> Capacitor_SMD:C_0402_1005Metric
- R10, R12, R14, R9: footprint Resistor_SMD:R_0805_2012Metric_Pad1.20x1.40mm_HandSolder -> Resistor_SMD:R_0402_1005Metric
- R16, R5, R8: footprint Resistor_SMD:R_0603_1608Metric -> Resistor_SMD:R_0402_1005Metric
- R47: value 1k -> 4k7; footprint Resistor_SMD:R_0805_2012Metric_Pad1.20x1.40mm_HandSolder -> Resistor_SMD:R_0402_1005Metric
- X1: footprint Oscillator:Oscillator_SMD_EuroQuartz_XO32-4Pin_3.2x2.5mm -> Oscillator:Oscillator_SMD_EuroQuartz_XO32-4Pin_3.2x2.5mm_HandSoldering
Connections:
- net RBIAS: now reaches R16.2, U2.24 (RBIAS)
- net VDDCR: now reaches C23.1, C24.1, U2.6 (VDDCR)
- net RST: now reaches C45.1, R47.2, U2.15 (RST)

Commit message: Various
Parts:
- added NT2: NetTie_2, NetTie:NetTie-2_SMD_Pad0.5mm, symbol Device:NetTie_2
- C21: footprint Capacitor_SMD:C_0805_2012Metric_Pad1.18x1.45mm_HandSolder -> Capacitor_SMD:C_0402_1005Metric
- X1: footprint Oscillator:Oscillator_SMD_EuroQuartz_XO32-4Pin_3.2x2.5mm_HandSoldering -> Oscillator:Oscillator_SMD_SeikoEpson_SG8002CE-4Pin_3.2x2.5mm
Connections:
- net GND: now also NT2.2; no longer C21.2, X1.2 (GND)
- new net CLK_GND: C21.2, NT2.1, X1.2 (GND)
Other:
- moved on the sheet: C21
Changed lines of the file:
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@@
   (junction (at 149.86 50.8) (diameter 0) (color 0 0 0 0)
+  )
+  (junction (at 77.47 123.19) (diameter 0) (color 0 0 0 0)
   )
   (junction (at 105.41 66.04) (diameter 0) (color 0 0 0 0)
@@
   (no_connect (at 116.84 115.57))
   (no_connect (at 116.84 107.95))
-  (wire (pts (xy 69.85 115.57) (xy 67.31 115.57))
-    (stroke (width 0) (type default) (color 0 0 0 0))
-  )
   (wire (pts (xy 132.08 64.77) (xy 132.08 43.18))
     (stroke (width 0) (type default) (color 0 0 0 0))
@@
     (stroke (width 0) (type default) (color 0 0 0 0))
   )
+  (wire (pts (xy 63.5 111.76) (xy 63.5 107.95))
+    (stroke (width 0) (type default) (color 0 0 0 0))
+  )
   (wire (pts (xy 166.37 85.09) (xy 166.37 78.74))
     (stroke (width 0) (type default) (color 0 0 0 0))
@@
     (stroke (width 0) (type default) (color 0 0 0 0))
   )
-  (wire (pts (xy 67.31 115.57) (xy 67.31 121.92))
-    (stroke (width 0) (type default) (color 0 0 0 0))
-  )
   (wire (pts (xy 199.39 82.55) (xy 199.39 95.25))
     (stroke (width 0) (type default) (color 0 0 0 0))
@@
     (stroke (width 0) (type default) (color 0 0 0 0))
   )
-  (wire (pts (xy 59.69 121.92) (xy 59.69 115.57))
-    (stroke (width 0) (type default) (color 0 0 0 0))
-  )
   (wire (pts (xy 181.61 64.77) (xy 181.61 71.12))
     (stroke (width 0) (type default) (color 0 0 0 0))
@@
     (stroke (width 0) (type default) (color 0 0 0 0))
   )
+  (wire (pts (xy 82.55 123.19) (xy 85.09 123.19))
+    (stroke (width 0) (type default) (color 0 0 0 0))
+  )
+  (wire (pts (xy 55.88 115.57) (xy 69.85 115.57))
+    (stroke (width 0) (type default) (color 0 0 0 0))
+  )
   (wire (pts (xy 154.94 90.17) (xy 181.61 90.17))
     (stroke (width 0) (type default) (color 0 0 0 0))
@@
     (stroke (width 0) (type default) (color 0 0 0 0))
   )
+  (wire (pts (xy 63.5 123.19) (xy 77.47 123.19))
+    (stroke (width 0) (type default) (color 0 0 0 0))
+  )
   (wire (pts (xy 181.61 43.18) (xy 181.61 64.77))
     (stroke (width 0) (type default) (color 0 0 0 0))
@@
     (stroke (width 0) (type default) (color 0 0 0 0))
   )
-  (wire (pts (xy 67.31 121.92) (xy 59.69 121.92))
-    (stroke (width 0) (type default) (color 0 0 0 0))
-  )
   (wire (pts (xy 81.28 91.44) (xy 72.39 91.44))
     (stroke (width 0) (type default) (color 0 0 0 0))
@@
     (stroke (width 0) (type default) (color 0 0 0 0))
   )
+  (wire (pts (xy 63.5 107.95) (xy 77.47 107.95))
+    (stroke (width 0) (type default) (color 0 0 0 0))
+  )
   (wire (pts (xy 142.24 50.8) (xy 149.86 50.8))
     (stroke (width 0) (type default) (color 0 0 0 0))
@@
     (stroke (width 0) (type default) (color 0 0 0 0))
   )
-  (wire (pts (xy 55.88 115.57) (xy 59.69 115.57))
-    (stroke (width 0) (type default) (color 0 0 0 0))
-  )
   (polyline (pts (xy 104.14 97.79) (xy 104.14 83.82))
     (stroke (width 0) (type default) (color 0 0 0 0))
@@
     (stroke (width 0) (type default) (color 0 0 0 0))
   )
+  (wire (pts (xy 63.5 119.38) (xy 63.5 123.19))
+    (stroke (width 0) (type default) (color 0 0 0 0))
+  )
   (wire (pts (xy 116.84 113.03) (xy 104.14 113.03))
     (stroke (width 0) (type default) (color 0 0 0 0))
@@
     (stroke (width 0) (type default) (color 0 0 0 0))
   )
-  (wire (pts (xy 77.47 107.95) (xy 63.5 107.95))
-    (stroke (width 0) (type default) (color 0 0 0 0))
-  )
-  (text "50MHz" (at 74.93 123.19 180)
+  (text "50MHz" (at 78.74 120.015 180)
     (effects (font (size 1.27 1.27)) (justify right bottom))
   )
@@
   (label "RX_P" (at 157.48 87.63 0)
     (effects (font (size 1.27 1.27)) (justify left bottom))
+  )
+  (label "CLK_GND" (at 77.47 123.19 180)
+    (effects (font (size 1.27 1.27)) (justify right bottom))
   )
   (label "LED2" (at 209.55 118.11 180)
@@
       (effects (font (size 1.27 1.27)) (justify left))
     )
-    (property "Footprint" "Oscillator:Oscillator_SMD_EuroQuartz_XO32-4Pin_3.2x2.5mm_HandSoldering" (id 2) (at 95.25 124.46 0)
+    (property "Footprint" "Oscillator:Oscillator_SMD_SeikoEpson_SG8002CE-4Pin_3.2x2.5mm" (id 2) (at 95.25 124.46 0)
       (effects (font (size 1.27 1.27)) hide)
     )
@@
     (pin "2")
   )
-  (symbol (lib_id "power:GND") (at 77.47 123.19 0) (unit 1)
-    (in_bom yes) (on_board yes)
-    (property "Reference" "#PWR015" (id 0) (at 77.47 129.54 0)
-      (effects (font (size 1.27 1.27)) hide)
-    )
-    (property "Value" "GND" (id 1) (at 77.597 127.5842 0))
-    (property "Footprint" "" (id 2) (at 77.47 123.19 0)
-      (effects (font (size 1.27 1.27)) hide)
-    )
-    (property "Datasheet" "" (id 3) (at 77.47 123.19 0)
-      (effects (font (size 1.27 1.27)) hide)
-    )
-    (pin "1")
-  )
   (symbol (lib_id "power:GND") (at 137.16 123.19 90) (unit 1)
     (in_bom yes) (on_board yes)
@@
     (pin "1")
   )
-  (symbol (lib_id "Device:C") (at 63.5 111.76 0) (unit 1)
-    (in_bom yes) (on_board yes)
-    (property "Reference" "C21" (id 0) (at 66.421 110.5916 0)
-      (effects (font (size 1.27 1.27)) (justify left))
-    )
-    (property "Value" "u1" (id 1) (at 66.421 112.903 0)
-      (effects (font (size 1.27 1.27)) (justify left))
-    )
-    (property "Footprint" "Capacitor_SMD:C_0805_2012Metric_Pad1.18x1.45mm_HandSolder" (id 2) (at 64.4652 115.57 0)
-      (effects (font (size 1.27 1.27)) hide)
-    )
-    (property "Datasheet" "~" (id 3) (at 63.5 111.76 0)
-      (effects (font (size 1.27 1.27)) hide)
-    )
-    (pin "1")
-    (pin "2")
-  )
-  (symbol (lib_id "power:GND") (at 63.5 115.57 0) (unit 1)
-    (in_bom yes) (on_board yes)
-    (property "Reference" "#PWR013" (id 0) (at 63.5 121.92 0)
-      (effects (font (size 1.27 1.27)) hide)
-    )
-    (property "Value" "GND" (id 1) (at 63.627 119.9642 0))
-    (property "Footprint" "" (id 2) (at 63.5 115.57 0)
-      (effects (font (size 1.27 1.27)) hide)
-    )
-    (property "Datasheet" "" (id 3) (at 63.5 115.57 0)
-      (effects (font (size 1.27 1.27)) hide)
-    )
-    (pin "1")
-  )
-  (symbol (lib_id "power:GND") (at 236.22 113.03 0) (unit 1)
-    (in_bom yes) (on_board yes)
-    (property "Reference" "#PWR026" (id 0) (at 236.22 119.38 0)
-      (effects (font (size 1.27 1.27)) hide)
-    )
-    (property "Value" "GND" (id 1) (at 236.347 116.2812 90)
-      (effects (font (size 1.27 1.27)) (justify right))
-    )
-    (property "Footprint" "" (id 2) (at 236.22 113.03 0)
-      (effects (font (size 1.27 1.27)) hide)
-    )
-    (property "Datasheet" "" (id 3) (at 236.22 113.03 0)
-      (effects (font (size 1.27 1.27)) hide)
-    )
-    (pin "1")
+  (symbol (lib_id "Device:C") (at 63.5 115.57 0) (unit 1)
+    (in_bom yes) (on_board yes)
+    (property "Reference" "C21" (id 0) (at 66.421 114.4016 0)
+      (effects (font (size 1.27 1.27)) (justify left))
+    )
+    (property "Value" "u1" (id 1) (at 66.421 116.713 0)
+      (effects (font (size 1.27 1.27)) (justify left))
+    )
+    (property "Footprint" "Capacitor_SMD:C_0402_1005Metric" (id 2) (at 64.4652 119.38 0)
+      (effects (font (size 1.27 1.27)) hide)
+    )
+    (property "Datasheet" "~" (id 3) (at 63.5 115.57 0)
+      (effects (font (size 1.27 1.27)) hide)
+    )
+    (pin "1")
+    (pin "2")
   )
   (symbol (lib_id "liebler_CONN:HR911105A") (at 255.27 102.87 0) (unit 1)
@@
       (effects (font (size 1.27 1.27)) hide)
     )
+    (pin "1")
+  )
+  (symbol (lib_id "Device:NetTie_2") (at 80.01 123.19 0) (unit 1)
+    (in_bom yes) (on_board yes)
+    (property "Reference" "NT2" (id 0) (at 80.01 126.365 0))
+    (property "Value" "NetTie_2" (id 1) (at 80.01 124.46 0))
+    (property "Footprint" "NetTie:NetTie-2_SMD_Pad0.5mm" (id 2) (at 80.01 123.19 0)
+      (effects (font (size 1.27 1.27)) hide)
+    )
+    (property "Datasheet" "~" (id 3) (at 80.01 123.19 0)
+      (effects (font (size 1.27 1.27)) hide)
+    )
+    (pin "1")
+    (pin "2")
+  )
+  (symbol (lib_id "power:GND") (at 85.09 123.19 0) (unit 1)
+    (in_bom yes) (on_board yes)
+    (property "Reference" "#PWR0152" (id 0) (at 85.09 129.54 0)
+      (effects (font (size 1.27 1.27)) hide)
+    )
+    (property "Value" "GND" (id 1) (at 85.217 127.5842 0))
+    (property "Footprint" "" (id 2) (at 85.09 123.19 0)
+      (effects (font (size 1.27 1.27)) hide)
+    )
+    (property "Datasheet" "" (id 3) (at 85.09 123.19 0)
+      (effects (font (size 1.27 1.27)) hide)
+    )
