File: pcb/sensactHsNano2/sensactHsNano2.kicad_pcb (KiCad board)
At the start: 2 copper layers, 90 x 54.8 mm, 122 parts, among them J1 HMI, J2 SensactBusConnector, J3 CAN+485, J4 HR911105A, J5 Audio, J6 Conn_01x03, J7 PROG, J8 Conn_01x10, J9 24V, Q1 BC817, Q2 BC817, SW1 TERM ON, SW2 OFF TERM ON, SW3 Reset, SW4 PROG_PWR, U1 TAS5805M, U11 L78L15_SOT89, U13 CH340C, U2 LAN8720A, U3 ESP32, U4 DS2482, U5 SN65HVD230, U6 MAX3485, U7 RY8310, U8 LM358, U9 MCP4728, X1 50MHz

Commit message: Improved sensactNano2
Parts:
- added J10: I2S_EXT, Connector_PinHeader_1.27mm:PinHeader_1x08_P1.27mm_Vertical, B.Cu at (156.3, 123.5)
- added JP1: RS485_BUZZER, Jumper:SolderJumper-2_P1.3mm_Open_RoundedPad1.0x1.5mm, F.Cu at (141.2, 132.9)
- added JP2: RS485_BACKLIGHT, Jumper:SolderJumper-2_P1.3mm_Open_RoundedPad1.0x1.5mm, F.Cu at (138.3, 115.7)
- C3, C9: footprint Capacitor_SMD:C_1206_3216Metric -> Capacitor_SMD:C_1210_3225Metric_Pad1.33x2.70mm_HandSolder
- J8: moved to B.Cu
- L1, L2, L3, L4: footprint liebler_PASSIVES:ASPIAIG-Q8080 -> liebler_PASSIVES:L_1040
- R1, R6: footprint Resistor_SMD:R_0603_1608Metric -> Resistor_SMD:R_0402_1005Metric
- R23: footprint Resistor_SMD:R_0805_2012Metric_Pad1.20x1.40mm_HandSolder -> Resistor_SMD:R_1206_3216Metric_Pad1.30x1.75mm_HandSolder
- R7: value 120R -> K12
- moved C44 33.1 mm to (167.6, 145.2)
- moved U11 33.1 mm to (163.0, 146.8)
- moved C43 33.1 mm to (167.6, 147.4)
- moved C22 17.6 mm to (160.5, 109.0), turned to 90 degrees
- moved C20 15.8 mm to (144.1, 134.7), turned to -90 degrees
- moved R23 14.7 mm to (188.0, 123.0)
- moved U5 14.2 mm to (164.7, 109.7), turned to 0 degrees
- moved D3 11.5 mm to (165.7, 109.7), turned to 0 degrees
- moved SW2 10.9 mm to (192.9, 122.2)
- moved R3 10.8 mm to (169.4, 111.6)
- moved R7 10.8 mm to (185.1, 112.6), turned to 90 degrees
- moved SW1 10.5 mm to (192.9, 111.4)
- moved J1 9.86 mm to (130.0, 145.3)
- moved R33 9.59 mm to (130.1, 148.9), turned to 0 degrees
- moved D1 8.44 mm to (165.7, 104.2)
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Connections:
- J1 pad 10: unconnected-(J1-Pad10) -> BACKLIGHT
- J3 pad 1: RS485A -> CANH
- J3 pad 2: RS485B -> CANL
- J3 pad 3: CANL -> RS485B
- J3 pad 4: CANH -> RS485A
- J8 pad 10: /AIN1 -> +24V
- J8 pad 5: /AIN2 -> +3V3
- J8 pad 6: /AIN3 -> +3V3
- J8 pad 9: /AIN0 -> +24V
- SW1 pad 1: unconnected-(SW1-Pad1) -> Net-(R7-Pad1)
- SW1 pad 2: Net-(R7-Pad1) -> CANL
- SW2 pad 1: unconnected-(SW2-Pad1) -> Net-(R23-Pad2)
- SW2 pad 3: Net-(R23-Pad2) -> RS485B
- SW4 pad 1: +24V -> unconnected-(SW4-Pad1)
- SW4 pad 3: unconnected-(SW4-Pad3) -> +24V
- U3 pad 14: I2S_SDAT -> I2S_SCLK
- U3 pad 27: CAN_TX -> SCLK
- U3 pad 28: SCLK -> CAN_TX
- U3 pad 29: ETH_MDIO -> ETH_MDC
- U3 pad 30: ETH_MDC -> ETH_MDIO
- U3 pad 9: I2S_SCLK -> I2S_SDAT
Routing:
- net GND: track 108.3 -> 162.9 mm, vias 29 -> 135
- net BACKLIGHT: track 0.00 -> 36.1 mm, vias 0 -> 3
- net RS485A: track 22.8 -> 47.2 mm
- net BUZZER: track 0.00 -> 22.6 mm, vias 0 -> 1
- net +3V3: track 185.1 -> 206.6 mm
- net CAN_RX: track 4.97 -> 24.7 mm, vias 0 -> 2
- net RS485B: track 32.0 -> 46.8 mm
- net +24V: track 232.1 -> 245.8 mm, vias 2 -> 6
- net AMP_PDN: track 52.7 -> 65.6 mm
- net SDA1: track 77.7 -> 65.0 mm, vias 2 -> 3
- net 485_RO: track 9.79 -> 21.3 mm, vias 0 -> 2
- net I2S_SCLK: track 19.4 -> 8.58 mm
- net 485_DI: track 26.8 -> 37.5 mm
- net SCL1: track 77.4 -> 67.9 mm
- net MOSI: track 12.4 -> 21.6 mm
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- removed copper zone on B.Cu, net +24V
Other:
- outline, holes or cut-outs redrawn
- board text added: "0..3V 0..10V"
- board text added: "100Mb"
- board text added: "24 GN 3V AC AB 24 GN 3V AD AA"
- board text added: "24V GND"
- board text added: "485 TERM OFF 485 TERM ON"
- board text added: "5V from USB ON OFF"
- board text added: "B+ B- A- A+"
- board text added: "CAN TERM OFF CAN TERM ON"
- board text added: "Ethernet LED1: On=Link Ok, Blink=Activity LED2: On=100MBits, Off=10MBits"
- board text added: "GN 3V OW"
- board text added: "Link/Act"
- board text added: "sensactHSnano2 Klaus Liebler 2022-06-22"
- board text removed: "140mm"
- board text removed: "155mm"
- board text removed: "AO0 VOUTB AIN2 GND AIN0 AO1 VOUTA AIN3 GND AIN1"
- board text removed: "B+ B- ebus/A- ebus/A+"
- board text removed: "ENAB"
- board text removed: "MC"
- board text removed: "ON"
- board text removed: "OW 3V GN"
- board text removed: "PROG"
- board text removed: "RED: POWER GREEN:INFO"
- board text removed: "TERM ON TERM OFF"
- board text removed: "sensactHSnano Klaus Liebler 2021-11-25"

Commit message: Various
Parts:
- added C48: u1, Capacitor_SMD:C_0805_2012Metric_Pad1.18x1.45mm_HandSolder, F.Cu at (151.9, 141.4)
- added JP3: SolderJumper_2_Open, Jumper:SolderJumper-2_P1.3mm_Open_RoundedPad1.0x1.5mm, F.Cu at (174.0, 143.6)
- added R2: r1, Resistor_SMD:R_1206_3216Metric_Pad1.30x1.75mm_HandSolder, F.Cu at (174.0, 143.6)
- added U10: INA219AxD, liebler_SEMICONDUCTORS:SOIC-8_3.9x4.9mm_Pitch1.27mm_handsolder, F.Cu at (156.7, 138.4)
Connections:
- D2 pad 1: +24V -> Net-(D2-Pad1)
Routing:
- net +24V: track 245.8 -> 269.0 mm
- net Net-(D2-Pad1): track 0.00 -> 20.7 mm
- net +3V3: track 206.6 -> 220.0 mm
- net SDA1: track 65.0 -> 69.3 mm
- net SCL1: track 67.9 -> 71.0 mm
- net /AO0: track 10.7 -> 11.3 mm
- net GNDA: vias 41 -> 40
- net GND: vias 135 -> 133

Commit message: Various
Parts:
- removed U13: CH340C, Package_SO:SOIC-16_3.9x9.9mm_P1.27mm
- added NT2: NetTie_2, NetTie:NetTie-2_SMD_Pad0.5mm, B.Cu at (127.7, 133.9)
- added U12: CH340K, liebler_SEMICONDUCTORS:SSOP-10_3.9x4.9mm_P1.00mm_EP, B.Cu at (127.9, 110.5)
- C21: footprint Capacitor_SMD:C_0805_2012Metric_Pad1.18x1.45mm_HandSolder -> Capacitor_SMD:C_0402_1005Metric; moved to B.Cu
- C30: moved to B.Cu
- D2: value 2A -> Schottky
- J7: footprint liebler_CONN:USB_C_Receptacle_HRO_TYPE-C-31-M-12_IMPROVED -> liebler_CONN:USB_C_Receptacle_HRO_TYPE-C-31-M-12_smaller
- Q1, Q2: footprint Package_TO_SOT_SMD:SOT-23 -> liebler_SEMICONDUCTORS:SOT-23_smaller
- U1: footprint liebler_SEMICONDUCTORS:TSSOP-28_4.4x9.7mm_Pitch0.65mm_pad_handsolder -> Package_SO:HTSSOP-28-1EP_4.4x9.7mm_P0.65mm_EP2.85x5.4mm_ThermalVias
- X1: footprint Oscillator:Oscillator_SMD_EuroQuartz_XO32-4Pin_3.2x2.5mm_HandSoldering -> Oscillator:Oscillator_SMD_SeikoEpson_SG8002CE-4Pin_3.2x2.5mm; moved to B.Cu
- moved C45 13.6 mm to (134.8, 121.0), turned to 90 degrees
- moved C30 11.6 mm to (125.7, 134.7)
- moved R47 10.9 mm to (134.8, 122.9), turned to 90 degrees
- moved C41 9.60 mm to (125.9, 114.8)
- moved C21 8.35 mm to (132.0, 134.4), turned to 90 degrees
- moved R14 8.33 mm to (129.7, 131.2), turned to 180 degrees
- moved R20 7.62 mm to (109.2, 125.1), turned to -90 degrees
- moved R32 7.48 mm to (129.4, 106.7), turned to 180 degrees
- moved C42 5.93 mm to (129.1, 114.8)
- moved Q2 5.41 mm to (130.4, 116.5)
- moved R44 4.77 mm to (159.6, 123.7), turned to 180 degrees
- moved R28 3.90 mm to (133.2, 119.0)
- moved R11 3.83 mm to (156.6, 120.8), turned to 90 degrees
- moved X1 3.08 mm to (129.7, 133.9), turned to 90 degrees
- moved R16 2.70 mm to (127.3, 123.2)
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Connections:
- C21 pad 2: GND -> /eth/CLK_GND
- C42 pad 2: GND -> Net-(C42-Pad2)
- U3 pad 5: SW1 -> CAN_RX
- U3 pad 6: CAN_RX -> SW1
- X1 pad 2: GND -> /eth/CLK_GND
Routing:
- net GND: track 162.9 -> 122.4 mm, vias 133 -> 92
- net +5P: track 26.0 -> 15.3 mm, vias 2 -> 3
- net +24V: track 269.0 -> 260.0 mm
- net PROG_RX: track 2.11 -> 9.73 mm
- net Net-(R14-Pad2): track 1.39 -> 8.65 mm, vias 0 -> 2
- net Net-(J4-Pad11): track 8.91 -> 1.70 mm, vias 1 -> 0
- net PROG_TX: track 7.30 -> 14.4 mm
- net AMP_PDN: track 65.6 -> 58.7 mm, vias 2 -> 3
- net Net-(R14-Pad1): track 8.92 -> 2.30 mm, vias 2 -> 0
- net PROG_EN: track 52.7 -> 58.6 mm
- net CANH: track 36.2 -> 30.7 mm
- net /prog/DTR: track 35.6 -> 40.6 mm
- net /eth/LED2: track 13.6 -> 18.1 mm
- net SCL1: track 71.0 -> 67.3 mm
- net /eth/VDD2A: track 50.1 -> 53.3 mm, vias 3 -> 4
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- added copper zone on B.Cu, net /eth/CLK_GND
Other:
- board text added: "485A"
- board text added: "485B"
- board text added: "A+"
- board text added: "A-"
- board text added: "B+"
- board text added: "B-"
- board text added: "CANH"
- board text added: "CANL"
- board text added: "Link"
- board text added: "SCL 3V3 IN0 SDA NC IN1 24V 24V GND GND"
- board text removed: "B+ B- A- A+"
- board text removed: "Link/Act"
- board text removed: "SCL 3V3 IN1 SDA NC IN2 24V 24V GND GND"
