File: pcb/sensactInpExt2/sensactInpExt.kicad_pcb (KiCad board)
At the start: 2 copper layers, 97 x 61 mm, 106 parts, among them J1 SensactBusConnector, J2 IN1-IN8, J3 IN8-IN16, J4 1Wire, SW1 A2, SW2 A1, SW3 A0, SW4 AD0, SW5 AD0, SW6 AD1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

Commit message: Various
Parts:
- added H10: MountingHole, MountingHole:MountingHole_3.2mm_M3, F.Cu at (131.3, 153.1)
- added H7: MountingHole, MountingHole:MountingHole_3.2mm_M3, F.Cu at (162.5, 132.0)
- added H8: MountingHole, MountingHole:MountingHole_3.2mm_M3, F.Cu at (137.5, 132.0)
- added H9: MountingHole, MountingHole:MountingHole_3.2mm_M3, F.Cu at (132.5, 145.2)
- H1, H2: footprint MountingHole:MountingHole_2.2mm_M2_DIN965 -> MountingHole:MountingHole_3.2mm_M3
- SW1: value A2 -> 0 A2 1
- SW2: value A1 -> 0 A1 1
- SW3: value A0 -> 0 A0 1
- SW4: value AD0 -> INT? INT0
- SW5: value AD0 -> INT1 INT2
- moved SW4 28.9 mm to (150.5, 125.0)
- moved SW5 24.1 mm to (159.2, 125.0)
- moved H3 17.7 mm to (150.0, 145.0)
- moved H1 12.6 mm to (139.8, 143.2)
- moved C1 12.1 mm to (144.2, 125.0)
- moved C19 12.1 mm to (144.2, 123.0)
- moved H4 11.3 mm to (160.0, 145.0)
- moved SW1 9.93 mm to (147.0, 109.3)
- moved H2 9.74 mm to (172.8, 143.2)
- moved DD1 7.90 mm to (138.0, 121.6)
- moved SW3 6.57 mm to (147.0, 116.5)
- moved C17 4.08 mm to (125.4, 150.7), turned to 180 degrees
- moved C18 3.71 mm to (125.4, 152.7)
- moved SW2 3.70 mm to (147.0, 112.9)
- moved J1 2.80 mm to (181.6, 132.4)
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Connections:
- J1 pad 7: Net-(J1-Pad7) -> unconnected-(J1-Pad7)
- J1 pad 8: Net-(J1-Pad8) -> unconnected-(J1-Pad8)
- U5 pad 6: Net-(U5-Pad6) -> unconnected-(U5-Pad6)
Routing:
- net Net-(DD1-Pad1): track 46.7 -> 11.8 mm, vias 2 -> 1
- net /INT0: track 7.50 -> 40.2 mm
- net /INT1: track 9.60 -> 35.7 mm
- net /INT2: track 7.85 -> 31.8 mm
- net /I15: track 20.4 -> 31.1 mm
- net /I16: track 26.0 -> 36.5 mm
- net /I14: track 19.0 -> 29.2 mm
- net /I13: track 22.7 -> 31.9 mm
- net Net-(SW4-Pad1): track 4.64 -> 12.4 mm
- net /I2: track 21.8 -> 16.2 mm
- net /I9: track 13.1 -> 18.4 mm
- net +3V3: track 255.2 -> 250.3 mm
- net /I11: track 12.3 -> 17.0 mm
- net /I3: track 19.6 -> 14.9 mm
- net /I10: track 10.9 -> 15.6 mm
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Other:
- outline, holes or cut-outs redrawn
- net class Default removed
- board text added: "3V SDA INT1 NC GND"
- board text added: "GND 1Wire"
- board text added: "IN1"
- board text added: "IN10"
- board text added: "IN11"
- board text added: "IN12"
- board text added: "IN13"
- board text added: "IN14"
- board text added: "IN15"
- board text added: "IN16"
- board text added: "IN16 IN15 IN14 IN13 IN12 IN11 IN10 IN9 IN8 IN7 IN6 IN5 IN4 IN3 IN2 IN1"
- board text added: "IN3"
- board text added: "IN4"
- board text added: "IN5"
- board text added: "IN6"
- board text added: "IN7"
- board text added: "IN8"
- board text added: "IN9"
- board text added: "SCL INT0 INT2 NC GND"
- board text removed: "1 GND"
- board text removed: "1W GND"
