File: pcb/sensactInpExt2/input4.kicad_sch (KiCad schematic)
At the start: 13 parts

Commit message: Various
Parts:
- gave numbers to parts that had none: 13
Changed lines of the file:
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@@
   (symbol (lib_id "power:+3V3") (at 171.45 77.47 270) (unit 1)
     (in_bom yes) (on_board yes)
-    (property "Reference" "#PWR?" (id 0) (at 167.64 77.47 0)
+    (property "Reference" "#PWR0104" (id 0) (at 167.64 77.47 0)
       (effects (font (size 1.27 1.27)) hide)
     )
@@
   (symbol (lib_id "Device:R") (at 133.35 73.66 270) (unit 1)
     (in_bom yes) (on_board yes)
-    (property "Reference" "R?" (id 0) (at 133.35 75.692 90))
+    (property "Reference" "R1" (id 0) (at 133.35 75.692 90))
     (property "Value" "10R" (id 1) (at 133.35 73.66 90))
     (property "Footprint" "Resistor_SMD:R_0603_1608Metric" (id 2) (at 133.35 71.882 90)
@@
   (symbol (lib_id "power:GND") (at 127 90.17 270) (unit 1)
     (in_bom yes) (on_board yes)
-    (property "Reference" "#PWR?" (id 0) (at 120.65 90.17 0)
+    (property "Reference" "#PWR0102" (id 0) (at 120.65 90.17 0)
       (effects (font (size 1.27 1.27)) hide)
     )
@@
   (symbol (lib_id "power:GND") (at 175.26 90.17 90) (unit 1)
     (in_bom yes) (on_board yes)
-    (property "Reference" "#PWR?" (id 0) (at 181.61 90.17 0)
+    (property "Reference" "#PWR0106" (id 0) (at 181.61 90.17 0)
       (effects (font (size 1.27 1.27)) hide)
     )
@@
   (symbol (lib_id "Device:C") (at 170.18 90.17 270) (unit 1)
     (in_bom yes) (on_board yes)
-    (property "Reference" "C?" (id 0) (at 172.72 90.805 0)
+    (property "Reference" "C8" (id 0) (at 172.72 90.805 0)
       (effects (font (size 1.27 1.27)) (justify left))
     )
@@
   (symbol (lib_id "Device:C") (at 132.08 64.77 270) (unit 1)
     (in_bom yes) (on_board yes)
-    (property "Reference" "C?" (id 0) (at 134.62 65.405 0)
+    (property "Reference" "C3" (id 0) (at 134.62 65.405 0)
       (effects (font (size 1.27 1.27)) (justify left))
     )
@@
   (symbol (lib_id "Device:R") (at 168.91 81.28 270) (unit 1)
     (in_bom yes) (on_board yes)
-    (property "Reference" "R?" (id 0) (at 168.91 83.312 90))
+    (property "Reference" "R14" (id 0) (at 168.91 83.312 90))
     (property "Value" "10R" (id 1) (at 168.91 81.28 90))
     (property "Footprint" "Resistor_SMD:R_0603_1608Metric" (id 2) (at 168.91 79.502 90)
@@
   (symbol (lib_id "Device:R") (at 137.16 68.58 0) (unit 1)
     (in_bom yes) (on_board yes)
-    (property "Reference" "R?" (id 0) (at 139.192 68.58 90))
+    (property "Reference" "R5" (id 0) (at 139.192 68.58 90))
     (property "Value" "1k" (id 1) (at 137.16 68.58 90))
     (property "Footprint" "Resistor_SMD:R_0603_1608Metric" (id 2) (at 135.382 68.58 90)
@@
   (symbol (lib_id "Device:R") (at 133.35 81.28 270) (unit 1)
     (in_bom yes) (on_board yes)
-    (property "Reference" "R?" (id 0) (at 133.35 83.312 90))
+    (property "Reference" "R2" (id 0) (at 133.35 83.312 90))
     (property "Value" "10R" (id 1) (at 133.35 81.28 90))
     (property "Footprint" "Resistor_SMD:R_0603_1608Metric" (id 2) (at 133.35 79.502 90)
@@
   (symbol (lib_id "Device:C") (at 170.18 64.77 270) (unit 1)
     (in_bom yes) (on_board yes)
-    (property "Reference" "C?" (id 0) (at 172.72 65.405 0)
+    (property "Reference" "C7" (id 0) (at 172.72 65.405 0)
       (effects (font (size 1.27 1.27)) (justify left))
     )
@@
   (symbol (lib_id "power:GND") (at 175.26 64.77 90) (unit 1)
     (in_bom yes) (on_board yes)
-    (property "Reference" "#PWR?" (id 0) (at 181.61 64.77 0)
+    (property "Reference" "#PWR0105" (id 0) (at 181.61 64.77 0)
       (effects (font (size 1.27 1.27)) hide)
     )
@@
   (symbol (lib_id "sensactInpExt-rescue:SRV05") (at 151.13 77.47 0) (unit 1)
     (in_bom yes) (on_board yes)
-    (property "Reference" "U?" (id 0) (at 151.13 71.12 0))
+    (property "Reference" "U1" (id 0) (at 151.13 71.12 0))
     (property "Value" "SRV05" (id 1) (at 151.13 83.82 0))
     (property "Footprint" "Package_TO_SOT_SMD:SOT-23-6" (id 2) (at 151.13 77.47 0)
@@
   (symbol (lib_id "Device:R") (at 137.16 86.36 0) (unit 1)
     (in_bom yes) (on_board yes)
-    (property "Reference" "R?" (id 0) (at 139.192 86.36 90))
+    (property "Reference" "R6" (id 0) (at 139.192 86.36 90))
     (property "Value" "1k" (id 1) (at 137.16 86.36 90))
     (property "Footprint" "Resistor_SMD:R_0805_2012Metric_Pad1.20x1.40mm_HandSolder" (id 2) (at 135.382 86.36 90)
@@
   (symbol (lib_id "power:GND") (at 127 64.77 270) (unit 1)
     (in_bom yes) (on_board yes)
-    (property "Reference" "#PWR?" (id 0) (at 120.65 64.77 0)
+    (property "Reference" "#PWR0103" (id 0) (at 120.65 64.77 0)
       (effects (font (size 1.27 1.27)) hide)
     )
@@
   (symbol (lib_id "Device:R") (at 168.91 73.66 270) (unit 1)
     (in_bom yes) (on_board yes)
-    (property "Reference" "R?" (id 0) (at 168.91 75.692 90))
+    (property "Reference" "R13" (id 0) (at 168.91 75.692 90))
     (property "Value" "10R" (id 1) (at 168.91 73.66 90))
     (property "Footprint" "Resistor_SMD:R_0603_1608Metric" (id 2) (at 168.91 71.882 90)
@@
   (symbol (lib_id "power:GND") (at 130.81 77.47 270) (unit 1)
     (in_bom yes) (on_board yes)
-    (property "Reference" "#PWR?" (id 0) (at 124.46 77.47 0)
+    (property "Reference" "#PWR0101" (id 0) (at 124.46 77.47 0)
       (effects (font (size 1.27 1.27)) hide)
     )
@@
   (symbol (lib_id "Device:R") (at 165.1 68.58 0) (unit 1)
     (in_bom yes) (on_board yes)
-    (property "Reference" "R?" (id 0) (at 167.132 68.58 90))
+    (property "Reference" "R9" (id 0) (at 167.132 68.58 90))
     (property "Value" "1k" (id 1) (at 165.1 68.58 90))
     (property "Footprint" "Resistor_SMD:R_0603_1608Metric" (id 2) (at 163.322 68.58 90)
@@
   (symbol (lib_id "Device:R") (at 165.1 86.36 0) (unit 1)
     (in_bom yes) (on_board yes)
-    (property "Reference" "R?" (id 0) (at 167.132 86.36 90))
+    (property "Reference" "R10" (id 0) (at 167.132 86.36 90))
     (property "Value" "1k" (id 1) (at 165.1 86.36 90))
     (property "Footprint" "Resistor_SMD:R_0603_1608Metric" (id 2) (at 163.322 86.36 90)
@@
   (symbol (lib_id "Device:C") (at 132.08 90.17 270) (unit 1)
     (in_bom yes) (on_board yes)
-    (property "Reference" "C?" (id 0) (at 134.62 90.805 0)
-      (effects (font (size 1.27 1.27)) (justify left))
-    )
+    (property "Reference" "C4" (id 0) (at 134.62 90.805 0)
+      (effects (font (size 1.27 1.27)) (justify left))
+    )
