File: pcb/sensactOutdoor/sensactOutdoor.kicad_pcb (KiCad board)
At the start: 2 copper layers, 100 x 81 mm, 146 parts, among them J1 48V, J10 LED_EXT, J11 EXT2, J13 RGB, J15 PWM_OUT, J16 24V, J2 Conn_01x03, J3 Conn_01x03, J4 PROG, J5 LED CC, J6 CAN BUS, J7 EXT1, J8 PWM_OUT, J9 230V, K1 ALDP105W, K2 ALDP105W, K3 ALDP105W, K4 ALDP105W, K5 ALDP105W, K6 ALDP105W, Q1 N, Q10 BC847, Q11 BC847, Q2 N, Q3 N, Q4 N, Q5 N, Q6 BC847, Q7 BC847, Q8 BC847, Q9 BC847, SW1 SW_SPDT, SW2 RESET, SW3 TERM ON->, U1 ESP32-WROOM-32U, U2 BP1808, U3 LM2596Board, U4 SN65HVD230, U5 AMS1117-3.3, U6 RF, U7 DCDC_MP2315, U8 EL817, U9 MAX98357_MODULE

Commit message: Various
Parts:
- removed J16: 24V, liebler_CONN:PhoenixContact_MSTBV_2,5_2-G-5,08_1x02_P5.08mm_Vertical
- removed R44: 4k7, Resistor_SMD:R_0805_2012Metric_Pad1.20x1.40mm_HandSolder
- added J12: OUT, liebler_CONN:KF128-5,00-3P, F.Cu at (28.7, 54.0)
- added JP1: PWM5_CAN, Jumper:SolderJumper-3_P1.3mm_Open_RoundedPad1.0x1.5mm, B.Cu at (47.9, 40.2)
- added M1: BxxyyS-1WR, liebler_MODULES:BxxxxS-1W, F.Cu at (39.9, 41.9)
- D19: value LPWM2 -> P2
- D20: value LPWM3 -> P3
- D21: value LPWM4 -> P4
- D8: value LPWM5 -> P5
- D9: value LPWM1 -> P1
- J1, J5: footprint liebler_CONN:PhoenixContact_MSTBV_2,5_2-G-5,08_1x02_P5.08mm_Vertical -> liebler_CONN:KF128-5,00-2P
- J15: value PWM_OUT -> OUT; footprint Connector_Phoenix_MC:PhoenixContact_MCV_1,5_2-G-3.5_1x02_P3.50mm_Vertical -> liebler_CONN:KF128-5,00-2P
- J2, J3: footprint Connector_Phoenix_GMSTB:PhoenixContact_GMSTBVA_2,5_3-G-7,62_1x03_P7.62mm_Vertical -> liebler_CONN:KF128-7,50-3P
- J8: value PWM_OUT -> OUT; footprint Connector_Phoenix_MC:PhoenixContact_MCV_1,5_4-G-3.5_1x04_P3.50mm_Vertical -> liebler_CONN:KF128-5,00-3P
- J9: footprint Connector_Phoenix_GMSTB:PhoenixContact_GMSTBVA_2,5_2-G-7,62_1x02_P7.62mm_Vertical -> liebler_CONN:KF128-7,50-2P
- Q1, Q2, Q3, Q4, Q5: value N -> AO3400A; footprint Package_TO_SOT_THT:TO-220F-3_Vertical -> Package_TO_SOT_SMD:SOT-23
- U4: value SN65HVD230 -> ISO1050DUB; footprint liebler_SEMICONDUCTORS:SOIC-8_3.9x4.9mm_Pitch1.27mm_handsolder -> Package_SO:SOP-8_6.62x9.15mm_P2.54mm
- moved U7 24.5 mm to (62.3, 84.4)
- moved R22 19.8 mm to (36.5, 56.5), turned to 180 degrees
- moved R21 17.6 mm to (38.5, 56.5), turned to 180 degrees
- moved R20 14.7 mm to (36.0, 51.5), turned to 180 degrees
- moved R19 12.4 mm to (38.0, 51.5)
- moved R15 10.8 mm to (37.0, 26.5), turned to 180 degrees
- moved R18 10.4 mm to (37.0, 31.5), turned to 180 degrees
- moved R43 10.3 mm to (40.5, 54.0)
- moved Q4 9.64 mm to (36.0, 49.0)
- moved Q5 9.45 mm to (36.0, 54.0)
- moved R14 9.31 mm to (39.0, 26.5), turned to 180 degrees
- moved Q1 9.26 mm to (36.0, 59.0)
- moved R17 7.88 mm to (39.0, 31.5), turned to 180 degrees
- moved J3 7.70 mm to (120.5, 64.8), turned to 90 degrees
- moved J2 7.65 mm to (120.5, 33.6), turned to 90 degrees
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Connections:
- D19 pad 1: GND -> Net-(D19-Pad1)
- D19 pad 2: Net-(D19-Pad2) -> PWM2
- D20 pad 1: GND -> Net-(D20-Pad1)
- D20 pad 2: Net-(D20-Pad2) -> PWM3
- D21 pad 1: GND -> Net-(D21-Pad1)
- D21 pad 2: Net-(D21-Pad2) -> PWM4
- D22 pad 3: GND -> Net-(D22-Pad3)
- D8 pad 1: GND -> Net-(D8-Pad1)
- D8 pad 2: Net-(D8-Pad2) -> PWM5
- D9 pad 1: GND -> Net-(D9-Pad1)
- D9 pad 2: Net-(D9-Pad2) -> PWM1
- J15 pad 1: /PWM_1 -> /PWM_2
- J15 pad 2: /PWM_2 -> /PWM_1
- J2 pad 1: /L1 -> /L3
- J2 pad 3: /L3 -> /L1
- J3 pad 1: /L4 -> /L6
- J3 pad 3: /L6 -> /L4
- J8 pad 1: +24V -> Net-(J8-Pad1)
- J8 pad 2: /PWM_3 -> Net-(J8-Pad1)
- J8 pad 3: /PWM_4 -> GND
- J9 pad 1: /L -> Net-(F1-Pad2)
- J9 pad 2: Net-(F1-Pad2) -> /L
- Q1 pad 2: /PWM_5 -> GND
- Q1 pad 3: GND -> /PWM_5
- Q2 pad 2: /PWM_1 -> GND
- Q2 pad 3: GND -> /PWM_1
- Q3 pad 2: /PWM_2 -> GND
- Q3 pad 3: GND -> /PWM_2
- Q4 pad 2: /PWM_3 -> GND
- Q4 pad 3: GND -> /PWM_3
- Q5 pad 2: /PWM_4 -> GND
- Q5 pad 3: GND -> /PWM_4
- R11 pad 1: CAN_TX -> PWM5
- R35 pad 1: CAN_TX -> Net-(D8-Pad1)
- R35 pad 2: Net-(D8-Pad2) -> GND
- R36 pad 1: PWM1 -> Net-(D9-Pad1)
- R36 pad 2: Net-(D9-Pad2) -> GND
- R41 pad 1: PWM2 -> Net-(D19-Pad1)
- R41 pad 2: Net-(D19-Pad2) -> GND
- R42 pad 1: PWM3 -> Net-(D20-Pad1)
- R42 pad 2: Net-(D20-Pad2) -> GND
- R43 pad 1: PWM4 -> Net-(D21-Pad1)
- R43 pad 2: Net-(D21-Pad2) -> GND
- U1 pad 14: CAN_TX -> Net-(JP1-Pad2)
- U4 pad 1: CAN_TX -> +3V3
- U4 pad 2: GND -> CAN_RX
- U4 pad 3: +3V3 -> CAN_TX
- U4 pad 4: CAN_RX -> GND
- U4 pad 5: unconnected-(U4-Pad5) -> Net-(D22-Pad3)
Routing:
- net Net-(D22-Pad3): track 0.00 -> 33.8 mm
- net PWM5: track 0.00 -> 29.0 mm, vias 0 -> 1
- net CAN_TX: track 29.7 -> 4.98 mm, vias 3 -> 0
- net +5V: track 244.2 -> 263.7 mm
- net Net-(M1-Pad4): track 1.98 -> 17.3 mm
- net CAN_RX: track 83.3 -> 92.9 mm, vias 3 -> 2
- net /PWM_2: track 15.0 -> 6.36 mm
- net /PWM_3: track 14.8 -> 6.36 mm
- net /PWM_1: track 14.5 -> 6.36 mm
- net /PWM_4: track 14.4 -> 6.36 mm
- net /PWM_5: track 14.0 -> 6.36 mm
- net PWM4: track 22.7 -> 30.2 mm
- net Net-(Q5-Pad1): track 9.98 -> 2.56 mm
- net +3V3: track 142.6 -> 149.8 mm, vias 6 -> 43
- net CE: track 42.5 -> 49.6 mm
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- added copper zone on B.Cu, net +3V3
Other:
- board text added: "sensactOutdoor V4 2022-08-21"
- board text removed: "sensactOutdoor V4 2022-08-02"
