File: pcb/sensactHsIO5-pca9685/sensactHsIO5.kicad_pcb (KiCad board)
At the start: 2 copper layers, 90 x 67.5 mm, 104 parts, among them J4 Conn_01x08, J5 Conn_01x08, J8 Bus, SW4 SW_DIP_x08, SW5 SW_DIP_x08, SW7 Auto Manu, U1 LM358, U3 PCA9685PW, U4 L78L15_SOT89, U8 ULN2803A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

Commit message: PCBs as ordered at JLCPCB
Parts:
- R1, R2: value 4k7 -> 4k7opt
- U3: footprint Package_SO:TSSOP-28_4.4x9.7mm_P0.65mm -> liebler_SEMICONDUCTORS:TSSOP-28_4.4x9.7mm_Pitch0.65mm_handsolder
- moved C7 0.71 mm to (142.2, 111.3)
- moved C2 0.67 mm to (143.5, 110.8)
- moved R7 0.63 mm to (143.1, 107.1)
- turned R12 to 180 degrees
- turned R13 to 180 degrees
- turned R3 to 180 degrees
- turned R5 to 180 degrees
- turned R6 to 180 degrees
- turned R9 to 180 degrees
Routing:
- net +3V3: track 150.8 -> 152.4 mm
- net Net-(R5-Pad1): track 16.3 -> 14.9 mm
- net Net-(R12-Pad1): track 7.88 -> 6.42 mm
- net Net-(R6-Pad1): track 13.5 -> 12.0 mm
- net Net-(R3-Pad1): track 19.1 -> 17.7 mm
- net Net-(R9-Pad1): track 10.7 -> 9.23 mm
- net Net-(R18-Pad1): track 4.78 -> 5.99 mm
- net /A0: track 14.1 -> 15.2 mm
- net /A1: track 12.1 -> 13.2 mm
- net /A2: track 11.3 -> 12.1 mm
- net Net-(R19-Pad1): track 7.27 -> 7.99 mm
- net /!OE: track 14.4 -> 15.0 mm
- net Net-(R17-Pad1): track 3.02 -> 3.69 mm
- net Net-(R24-Pad1): track 18.5 -> 19.2 mm
- net Net-(R25-Pad1): track 21.3 -> 22.0 mm
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
Commit message: Various updates, new version with ESP32 in beta test :-)
Parts:
- added J1: Conn_01x08, liebler_CONN:PhoenixContact_MC_0,5_8-G-2.5_1x08_P2.50mm_Horizontal, B.Cu at (114.0, 125.8)
- added J2: Conn_01x08, liebler_CONN:PhoenixContact_MC_0,5_8-G-2.5_1x08_P2.50mm_Horizontal, B.Cu at (114.0, 148.6)
- added J3: Conn_01x08, liebler_CONN:PhoenixContact_MC_0,5_8-G-2.5_1x08_P2.50mm_Horizontal, B.Cu at (186.1, 112.2)
- R12, R13, R15, R16, R17, R18, R19, R21, R22, R23, R24, R25, R3, R5, R6, R9: footprint Resistor_SMD:R_0402_1005Metric -> Resistor_SMD:R_0805_2012Metric
- moved JP34 14.3 mm to (178.0, 145.9)
- moved JP33 14.3 mm to (178.0, 143.3)
- moved J8 13.5 mm to (181.8, 147.8)
- moved R2 13.5 mm to (183.1, 149.2)
- moved R1 13.0 mm to (180.2, 147.2)
- moved R25 8.20 mm to (163.5, 104.6)
- moved R3 7.25 mm to (135.4, 104.6)
- moved R24 2.69 mm to (165.4, 101.2), turned to 90 degrees
- moved R16 2.19 mm to (149.2, 99.2), turned to 90 degrees
- moved R23 2.05 mm to (163.5, 101.2), turned to 90 degrees
- moved R15 1.98 mm to (143.0, 101.2), turned to 90 degrees
- moved R5 1.67 mm to (133.5, 101.2), turned to 90 degrees
- moved R17 1.56 mm to (154.0, 101.2), turned to 90 degrees
- moved R22 1.54 mm to (161.6, 101.2), turned to 90 degrees
- moved R13 1.43 mm to (141.1, 101.2), turned to 90 degrees
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Routing:
- net +24V: track 143.8 -> 248.0 mm
- net Net-(U3-LED0): track 22.0 -> 11.7 mm
- net SDA1: track 42.9 -> 51.7 mm
- net +3V3: track 152.4 -> 161.1 mm
- net Net-(U3-LED15): track 17.7 -> 9.63 mm
- net SCL1: track 43.0 -> 51.0 mm
- net CPU0: track 95.2 -> 102.6 mm
- net CPU15: track 35.1 -> 40.5 mm
- net Net-(U3-LED1): track 19.2 -> 15.3 mm
- net Net-(U3-LED2): track 16.3 -> 13.1 mm
- net Net-(U3-LED3): track 13.6 -> 11.0 mm
- net /io/CONN0: track 11.9 -> 14.4 mm
- net /io/CONN1: track 11.9 -> 14.3 mm
- net Net-(U3-LED8): track 2.37 -> 4.64 mm
- net /io/CONN6: track 11.8 -> 14.0 mm
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Other:
- board text added: "24V"
- board text added: "3V3"
- board text added: "GND"
