File: pcb/sensactHsNano3/psu.kicad_sch (KiCad schematic)
At the start: 10 parts, among them U7 RY8310

Commit message: Various changes
Other:
- note added: "PSU"
Changed lines of the file:
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@@
+    (stroke (width 0) (type default))
+  )
+  (polyline (pts (xy 140.97 72.39) (xy 36.83 72.39))
     (stroke (width 0) (type default))
   )
   (wire (pts (xy 85.725 26.67) (xy 93.345 26.67))
+    (stroke (width 0) (type default))
+  )
+  (polyline (pts (xy 36.83 22.86) (xy 140.97 22.86))
     (stroke (width 0) (type default))
   )
@@
     (stroke (width 0) (type default))
   )
+  (polyline (pts (xy 140.97 22.86) (xy 140.97 72.39))
+    (stroke (width 0) (type default))
+  )
   (wire (pts (xy 45.085 66.04) (xy 51.435 66.04))
     (stroke (width 0) (type default))
@@
   )
   (wire (pts (xy 40.005 43.18) (xy 40.005 66.04))
+    (stroke (width 0) (type default))
+  )
+  (polyline (pts (xy 36.83 22.86) (xy 36.83 72.39))
     (stroke (width 0) (type default))
   )
@@
     (effects (font (size 1.27 1.27)) (justify left bottom))
   )
+  (text "PSU" (at 36.83 22.86 0)
+    (effects (font (size 1.27 1.27)) (justify left bottom))
+  )
