File: pcb/din_schiene_seitenwand/din_schiene_seitenwand.kicad_pcb (KiCad board)
At the start: 2 copper layers, 90 x 66 mm, 0 parts

Commit message: Updated various PCB
Other:
- outline, holes or cut-outs redrawn
Changed lines of the file:
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@@
   (net 0 "")
   (gr_line (start 132.5 149) (end 167.5 149) (layer "Dwgs.User") (width 0.15))
-  (gr_line (start 168.75 153) (end 176.25 153) (layer "Edge.Cuts") (width 0.1))
-  (gr_line (start 195 156) (end 169.25 156) (layer "Edge.Cuts") (width 0.1))
+  (gr_arc (start 172 90) (mid 172.353553 90.146447) (end 172.5 90.5) (layer "Edge.Cuts") (width 0.1))
+  (gr_line (start 168.75 153) (end 175.75 153) (layer "Edge.Cuts") (width 0.1))
+  (gr_arc (start 194.5 153) (mid 194.853553 153.146447) (end 195 153.5) (layer "Edge.Cuts") (width 0.1))
+  (gr_line (start 194.5 156) (end 169.25 156) (layer "Edge.Cuts") (width 0.1))
   (gr_line (start 172.5 93.6) (end 172.5 106) (layer "Edge.Cuts") (width 0.1))
-  (gr_line (start 105 156) (end 105 150) (layer "Edge.Cuts") (width 0.1))
-  (gr_line (start 168.5 93.6) (end 168.5 92) (layer "Edge.Cuts") (width 0.1))
-  (gr_line (start 195 106) (end 195 150) (layer "Edge.Cuts") (width 0.1))
-  (gr_circle (center 132 153) (end 132 152) (layer "Edge.Cuts") (width 0.1) (fill none))
+  (gr_line (start 105 155.5) (end 105 150) (layer "Edge.Cuts") (width 0.1))
+  (gr_arc (start 176.25 152.5) (mid 176.603553 153.353553) (end 175.75 153) (layer "Edge.Cuts") (width 0.1))
+  (gr_arc (start 195 155.5) (mid 194.853553 155.853553) (end 194.5 156) (layer "Edge.Cuts") (width 0.1))
+  (gr_line (start 168.5 93.1) (end 168.5 92.5) (layer "Edge.Cuts") (width 0.1))
+  (gr_line (start 195 150) (end 188 150) (layer "Edge.Cuts") (width 0.1))
+  (gr_line (start 195 106.5) (end 195 150) (layer "Edge.Cuts") (width 0.1))
+  (gr_circle (center 131.5 153.5) (end 131.5 152.5) (layer "Edge.Cuts") (width 0.1) (fill none))
   (gr_line (start 127.5 106) (end 127.5 93.6) (layer "Edge.Cuts") (width 0.1))
+  (gr_arc (start 194.5 106) (mid 194.853553 106.146447) (end 195 106.5) (layer "Edge.Cuts") (width 0.1))
+  (gr_arc (start 105.5 156) (mid 105.146447 155.853553) (end 105 155.5) (layer "Edge.Cuts") (width 0.1))
   (gr_circle (center 170.25 103.75) (end 170.25 102.75) (layer "Edge.Cuts") (width 0.1) (fill none))
-  (gr_line (start 168.5 92) (end 172.5 92) (layer "Edge.Cuts") (width 0.1))
-  (gr_line (start 127.5 92) (end 131.5 92) (layer "Edge.Cuts") (width 0.1))
-  (gr_line (start 176.25 153) (end 176.25 150) (layer "Edge.Cuts") (width 0.1))
-  (gr_line (start 105 106) (end 127.5 106) (layer "Edge.Cuts") (width 0.1))
+  (gr_line (start 169 92) (end 172.5 92) (layer "Edge.Cuts") (width 0.1))
+  (gr_line (start 188 153) (end 194.5 153) (layer "Edge.Cuts") (width 0.1))
+  (gr_arc (start 169 93.6) (mid 168.146447 93.953553) (end 168.5 93.1) (layer "Edge.Cuts") (width 0.1))
+  (gr_line (start 127.5 92) (end 131 92) (layer "Edge.Cuts") (width 0.1))
+  (gr_line (start 176.25 152.5) (end 176.25 150.5) (layer "Edge.Cuts") (width 0.1))
+  (gr_line (start 105.5 106) (end 127.5 106) (layer "Edge.Cuts") (width 0.1))
   (gr_line (start 172.5 92) (end 172.5 90.5) (layer "Edge.Cuts") (width 0.1))
   (gr_circle (center 178.25 151.5) (end 178.25 150.5) (layer "Edge.Cuts") (width 0.1) (fill none))
-  (gr_line (start 195 150) (end 195 156) (layer "Edge.Cuts") (width 0.1))
+  (gr_line (start 195 153.5) (end 195 155.5) (layer "Edge.Cuts") (width 0.1))
   (gr_line (start 128 90) (end 172 90) (layer "Edge.Cuts") (width 0.1))
+  (gr_arc (start 187.5 150.5) (mid 187.146447 149.646447) (end 188 150) (layer "Edge.Cuts") (width 0.1))
+  (gr_arc (start 131 92) (mid 131.853553 91.646447) (end 131.5 92.5) (layer "Edge.Cuts") (width 0.1))
   (gr_line (start 169.25 156) (end 168.75 153) (layer "Edge.Cuts") (width 0.1))
-  (gr_line (start 172 90) (end 172.5 90.5) (layer "Edge.Cuts") (width 0.1))
+  (gr_arc (start 131.5 93.1) (mid 131.853553 93.953553) (end 131 93.6) (layer "Edge.Cuts") (width 0.1))
   (gr_line (start 150 150) (end 132.5 150) (layer "Edge.Cuts") (width 0.1))
-  (gr_line (start 134 151.5) (end 134 156) (layer "Edge.Cuts") (width 0.1))
-  (gr_line (start 128 90) (end 127.5 90.5) (layer "Edge.Cuts") (width 0.1))
+  (gr_line (start 134 151.6) (end 134 156) (layer "Edge.Cuts") (width 0.1))
   (gr_line (start 127.5 92) (end 127.5 90.5) (layer "Edge.Cuts") (width 0.1))
-  (gr_line (start 172.5 106) (end 195 106) (layer "Edge.Cuts") (width 0.1))
-  (gr_line (start 176.25 150) (end 150 150) (layer "Edge.Cuts") (width 0.1))
-  (gr_line (start 105 150) (end 105 106) (layer "Edge.Cuts") (width 0.1))
-  (gr_line (start 132.5 150) (end 132.5 151) (layer "Edge.Cuts") (width 0.1))
-  (gr_line (start 134 156) (end 105 156) (layer "Edge.Cuts") (width 0.1))
-  (gr_line (start 172.5 93.6) (end 168.5 93.6) (layer "Edge.Cuts") (width 0.1))
-  (gr_line (start 132.5 151) (end 134 151.5) (layer "Edge.Cuts") (width 0.1))
-  (gr_line (start 131.5 92) (end 131.5 93.6) (layer "Edge.Cuts") (width 0.1))
+  (gr_line (start 172.5 106) (end 194.5 106) (layer "Edge.Cuts") (width 0.1))
+  (gr_arc (start 175.75 150) (mid 176.603553 149.646447) (end 176.25 150.5) (layer "Edge.Cuts") (width 0.1))
+  (gr_line (start 175.75 150) (end 150 150) (layer "Edge.Cuts") (width 0.1))
+  (gr_line (start 105 150) (end 105 106.5) (layer "Edge.Cuts") (width 0.1))
+  (gr_arc (start 188 153) (mid 187.146447 153.353553) (end 187.5 152.5) (layer "Edge.Cuts") (width 0.1))
+  (gr_arc (start 127.5 90.5) (mid 127.646447 90.146447) (end 128 90) (layer "Edge.Cuts") (width 0.1))
+  (gr_line (start 132.5 150) (end 132.5 151.2) (layer "Edge.Cuts") (width 0.1))
+  (gr_line (start 134 156) (end 105.5 156) (layer "Edge.Cuts") (width 0.1))
+  (gr_arc (start 105 106.5) (mid 105.146447 106.146447) (end 105.5 106) (layer "Edge.Cuts") (width 0.1))
+  (gr_arc (start 168.5 92.5) (mid 168.146447 91.646447) (end 169 92) (layer "Edge.Cuts") (width 0.1))
+  (gr_line (start 172.5 93.6) (end 169 93.6) (layer "Edge.Cuts") (width 0.1))
+  (gr_line (start 187.5 150.5) (end 187.5 152.5) (layer "Edge.Cuts") (width 0.1))
+  (gr_line (start 132.5 151.2) (end 134 151.6) (layer "Edge.Cuts") (width 0.1))
+  (gr_line (start 131.5 92.5) (end 131.5 93.1) (layer "Edge.Cuts") (width 0.1))
   (gr_circle (center 129.75 103.75) (end 129.75 102.75) (layer "Edge.Cuts") (width 0.1) (fill none))
-  (gr_line (start 131.5 93.6) (end 127.5 93.6) (layer "Edge.Cuts") (width 0.1))
+  (gr_line (start 131 93.6) (end 127.5 93.6) (layer "Edge.Cuts") (width 0.1))
 )

Commit message: Various
Other:
- outline, holes or cut-outs redrawn
Changed lines of the file:
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@@
   (gr_arc (start 195 155.5) (mid 194.853553 155.853553) (end 194.5 156) (layer "Edge.Cuts") (width 0.1))
   (gr_line (start 168.5 93.1) (end 168.5 92.5) (layer "Edge.Cuts") (width 0.1))
-  (gr_line (start 195 150) (end 188 150) (layer "Edge.Cuts") (width 0.1))
-  (gr_line (start 195 106.5) (end 195 150) (layer "Edge.Cuts") (width 0.1))
+  (gr_line (start 194.5 150) (end 188 150) (layer "Edge.Cuts") (width 0.1))
+  (gr_line (start 195 106.5) (end 195 149.5) (layer "Edge.Cuts") (width 0.1))
   (gr_circle (center 131.5 153.5) (end 131.5 152.5) (layer "Edge.Cuts") (width 0.1) (fill none))
   (gr_line (start 127.5 106) (end 127.5 93.6) (layer "Edge.Cuts") (width 0.1))
@@
   (gr_circle (center 170.25 103.75) (end 170.25 102.75) (layer "Edge.Cuts") (width 0.1) (fill none))
   (gr_line (start 169 92) (end 172.5 92) (layer "Edge.Cuts") (width 0.1))
+  (gr_circle (center 129.75 106.5) (end 129.75 105.5) (layer "Edge.Cuts") (width 0.1) (fill none))
   (gr_line (start 188 153) (end 194.5 153) (layer "Edge.Cuts") (width 0.1))
   (gr_arc (start 169 93.6) (mid 168.146447 93.953553) (end 168.5 93.1) (layer "Edge.Cuts") (width 0.1))
@@
   (gr_circle (center 178.25 151.5) (end 178.25 150.5) (layer "Edge.Cuts") (width 0.1) (fill none))
   (gr_line (start 195 153.5) (end 195 155.5) (layer "Edge.Cuts") (width 0.1))
+  (gr_circle (center 170.25 106.5) (end 170.25 105.5) (layer "Edge.Cuts") (width 0.1) (fill none))
   (gr_line (start 128 90) (end 172 90) (layer "Edge.Cuts") (width 0.1))
   (gr_arc (start 187.5 150.5) (mid 187.146447 149.646447) (end 188 150) (layer "Edge.Cuts") (width 0.1))
   (gr_arc (start 131 92) (mid 131.853553 91.646447) (end 131.5 92.5) (layer "Edge.Cuts") (width 0.1))
   (gr_line (start 169.25 156) (end 168.75 153) (layer "Edge.Cuts") (width 0.1))
+  (gr_arc (start 195 149.5) (mid 194.853553 149.853553) (end 194.5 150) (layer "Edge.Cuts") (width 0.1))
   (gr_arc (start 131.5 93.1) (mid 131.853553 93.953553) (end 131 93.6) (layer "Edge.Cuts") (width 0.1))
   (gr_line (start 150 150) (end 132.5 150) (layer "Edge.Cuts") (width 0.1))

Commit message: Various changes
Other:
- board size 90 x 66 mm -> 90 x 71 mm
Changed lines of the file:
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@@
   (gr_line (start 132.5 149) (end 167.5 149)
     (stroke (width 0.15) (type solid)) (layer "Dwgs.User"))
-  (gr_arc (start 172 90) (mid 172.353553 90.146447) (end 172.5 90.5)
+  (gr_arc (start 172 85) (mid 172.353553 85.146447) (end 172.5 85.5)
     (stroke (width 0.1) (type solid)) (layer "Edge.Cuts"))
-  (gr_line (start 168.75 153) (end 175.75 153)
+  (gr_line (start 169.75 153) (end 175.75 153)
     (stroke (width 0.1) (type solid)) (layer "Edge.Cuts"))
   (gr_arc (start 194.5 153) (mid 194.853553 153.146447) (end 195 153.5)
     (stroke (width 0.1) (type solid)) (layer "Edge.Cuts"))
-  (gr_line (start 194.5 156) (end 169.25 156)
+  (gr_line (start 194.5 156) (end 170.25 156)
     (stroke (width 0.1) (type solid)) (layer "Edge.Cuts"))
-  (gr_line (start 172.5 93.6) (end 172.5 106)
+  (gr_line (start 172.5 88.6) (end 172.5 106)
     (stroke (width 0.1) (type solid)) (layer "Edge.Cuts"))
   (gr_line (start 105 155.5) (end 105 150)
@@
   (gr_arc (start 195 155.5) (mid 194.853553 155.853553) (end 194.5 156)
     (stroke (width 0.1) (type solid)) (layer "Edge.Cuts"))
-  (gr_line (start 168.5 93.1) (end 168.5 92.5)
+  (gr_line (start 168.5 88.1) (end 168.5 87.5)
     (stroke (width 0.1) (type solid)) (layer "Edge.Cuts"))
   (gr_line (start 194.5 150) (end 188 150)
@@
   (gr_circle (center 131.5 153.5) (end 131.5 152.5)
     (stroke (width 0.1) (type solid)) (fill none) (layer "Edge.Cuts"))
-  (gr_line (start 127.5 106) (end 127.5 93.6)
+  (gr_line (start 127.5 106) (end 127.5 88.6)
     (stroke (width 0.1) (type solid)) (layer "Edge.Cuts"))
   (gr_arc (start 194.5 106) (mid 194.853553 106.146447) (end 195 106.5)
@@
   (gr_circle (center 170.25 103.75) (end 170.25 102.75)
     (stroke (width 0.1) (type solid)) (fill none) (layer "Edge.Cuts"))
-  (gr_line (start 169 92) (end 172.5 92)
+  (gr_line (start 169 87) (end 172.5 87)
     (stroke (width 0.1) (type solid)) (layer "Edge.Cuts"))
   (gr_circle (center 129.75 106.5) (end 129.75 105.5)
@@
   (gr_line (start 188 153) (end 194.5 153)
     (stroke (width 0.1) (type solid)) (layer "Edge.Cuts"))
-  (gr_arc (start 169 93.6) (mid 168.146447 93.953553) (end 168.5 93.1)
+  (gr_arc (start 169 88.6) (mid 168.146447 88.953553) (end 168.5 88.1)
     (stroke (width 0.1) (type solid)) (layer "Edge.Cuts"))
-  (gr_line (start 127.5 92) (end 131 92)
+  (gr_line (start 127.5 87) (end 131 87)
     (stroke (width 0.1) (type solid)) (layer "Edge.Cuts"))
   (gr_line (start 176.25 152.5) (end 176.25 150.5)
@@
   (gr_line (start 105.5 106) (end 127.5 106)
     (stroke (width 0.1) (type solid)) (layer "Edge.Cuts"))
-  (gr_line (start 172.5 92) (end 172.5 90.5)
+  (gr_line (start 172.5 87) (end 172.5 85.5)
     (stroke (width 0.1) (type solid)) (layer "Edge.Cuts"))
   (gr_circle (center 178.25 151.5) (end 178.25 150.5)
@@
   (gr_circle (center 170.25 106.5) (end 170.25 105.5)
     (stroke (width 0.1) (type solid)) (fill none) (layer "Edge.Cuts"))
-  (gr_line (start 128 90) (end 172 90)
+  (gr_line (start 128 85) (end 172 85)
     (stroke (width 0.1) (type solid)) (layer "Edge.Cuts"))
   (gr_arc (start 187.5 150.5) (mid 187.146447 149.646447) (end 188 150)
     (stroke (width 0.1) (type solid)) (layer "Edge.Cuts"))
-  (gr_arc (start 131 92) (mid 131.853553 91.646447) (end 131.5 92.5)
+  (gr_arc (start 131 87) (mid 131.853553 86.646447) (end 131.5 87.5)
     (stroke (width 0.1) (type solid)) (layer "Edge.Cuts"))
-  (gr_line (start 169.25 156) (end 168.75 153)
+  (gr_line (start 170.25 156) (end 169.75 153)
     (stroke (width 0.1) (type solid)) (layer "Edge.Cuts"))
   (gr_arc (start 195 149.5) (mid 194.853553 149.853553) (end 194.5 150)
     (stroke (width 0.1) (type solid)) (layer "Edge.Cuts"))
-  (gr_arc (start 131.5 93.1) (mid 131.853553 93.953553) (end 131 93.6)
+  (gr_arc (start 131.5 88.1) (mid 131.853553 88.953553) (end 131 88.6)
     (stroke (width 0.1) (type solid)) (layer "Edge.Cuts"))
   (gr_line (start 150 150) (end 132.5 150)
@@
   (gr_line (start 134 151.6) (end 134 156)
     (stroke (width 0.1) (type solid)) (layer "Edge.Cuts"))
-  (gr_line (start 127.5 92) (end 127.5 90.5)
+  (gr_line (start 127.5 87) (end 127.5 85.5)
     (stroke (width 0.1) (type solid)) (layer "Edge.Cuts"))
   (gr_line (start 172.5 106) (end 194.5 106)
@@
   (gr_arc (start 188 153) (mid 187.146447 153.353553) (end 187.5 152.5)
     (stroke (width 0.1) (type solid)) (layer "Edge.Cuts"))
-  (gr_arc (start 127.5 90.5) (mid 127.646447 90.146447) (end 128 90)
+  (gr_arc (start 127.5 85.5) (mid 127.646447 85.146447) (end 128 85)
     (stroke (width 0.1) (type solid)) (layer "Edge.Cuts"))
   (gr_line (start 132.5 150) (end 132.5 151.2)
@@
   (gr_arc (start 105 106.5) (mid 105.146447 106.146447) (end 105.5 106)
     (stroke (width 0.1) (type solid)) (layer "Edge.Cuts"))
-  (gr_arc (start 168.5 92.5) (mid 168.146447 91.646447) (end 169 92)
+  (gr_arc (start 168.5 87.5) (mid 168.146447 86.646447) (end 169 87)
     (stroke (width 0.1) (type solid)) (layer "Edge.Cuts"))
-  (gr_line (start 172.5 93.6) (end 169 93.6)
+  (gr_line (start 172.5 88.6) (end 169 88.6)
     (stroke (width 0.1) (type solid)) (layer "Edge.Cuts"))
   (gr_line (start 187.5 150.5) (end 187.5 152.5)
@@
   (gr_line (start 132.5 151.2) (end 134 151.6)
     (stroke (width 0.1) (type solid)) (layer "Edge.Cuts"))
-  (gr_line (start 131.5 92.5) (end 131.5 93.1)
+  (gr_line (start 131.5 87.5) (end 131.5 88.1)
     (stroke (width 0.1) (type solid)) (layer "Edge.Cuts"))
   (gr_circle (center 129.75 103.75) (end 129.75 102.75)
     (stroke (width 0.1) (type solid)) (fill none) (layer "Edge.Cuts"))
-  (gr_line (start 131 93.6) (end 127.5 93.6)
+  (gr_line (start 131 88.6) (end 127.5 88.6)
     (stroke (width 0.1) (type solid)) (layer "Edge.Cuts"))
 )
