File: pcb/sensactHsHMI_smaller/sensactHsHMI_smaller.kicad_pcb (KiCad board)
At the start: 2 copper layers, 45 x 22 mm, 26 parts, among them J1 Conn_01x10, Q1 AO3400A, Q2 Q_NPN_BEC, Q3 Q_NPN_BEC, SW1 SW_Push, SW5 Rotary_Encoder_Switch_with_Mo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, X1 LH114

Commit message: Various
Parts:
- removed BZ1: Buzzer, liebler_MECH:XDCR_CMT-7525-80-SMT-TR_handsolder
- removed D1: LED, liebler_OPTO:LED_PLCC_2835_Handsoldering
- removed JP2: BUZ_DIR, Jumper:SolderJumper-2_P1.3mm_Bridged_RoundedPad1.0x1.5mm
- removed Q2, Q3: Q_NPN_BEC, liebler_SEMICONDUCTORS:SOT-23_Handsoldering
- removed R10: 1k, Resistor_SMD:R_0805_2012Metric_Pad1.20x1.40mm_HandSolder
- removed TP1: LED_ON, TestPoint:TestPoint_Pad_D2.0mm
- added C3: 10n, Capacitor_SMD:C_0603_1608Metric_Pad1.08x0.95mm_HandSolder, B.Cu at (90.1, 104.0)
- added C4: 1u, Capacitor_SMD:C_0603_1608Metric_Pad1.08x0.95mm_HandSolder, B.Cu at (78.3, 96.0)
- added C5: u1, Capacitor_SMD:C_0603_1608Metric_Pad1.08x0.95mm_HandSolder, B.Cu at (87.2, 94.4)
- added LS1: Speaker, liebler_MECH:Speaker_1511, B.Cu at (106.3, 100.3)
- added U1: MD8002A, liebler_SEMICONDUCTORS:SOIC-8_3.9x4.9mm_P1.27mm_handsolder, B.Cu at (82.8, 95.0)
- C1, C2: footprint Capacitor_SMD:C_0805_2012Metric_Pad1.18x1.45mm_HandSolder -> Capacitor_SMD:C_0603_1608Metric_Pad1.08x0.95mm_HandSolder
- R1, R11, R12, R5, R6, R8, R9: footprint Resistor_SMD:R_0805_2012Metric_Pad1.20x1.40mm_HandSolder -> Resistor_SMD:R_0603_1608Metric_Pad0.98x0.95mm_HandSolder
- R3: value 1k -> k47; footprint Resistor_SMD:R_0805_2012Metric_Pad1.20x1.40mm_HandSolder -> Resistor_SMD:R_0603_1608Metric_Pad0.98x0.95mm_HandSolder
- R4: value 10R -> 10k; footprint Resistor_SMD:R_0805_2012Metric_Pad1.20x1.40mm_HandSolder -> Resistor_SMD:R_0603_1608Metric_Pad0.98x0.95mm_HandSolder
- R7: value k22 -> 22k; footprint Resistor_SMD:R_1206_3216Metric_Pad1.30x1.75mm_HandSolder -> Resistor_SMD:R_0603_1608Metric_Pad0.98x0.95mm_HandSolder
- moved R8 24.3 mm to (90.1, 107.0), turned to 0 degrees
- moved R6 21.7 mm to (90.1, 105.5), turned to 180 degrees
- moved R4 20.2 mm to (90.1, 102.5), turned to 180 degrees
- moved R3 13.9 mm to (90.1, 101.0)
- moved Q1 12.6 mm to (98.0, 106.2)
- moved R12 12.3 mm to (97.8, 102.7)
- moved R9 11.5 mm to (112.8, 106.0), turned to 90 degrees
- moved R1 9.97 mm to (93.5, 107.0), turned to 0 degrees
- moved R7 8.97 mm to (87.2, 97.7), turned to 90 degrees
- moved R5 8.57 mm to (93.8, 104.0), turned to 180 degrees
- moved C1 6.79 mm to (93.8, 105.5), turned to 180 degrees
- moved R2 5.77 mm to (99.5, 102.7), turned to 90 degrees
- moved J1 5.70 mm to (94.2, 100.1), turned to 0 degrees
- moved C2 5.32 mm to (99.7, 95.0)
- moved R11 2.53 mm to (88.8, 94.4), turned to -90 degrees
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Connections:
- R3 pad 2: Net-(Q2-B) -> Net-(C3-Pad2)
- R4 pad 1: Net-(JP2-B) -> Net-(C3-Pad2)
- R4 pad 2: Net-(BZ1-+) -> Net-(U1--IN)
- R7 pad 1: +3.3VP -> Net-(U1--IN)
Routing:
- net +3.3VP: track 55.4 -> 94.9 mm, vias 1 -> 4
- net Net-(U1-VO2): track 0.00 -> 35.7 mm
- net Net-(R8-Pad2): track 3.55 -> 27.8 mm
- net Net-(U1-VO1): track 0.58 -> 23.2 mm, vias 1 -> 0
- net /BUZZER: track 29.0 -> 6.48 mm, vias 0 -> 2
- net Net-(R6-Pad1): track 8.86 -> 30.5 mm
- net Net-(U1--IN): track 0.00 -> 15.3 mm
- net Net-(R9-Pad2): track 14.5 -> 2.40 mm
- net Net-(JP2-B): track 11.4 -> 0.00 mm
- net GND1: track 0.00 -> 7.96 mm, vias 41 -> 19
- net Net-(Q2-B): track 6.84 -> 0.00 mm
- net Net-(C3-Pad2): track 0.00 -> 3.97 mm
- net /SW: track 57.5 -> 53.9 mm
- net Net-(U1-+IN): track 0.00 -> 3.36 mm
- net /BACKLIGHT: track 9.46 -> 6.29 mm
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