File: pcb/sensactHsHMI_smaller/sensactHsHMI_smaller.kicad_sch (KiCad schematic)
At the start: 26 parts, among them J1 Conn_01x10, Q1 AO3400A, Q2 Q_NPN_BEC, Q3 Q_NPN_BEC, SW1 SW_Push, SW5 Rotary_Encoder_Switch_with_Mo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, X1 LH114

Commit message: Various
Parts:
- removed BZ1: Buzzer, liebler_MECH:XDCR_CMT-7525-80-SMT-TR_handsolder, symbol Device:Buzzer
- removed D1: LED, liebler_OPTO:LED_PLCC_2835_Handsoldering, symbol Device:LED
- removed JP2: BUZ_DIR, Jumper:SolderJumper-2_P1.3mm_Bridged_RoundedPad1.0x1.5mm, symbol Jumper:Jumper_2_Bridged
- removed Q2, Q3: Q_NPN_BEC, liebler_SEMICONDUCTORS:SOT-23_Handsoldering, symbol Device:Q_NPN_BEC
- removed R10: 1k, Resistor_SMD:R_0805_2012Metric_Pad1.20x1.40mm_HandSolder, symbol Device:R
- removed TP1: LED_ON, TestPoint:TestPoint_Pad_D2.0mm, symbol Connector:TestPoint
- added C3: 10n, Capacitor_SMD:C_0603_1608Metric_Pad1.08x0.95mm_HandSolder, symbol Device:C
- added C4: 1u, Capacitor_SMD:C_0603_1608Metric_Pad1.08x0.95mm_HandSolder, symbol Device:C
- added C5: u1, Capacitor_SMD:C_0603_1608Metric_Pad1.08x0.95mm_HandSolder, symbol Device:C
- added LS1: Speaker, liebler_MECH:Speaker_1511, symbol Device:Speaker
- added U1: MD8002A, liebler_SEMICONDUCTORS:SOIC-8_3.9x4.9mm_P1.27mm_handsolder, symbol liebler_SEMICONDUCTORS:MD8002A
- C1, C2: footprint Capacitor_SMD:C_0805_2012Metric_Pad1.18x1.45mm_HandSolder -> Capacitor_SMD:C_0603_1608Metric_Pad1.08x0.95mm_HandSolder
- R1, R11, R12, R5, R6, R8, R9: footprint Resistor_SMD:R_0805_2012Metric_Pad1.20x1.40mm_HandSolder -> Resistor_SMD:R_0603_1608Metric_Pad0.98x0.95mm_HandSolder
- R3: value 1k -> k47; footprint Resistor_SMD:R_0805_2012Metric_Pad1.20x1.40mm_HandSolder -> Resistor_SMD:R_0603_1608Metric_Pad0.98x0.95mm_HandSolder
- R4: value 10R -> 10k; footprint Resistor_SMD:R_0805_2012Metric_Pad1.20x1.40mm_HandSolder -> Resistor_SMD:R_0603_1608Metric_Pad0.98x0.95mm_HandSolder
- R7: value k22 -> 22k; footprint Resistor_SMD:R_1206_3216Metric_Pad1.30x1.75mm_HandSolder -> Resistor_SMD:R_0603_1608Metric_Pad0.98x0.95mm_HandSolder
Connections:
- net +3.3VP: now also C5.1, U1.6 (VDD); no longer R7.1
- net GND1: now also C3.1, C4.1, C5.2, U1.1 (SD), U1.7 (GND)
- net at R3.2: now also R4.1, C3.2
- net at R4.2: now also R7.1, U1.4 (-IN)
- net at R7.2: now also LS1.2, U1.5 (VO1)
- new net: LS1.1, U1.8 (VO2)
- new net: C4.2, U1.2 (BYP), U1.3 (+IN)
