File: pcb/sensactUpBase/sensactUpBase.kicad_pcb (KiCad board)
At the start: 2 copper layers, 50 x 50 mm, 8 parts, among them J1 BaseConnect, J10 24 GN CH CL 24 GN CH CL, J3 T2 T1 T1, J4 B RS485 A, J9 T3 T4 T5 T6 T7 GN 3V GN SC SD, U1 PCA9555PW

Commit message: Updated various PCB
Parts:
- J4: value B RS485 A -> A RS485 B
Connections:
- J1 pad 1: RS485B -> RS485A
- J1 pad 3: RS485A -> RS485B
- J1 pad 6: GND -> SDA
- J1 pad 7: SDA -> GND
- J4 pad 1: RS485A -> RS485B
- J4 pad 3: RS485B -> RS485A
Routing:
- net SDA: track 38.8 -> 46.0 mm
- net RS485A: track 11.8 -> 10.2 mm

Commit message: PCBs as ordered at JLCPCB
Parts:
- added J5: Conn_01x04, Connector_PinHeader_2.54mm:PinHeader_1x04_P2.54mm_Vertical, F.Cu at (119.1, 113.2)
- J3: value T2 T1 T1 -> GND T0 T1
- J9: value T3 T4 T5 T6 T7 GN 3V GN SC SD -> T11 T10 T9 T8 T7 T6 T5 T4 T3 T2
- moved C1 2.19 mm to (114.0, 94.1)
- moved C2 2.12 mm to (112.0, 94.1)
Connections:
- J3 pad 1: /T2 -> GND
- J3 pad 2: /T1 -> /T0
- J3 pad 3: /T0 -> /T1
- J9 pad 1: /T3 -> /T11
- J9 pad 10: SDA -> /T2
- J9 pad 2: /T4 -> /T10
- J9 pad 3: /T5 -> /T9
- J9 pad 4: /T6 -> /T8
- J9 pad 6: GND -> /T6
- J9 pad 7: +3V3 -> /T5
- J9 pad 8: GND -> /T4
- J9 pad 9: SCL -> /T3
- U1 pad 10: unconnected-(U1-Pad10) -> /T6
- U1 pad 11: unconnected-(U1-Pad11) -> /T7
- U1 pad 13: /T0 -> /T8
- U1 pad 14: /T1 -> /T9
- U1 pad 15: /T2 -> /T10
- U1 pad 16: /T3 -> /T11
- U1 pad 17: /T4 -> unconnected-(U1-Pad17)
- U1 pad 18: /T5 -> unconnected-(U1-Pad18)
- U1 pad 19: /T6 -> unconnected-(U1-Pad19)
- U1 pad 20: /T7 -> unconnected-(U1-Pad20)
- U1 pad 4: unconnected-(U1-Pad4) -> /T0
- U1 pad 5: unconnected-(U1-Pad5) -> /T1
- U1 pad 6: unconnected-(U1-Pad6) -> /T2
- U1 pad 7: unconnected-(U1-Pad7) -> /T3
- U1 pad 8: unconnected-(U1-Pad8) -> /T4
- U1 pad 9: unconnected-(U1-Pad9) -> /T5
Routing:
- net /T11: track 0.00 -> 23.6 mm
- net /T2: track 38.2 -> 21.6 mm
- net /T9: track 0.00 -> 16.2 mm
- net /T10: track 0.00 -> 13.7 mm
- net +3V3: track 18.1 -> 31.1 mm
- net SDA: track 46.0 -> 34.6 mm
- net /T1: track 42.8 -> 34.7 mm
- net /T7: track 9.06 -> 16.7 mm, vias 0 -> 1
- net /T4: track 12.4 -> 19.2 mm
- net /T6: track 6.77 -> 12.6 mm, vias 0 -> 1
- net /T8: track 0.00 -> 4.59 mm
- net /T3: track 20.3 -> 24.7 mm
- net /T5: track 14.8 -> 18.6 mm, vias 0 -> 1
- net /T0: track 35.4 -> 36.2 mm
- net SCL: track 32.6 -> 32.0 mm
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Other:
- board text added: "GN SC SD 3V"

Commit message: sensactUpControl
Parts:
- added N1: Housing, Symbol:KiCad-Logo2_5mm_SilkScreen, F.Cu at (100.0, 100.0)
- C2: value u1 -> 1u
