File: pcb/sensactUp_as_Hs/sensactUp_as_Hs.kicad_sch (KiCad schematic)
At the start: 55 parts, among them J10 ROT1, J11 OneWire, J12 LED Driver, J2 SensactBusConnector, J3 24V+CAN IN, J4 LED, J5 ROT2, J6 LED Driver, J7 LED, J8 LED, J9 LED, SW3 TERM OFF, U1 DS18B20, U10 TPL7407LAPW, U11 DS2482, U2 ESP32-S3-DevKitC, U3 DCDC_MP2315, U4 DCDC_MP2315, U5 SN65HVD230, U7 PCA9685PW, U8 MAX98357_MODULE, U9 TPL7407LAPW

Commit message: added sensactUp_as_Hs and fixed various compile errors. Untested!
Parts:
- removed R7: 1k, Resistor_SMD:R_0805_2012Metric_Pad1.20x1.40mm_HandSolder, symbol Device:R
- added C7: u1, Capacitor_SMD:C_0805_2012Metric_Pad1.18x1.45mm_HandSolder, symbol Device:C
- added J1: 5V OUT, liebler_CONN:PhoenixContact_MCV_1,5_5-G-3.81_1x05_P3.81mm_Vertical_smallerCourtyard, symbol Connector_Generic:Conn_01x05
- added U6: 74AHCT125, liebler_SEMICONDUCTORS:SOIC-14_3.9x8.7mm_P1.27mm_handsolder, symbol 74xx:74AHCT125
Connections:
- net +12V: now also J1.2 (Pin_2)
- net +24V: now also J1.5 (Pin_5)
- net +5V: now also C7.2, U6.14 (VCC)
- net GND: now also C7.1, J1.1 (Pin_1), U6.1, U6.10, U6.12, U6.13, U6.4, U6.7 (GND), U6.9
- net L1: now also U2.11 (GPIO18/ADC2_CH7); no longer U2.10 (GPIO17/ADC2_CH6)
- net L2: now also U2.12 (GPIO8/ADC1_CH7); no longer U2.11 (GPIO18/ADC2_CH7)
- net L4: now also U2.13 (GPIO3/ADC1_CH2); no longer U2.12 (GPIO8/ADC1_CH7)
- net Onewire: no longer U1.2 (DQ), U2.13 (GPIO3/ADC1_CH2)
- net OneWireExt: now reaches J11.4 (Pin_4), U11.2 (IO)
- net OneWireExt: now also U1.2 (DQ)
- net RGB_11: now reaches U2.33 (GPIO36)
- net RGB_11: now also U6.5
- new net RGB_1: J1.3 (Pin_3), U6.6
- new net RGB_2: J1.4 (Pin_4), U6.3
- new net RGB_22: U2.10 (GPIO17/ADC2_CH6), U6.2
- no-connect marks 14 -> 13
Other:
- note added: "CAN"
- note added: "CPU"
- note added: "Connectors"
- note added: "Debounce"
- note added: "I2C-Expander"
- note added: "Low Side Driver"
- note added: "OneWire"
- note added: "PSU"
- note added: "Pull-Ups"
- note added: "SensactBus"
- note added: "Sound"
- moved on the sheet: C1, C10, C11, C12, C2, C3, C4, C5, C6, C8, C9, D1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
